File: HARDWARE/ETH1CREF1A/Isolation.kicad_sch (KiCad schematic)
At the start: 2 parts, among them U904 ADuM1401xRW

Commit message: Hardware
Connections:
- net +5V: no longer R909.1, U904.1 (VDD1)
- new net +3.3V: R909.1, U904.1 (VDD1)
Changed lines of the file:
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@@
     (effects (font (size 1.27 1.27)) (justify left))
-  )
-  (symbol (lib_id "power:+5V") (at 102.235 71.12 0) (unit 1)
-    (in_bom yes) (on_board yes) (dnp no) (fields_autoplaced)
-    (property "Reference" "#PWR0925" (at 102.235 74.93 0)
-      (effects (font (size 1.27 1.27)) hide)
-    )
-    (property "Value" "+5V" (at 102.235 66.675 0)
-      (effects (font (size 1.27 1.27)))
-    )
-    (property "Footprint" "" (at 102.235 71.12 0)
-      (effects (font (size 1.27 1.27)) hide)
-    )
-    (property "Datasheet" "" (at 102.235 71.12 0)
-      (effects (font (size 1.27 1.27)) hide)
-    )
-    (pin "1")
-    (instances
-      (project "ETH1CREF1A"
-        (path "/f534bde3-7724-4aa2-8c73-8f0531e01e95/ebac98f6-7cea-4b7b-a7eb-72e971f44089"
-          (reference "#PWR0925") (unit 1)
-        )
-        (path "/f534bde3-7724-4aa2-8c73-8f0531e01e95/2dec562b-bf90-4748-bf0c-0c9213a8713f"
-          (reference "#PWR01030") (unit 1)
-        )
-      )
-    )
   )
   (symbol (lib_id "Isolator:ADuM1401xRW") (at 136.525 88.265 0) (unit 1)
@@
     )
   )
+  (symbol (lib_id "power:+3.3V") (at 120.015 71.12 0) (unit 1)
+    (in_bom yes) (on_board yes) (dnp no)
+    (property "Reference" "#PWR01037" (at 120.015 74.93 0)
+      (effects (font (size 1.27 1.27)) hide)
+    )
+    (property "Value" "+3.3V" (at 120.015 66.675 0)
+      (effects (font (size 1.27 1.27)))
+    )
+    (property "Footprint" "" (at 120.015 71.12 0)
+      (effects (font (size 1.27 1.27)) hide)
+    )
+    (property "Datasheet" "" (at 120.015 71.12 0)
+      (effects (font (size 1.27 1.27)) hide)
+    )
+    (pin "1")
+    (instances
+      (project "ETH1CREF1A"
+        (path "/f534bde3-7724-4aa2-8c73-8f0531e01e95/2dec562b-bf90-4748-bf0c-0c9213a8713f"
+          (reference "#PWR01037") (unit 1)
+        )
+      )
+    )
+  )
   (symbol (lib_id "ETH1CREF1A:+5VF") (at 151.765 93.345 270) (unit 1)
     (in_bom yes) (on_board yes) (dnp no) (fields_autoplaced)
@@
     )
   )
+  (symbol (lib_id "power:+3.3V") (at 102.235 71.12 0) (unit 1)
+    (in_bom yes) (on_board yes) (dnp no)
+    (property "Reference" "#PWR01030" (at 102.235 74.93 0)
+      (effects (font (size 1.27 1.27)) hide)
+    )
+    (property "Value" "+3.3V" (at 102.235 66.675 0)
+      (effects (font (size 1.27 1.27)))
+    )
+    (property "Footprint" "" (at 102.235 71.12 0)
+      (effects (font (size 1.27 1.27)) hide)
+    )
+    (property "Datasheet" "" (at 102.235 71.12 0)
+      (effects (font (size 1.27 1.27)) hide)
+    )
+    (pin "1")
+    (instances
+      (project "ETH1CREF1A"
+        (path "/f534bde3-7724-4aa2-8c73-8f0531e01e95/2dec562b-bf90-4748-bf0c-0c9213a8713f"
+          (reference "#PWR01030") (unit 1)
+        )
+      )
+    )
+  )
   (symbol (lib_id "ETH1CREF1A:+5VF") (at 153.67 71.755 0) (unit 1)
     (in_bom yes) (on_board yes) (dnp no) (fields_autoplaced)
@@
         )
       )
-    )
-  )
-  (symbol (lib_id "power:+5V") (at 120.015 71.12 0) (unit 1)
-    (in_bom yes) (on_board yes) (dnp no) (fields_autoplaced)
-    (property "Reference" "#PWR0922" (at 120.015 74.93 0)
-      (effects (font (size 1.27 1.27)) hide)
-    )
-    (property "Value" "+5V" (at 120.015 66.675 0)
-      (effects (font (size 1.27 1.27)))
-    )
-    (property "Footprint" "" (at 120.015 71.12 0)
-      (effects (font (size 1.27 1.27)) hide)
-    )
-    (property "Datasheet" "" (at 120.015 71.12 0)
-      (effects (font (size 1.27 1.27)) hide)
-    )
-    (pin "1")
-    (instances
-      (project "ETH1CREF1A"
-        (path "/f534bde3-7724-4aa2-8c73-8f0531e01e95/ebac98f6-7cea-4b7b-a7eb-72e971f44089"
-          (reference "#PWR0922") (unit 1)
-        )
-        (path "/f534bde3-7724-4aa2-8c73-8f0531e01e95/2dec562b-bf90-4748-bf0c-0c9213a8713f"
-          (reference "#PWR01031") (unit 1)
-        )
-      )
