File: HARDWARE/ETH1CREF1A/Power_Float.kicad_sch (KiCad schematic)
At the start: 46 parts, among them U302 THL15-2415WI, U403 LT8330_S6, U404 LT8330_S6, U406 MC7815BD2TG, U407 MC7915BD2TG, U408 TSR1-2490, U409 LM1117DTX-5.0/NOPB

Commit message: Hardware
Connections:
- net +24V renamed VCCQ
Changed lines of the file:
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@@
     (stroke (width 0) (type default))
-  )
-  (symbol (lib_id "power:+24V") (at 20.32 24.13 0) (unit 1)
-    (in_bom yes) (on_board yes) (dnp no) (fields_autoplaced)
-    (property "Reference" "#PWR0748" (at 20.32 27.94 0)
-      (effects (font (size 1.27 1.27)) hide)
-    )
-    (property "Value" "+24V" (at 20.32 19.05 0)
-      (effects (font (size 1.27 1.27)))
-    )
-    (property "Footprint" "" (at 20.32 24.13 0)
-      (effects (font (size 1.27 1.27)) hide)
-    )
-    (property "Datasheet" "" (at 20.32 24.13 0)
-      (effects (font (size 1.27 1.27)) hide)
-    )
-    (pin "1")
-    (instances
-      (project "ETH1CREF1A"
-        (path "/f534bde3-7724-4aa2-8c73-8f0531e01e95/a041155b-e8ef-423b-852e-7aa27332d611"
-          (reference "#PWR0748") (unit 1)
-        )
-      )
-    )
   )
   (symbol (lib_id "Device:C") (at 117.475 38.735 0) (unit 1)
@@
         )
       )
+    )
+  )
+  (symbol (lib_id "power:VCCQ") (at 20.32 24.13 0) (unit 1)
+    (in_bom yes) (on_board yes) (dnp no) (fields_autoplaced)
+    (property "Reference" "#PWR0605" (at 20.32 27.94 0)
+      (effects (font (size 1.27 1.27)) hide)
+    )
+    (property "Value" "VCCQ" (at 20.32 19.685 0)
+      (effects (font (size 1.27 1.27)))
+    )
+    (property "Footprint" "" (at 20.32 24.13 0)
+      (effects (font (size 1.27 1.27)) hide)
+    )
+    (property "Datasheet" "" (at 20.32 24.13 0)
+      (effects (font (size 1.27 1.27)) hide)
+    )
+    (pin "1")
+    (instances
+      (project "ETH1CREF1A"
+        (path "/f534bde3-7724-4aa2-8c73-8f0531e01e95/62654dcd-3414-4e70-b8e6-16734596bf10"
+          (reference "#PWR0605") (unit 1)
+        )
+        (path "/f534bde3-7724-4aa2-8c73-8f0531e01e95/a041155b-e8ef-423b-852e-7aa27332d611"
+          (reference "#PWR0750") (unit 1)
+        )
+      )
