File: HARDWARE/ETH1CREF1A/Connect.kicad_sch (KiCad schematic)
At the start: 1 part, among them J301 C64AC

Commit message: Hardware
Connections:
- net GND renamed GNDPWR
Changed lines of the file:
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@@
+    )
+  )
+  (symbol (lib_id "power:GNDPWR") (at 91.44 161.29 270) (unit 1)
+    (in_bom yes) (on_board yes) (dnp no)
+    (property "Reference" "#PWR054" (at 86.36 161.29 0)
+      (effects (font (size 1.27 1.27)) hide)
+    )
+    (property "Value" "GNDPWR" (at 88.265 161.29 90)
+      (effects (font (size 1.27 1.27)) (justify right))
+    )
+    (property "Footprint" "" (at 90.17 161.29 0)
+      (effects (font (size 1.27 1.27)) hide)
+    )
+    (property "Datasheet" "" (at 90.17 161.29 0)
+      (effects (font (size 1.27 1.27)) hide)
+    )
+    (pin "1")
+    (instances
+      (project "LVPREAMP"
+        (path "/d9f0a433-7915-4d06-b15f-b0ab88f0ad0e/21a7a1f7-d5d8-4a6f-a62d-dc3b0da715d9"
+          (reference "#PWR054") (unit 1)
+        )
+      )
+      (project "ETH1CREF1A"
+        (path "/f534bde3-7724-4aa2-8c73-8f0531e01e95/62654dcd-3414-4e70-b8e6-16734596bf10"
+          (reference "#PWR0602") (unit 1)
+        )
+        (path "/f534bde3-7724-4aa2-8c73-8f0531e01e95/9ff2535d-59f2-4797-8e3c-626128a41417"
+          (reference "#PWR0501") (unit 1)
+        )
+      )
     )
   )
@@
         )
       )
-    )
-  )
-  (symbol (lib_id "power:GND") (at 91.44 161.29 270) (unit 1)
-    (in_bom yes) (on_board yes) (dnp no)
-    (property "Reference" "#PWR0305" (at 85.09 161.29 0)
-      (effects (font (size 1.27 1.27)) hide)
-    )
-    (property "Value" "GND" (at 87.0458 161.417 0)
-      (effects (font (size 1.27 1.27)))
-    )
-    (property "Footprint" "" (at 91.44 161.29 0)
-      (effects (font (size 1.27 1.27)) hide)
-    )
-    (property "Datasheet" "" (at 91.44 161.29 0)
-      (effects (font (size 1.27 1.27)) hide)
-    )
-    (pin "1")
-    (instances
-      (project "ETH1CSMU2"
-        (path "/1fc6a863-b4aa-4691-87d2-d385f614c99b/be6d7d94-212c-4f17-9376-b8ad68397098"
-          (reference "#PWR0305") (unit 1)
-        )
-      )
-      (project "ETH1CREF1A"
-        (path "/f534bde3-7724-4aa2-8c73-8f0531e01e95/9ff2535d-59f2-4797-8e3c-626128a41417"
-          (reference "#PWR0305") (unit 1)
-        )
-      )

Commit message: Hardware
Changed lines of the file:
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@@
     (stroke (width 0) (type default))
-  )
-  (label "D" (at 86.36 46.99 0) (fields_autoplaced)
-    (effects (font (size 1.27 1.27)) (justify left bottom))
-  )
-  (label "A" (at 86.36 31.75 0) (fields_autoplaced)
-    (effects (font (size 1.27 1.27)) (justify left bottom))
   )
   (label "TX+" (at 87.63 124.46 0) (fields_autoplaced)
     (effects (font (size 1.27 1.27)) (justify left bottom))
   )
-  (label "F" (at 86.36 57.15 0) (fields_autoplaced)
-    (effects (font (size 1.27 1.27)) (justify left bottom))
-  )
   (label "TX-" (at 87.63 129.54 0) (fields_autoplaced)
     (effects (font (size 1.27 1.27)) (justify left bottom))
@@
     (effects (font (size 1.27 1.27)) (justify left bottom))
   )
-  (label "E" (at 86.36 52.07 0) (fields_autoplaced)
-    (effects (font (size 1.27 1.27)) (justify left bottom))
-  )
-  (label "B" (at 86.36 36.83 0) (fields_autoplaced)
-    (effects (font (size 1.27 1.27)) (justify left bottom))
-  )
   (label "RX-" (at 87.63 127 0) (fields_autoplaced)
     (effects (font (size 1.27 1.27)) (justify left bottom))
   )
-  (label "C" (at 86.36 41.91 0) (fields_autoplaced)
-    (effects (font (size 1.27 1.27)) (justify left bottom))
+  (hierarchical_label "E" (shape bidirectional) (at 86.36 52.07 180) (fields_autoplaced)
+    (effects (font (size 1.27 1.27)) (justify right))
   )
   (hierarchical_label "RX+" (shape bidirectional) (at 86.36 121.92 180) (fields_autoplaced)
     (effects (font (size 1.27 1.27)) (justify right))
   )
+  (hierarchical_label "A" (shape bidirectional) (at 86.36 31.75 180) (fields_autoplaced)
+    (effects (font (size 1.27 1.27)) (justify right))
+  )
+  (hierarchical_label "D" (shape bidirectional) (at 86.36 46.99 180) (fields_autoplaced)
+    (effects (font (size 1.27 1.27)) (justify right))
+  )
+  (hierarchical_label "C" (shape bidirectional) (at 86.36 41.91 180) (fields_autoplaced)
+    (effects (font (size 1.27 1.27)) (justify right))
+  )
   (hierarchical_label "TX+" (shape bidirectional) (at 86.36 124.46 180) (fields_autoplaced)
     (effects (font (size 1.27 1.27)) (justify right))
@@
   )
   (hierarchical_label "RX-" (shape bidirectional) (at 86.36 127 180) (fields_autoplaced)
+    (effects (font (size 1.27 1.27)) (justify right))
+  )
+  (hierarchical_label "B" (shape bidirectional) (at 86.36 36.83 180) (fields_autoplaced)
+    (effects (font (size 1.27 1.27)) (justify right))
+  )
+  (hierarchical_label "F" (shape bidirectional) (at 86.36 57.15 180) (fields_autoplaced)
     (effects (font (size 1.27 1.27)) (justify right))
   )
@@
       (project "ETH1CREF1A"
         (path "/f534bde3-7724-4aa2-8c73-8f0531e01e95/9ff2535d-59f2-4797-8e3c-626128a41417"
-          (reference "#FLG0301") (unit 1)
+          (reference "#FLG0501") (unit 1)
         )
       )
@@
       (project "ETH1CREF1A"
         (path "/f534bde3-7724-4aa2-8c73-8f0531e01e95/9ff2535d-59f2-4797-8e3c-626128a41417"
-          (reference "#PWR0306") (unit 1)
+          (reference "#PWR0504") (unit 1)
         )
       )
@@
         )
         (path "/f534bde3-7724-4aa2-8c73-8f0531e01e95/9ff2535d-59f2-4797-8e3c-626128a41417"
+          (reference "#PWR0503") (unit 1)
+        )
+      )
+    )
+  )
+  (symbol (lib_id "power:Earth") (at 91.44 133.35 270) (unit 1)
+    (in_bom yes) (on_board yes) (dnp no)
+    (property "Reference" "#PWR0304" (at 85.09 133.35 0)
+      (effects (font (size 1.27 1.27)) hide)
+    )
+    (property "Value" "Earth" (at 87.63 133.35 0)
+      (effects (font (size 1.27 1.27)) hide)
+    )
+    (property "Footprint" "" (at 91.44 133.35 0)
+      (effects (font (size 1.27 1.27)) hide)
+    )
+    (property "Datasheet" "~" (at 91.44 133.35 0)
+      (effects (font (size 1.27 1.27)) hide)
+    )
+    (pin "1")
+    (instances
+      (project "ETH1CSMU2"
+        (path "/1fc6a863-b4aa-4691-87d2-d385f614c99b/be6d7d94-212c-4f17-9376-b8ad68397098"
+          (reference "#PWR0304") (unit 1)
+        )
+      )
+      (project "ETH1CREF1A"
+        (path "/f534bde3-7724-4aa2-8c73-8f0531e01e95/9ff2535d-59f2-4797-8e3c-626128a41417"
+          (reference "#PWR0502") (unit 1)
+        )
+      )
+    )
+  )
+  (symbol (lib_id "power:Earth") (at 91.44 113.03 270) (unit 1)
+    (in_bom yes) (on_board yes) (dnp no)
+    (property "Reference" "#PWR0303" (at 85.09 113.03 0)
+      (effects (font (size 1.27 1.27)) hide)
+    )
+    (property "Value" "Earth" (at 87.63 113.03 0)
+      (effects (font (size 1.27 1.27)) hide)
+    )
+    (property "Footprint" "" (at 91.44 113.03 0)
+      (effects (font (size 1.27 1.27)) hide)
+    )
+    (property "Datasheet" "~" (at 91.44 113.03 0)
+      (effects (font (size 1.27 1.27)) hide)
+    )
+    (pin "1")
+    (instances
+      (project "ETH1CSMU2"
+        (path "/1fc6a863-b4aa-4691-87d2-d385f614c99b/be6d7d94-212c-4f17-9376-b8ad68397098"
+          (reference "#PWR0303") (unit 1)
+        )
+      )
+      (project "ETH1CREF1A"
+        (path "/f534bde3-7724-4aa2-8c73-8f0531e01e95/9ff2535d-59f2-4797-8e3c-626128a41417"
           (reference "#PWR0501") (unit 1)
-        )
-      )
-    )
-  )
-  (symbol (lib_id "power:Earth") (at 91.44 133.35 270) (unit 1)
-    (in_bom yes) (on_board yes) (dnp no)
-    (property "Reference" "#PWR0304" (at 85.09 133.35 0)
-      (effects (font (size 1.27 1.27)) hide)
-    )
-    (property "Value" "Earth" (at 87.63 133.35 0)
-      (effects (font (size 1.27 1.27)) hide)
-    )
-    (property "Footprint" "" (at 91.44 133.35 0)
-      (effects (font (size 1.27 1.27)) hide)
-    )
-    (property "Datasheet" "~" (at 91.44 133.35 0)
-      (effects (font (size 1.27 1.27)) hide)
-    )
-    (pin "1")
-    (instances
-      (project "ETH1CSMU2"
-        (path "/1fc6a863-b4aa-4691-87d2-d385f614c99b/be6d7d94-212c-4f17-9376-b8ad68397098"
-          (reference "#PWR0304") (unit 1)
-        )
-      )
-      (project "ETH1CREF1A"
-        (path "/f534bde3-7724-4aa2-8c73-8f0531e01e95/9ff2535d-59f2-4797-8e3c-626128a41417"
-          (reference "#PWR0304") (unit 1)
-        )
-      )
-    )
-  )
-  (symbol (lib_id "power:Earth") (at 91.44 113.03 270) (unit 1)
-    (in_bom yes) (on_board yes) (dnp no)
-    (property "Reference" "#PWR0303" (at 85.09 113.03 0)
-      (effects (font (size 1.27 1.27)) hide)
-    )
-    (property "Value" "Earth" (at 87.63 113.03 0)
-      (effects (font (size 1.27 1.27)) hide)
-    )
-    (property "Footprint" "" (at 91.44 113.03 0)
-      (effects (font (size 1.27 1.27)) hide)
-    )
-    (property "Datasheet" "~" (at 91.44 113.03 0)
-      (effects (font (size 1.27 1.27)) hide)
-    )
-    (pin "1")
-    (instances
-      (project "ETH1CSMU2"
-        (path "/1fc6a863-b4aa-4691-87d2-d385f614c99b/be6d7d94-212c-4f17-9376-b8ad68397098"
-          (reference "#PWR0303") (unit 1)
-        )
-      )
-      (project "ETH1CREF1A"
-        (path "/f534bde3-7724-4aa2-8c73-8f0531e01e95/9ff2535d-59f2-4797-8e3c-626128a41417"
-          (reference "#PWR0303") (unit 1)
         )
       )
@@
       (project "ETH1CREF1A"
         (path "/f534bde3-7724-4aa2-8c73-8f0531e01e95/9ff2535d-59f2-4797-8e3c-626128a41417"
-          (reference "#PWR0307") (unit 1)
+          (reference "#PWR0505") (unit 1)
         )
       )
@@
       (project "ETH1CREF1A"
         (path "/f534bde3-7724-4aa2-8c73-8f0531e01e95/9ff2535d-59f2-4797-8e3c-626128a41417"
-          (reference "J301") (unit 1)
+          (reference "J501") (unit 1)
         )
       )
@@
       (project "ETH1CREF1A"
         (path "/f534bde3-7724-4aa2-8c73-8f0531e01e95/9ff2535d-59f2-4797-8e3c-626128a41417"
-          (reference "#PWR0308") (unit 1)
-        )
-      )
+          (reference "#PWR0506") (unit 1)
+        )
+      )

Commit message: Hardware
Parts:
- J301: footprint ETH1CSMU2:Socket_DIN41612-CaseC1-AC-Male-64Pin-2rows -> ETH1CREF1A:Socket_DIN41612-CaseC1-AC-Male-64Pin-2rows
Changed lines of the file:
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@@
     (effects (font (size 1.27 1.27)) (justify right))
-  )
-  (symbol (lib_id "power:PWR_FLAG") (at 116.84 182.88 180) (unit 1)
-    (in_bom yes) (on_board yes) (dnp no) (fields_autoplaced)
-    (property "Reference" "#FLG0301" (at 116.84 184.785 0)
-      (effects (font (size 1.27 1.27)) hide)
-    )
-    (property "Value" "PWR_FLAG" (at 116.84 187.3234 0)
-      (effects (font (size 1.27 1.27)))
-    )
-    (property "Footprint" "" (at 116.84 182.88 0)
-      (effects (font (size 1.27 1.27)) hide)
-    )
-    (property "Datasheet" "~" (at 116.84 182.88 0)
-      (effects (font (size 1.27 1.27)) hide)
-    )
-    (pin "1")
-    (instances
-      (project "ETH1CSMU2"
-        (path "/1fc6a863-b4aa-4691-87d2-d385f614c99b/be6d7d94-212c-4f17-9376-b8ad68397098"
-          (reference "#FLG0301") (unit 1)
-        )
-      )
-      (project "ETH1CREF1A"
-        (path "/f534bde3-7724-4aa2-8c73-8f0531e01e95/9ff2535d-59f2-4797-8e3c-626128a41417"
-          (reference "#FLG0501") (unit 1)
-        )
-      )
-    )
   )
   (symbol (lib_id "power:+24V") (at 91.44 181.61 90) (unit 1)
@@
       (effects (font (size 1.27 1.27)) (justify left))
     )
-    (property "Footprint" "ETH1CSMU2:Socket_DIN41612-CaseC1-AC-Male-64Pin-2rows" (at 101.6 105.41 0)
+    (property "Footprint" "ETH1CREF1A:Socket_DIN41612-CaseC1-AC-Male-64Pin-2rows" (at 101.6 105.41 0)
       (effects (font (size 1.27 1.27)) hide)
     )
@@
         )
       )
-    )
-  )
-  (symbol (lib_id "power:+24V") (at 116.84 182.88 0) (unit 1)
-    (in_bom yes) (on_board yes) (dnp no) (fields_autoplaced)
-    (property "Reference" "#PWR0308" (at 116.84 186.69 0)
-      (effects (font (size 1.27 1.27)) hide)
-    )
-    (property "Value" "+24V" (at 116.84 179.3042 0)
-      (effects (font (size 1.27 1.27)))
-    )
-    (property "Footprint" "" (at 116.84 182.88 0)
-      (effects (font (size 1.27 1.27)) hide)
-    )
-    (property "Datasheet" "" (at 116.84 182.88 0)
-      (effects (font (size 1.27 1.27)) hide)
-    )
-    (pin "1")
-    (instances
-      (project "ETH1CSMU2"
-        (path "/1fc6a863-b4aa-4691-87d2-d385f614c99b/be6d7d94-212c-4f17-9376-b8ad68397098"
-          (reference "#PWR0308") (unit 1)
-        )
-      )
-      (project "ETH1CREF1A"
-        (path "/f534bde3-7724-4aa2-8c73-8f0531e01e95/9ff2535d-59f2-4797-8e3c-626128a41417"
-          (reference "#PWR0506") (unit 1)
-        )
-      )

Commit message: Hardware
Other:
- moved on the sheet: J301
