File: HARDWARE/ETH1CREF1A/Ethernet.kicad_sch (KiCad schematic)
At the start: 43 parts, among them U201 LAN8742A, U202 LC03-3.3, U203 LC03-3.3, Y201 NX5032GA-25.000000MHZ-LN-CD-1

Commit message: Hardware
Parts:
- L201: footprint ETH1CSMU2:749010012A -> ETH1CREF1A:749010012A
- U202, U203: footprint ETH1CSMU2:SO8E -> ETH1CREF1A:SO8E
- Y201: footprint ETH1CSMU2:NX5032GA -> ETH1CREF1A:NX5032GA
Changed lines of the file:
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@@
       (effects (font (size 1.27 1.27)))
     )
-    (property "Footprint" "ETH1CSMU2:749010012A" (at 234.95 74.93 0)
+    (property "Footprint" "ETH1CREF1A:749010012A" (at 234.95 74.93 0)
       (effects (font (size 1.27 1.27)) hide)
     )
@@
       (effects (font (size 1.524 1.524)))
     )
-    (property "Footprint" "ETH1CSMU2:SO8E" (at 262.89 72.39 0)
+    (property "Footprint" "ETH1CREF1A:SO8E" (at 262.89 72.39 0)
       (effects (font (size 1.524 1.524)) hide)
     )
@@
       (effects (font (size 1.524 1.524)))
     )
-    (property "Footprint" "ETH1CSMU2:SO8E" (at 262.89 92.71 0)
+    (property "Footprint" "ETH1CREF1A:SO8E" (at 262.89 92.71 0)
       (effects (font (size 1.524 1.524)) hide)
     )
@@
       (effects (font (size 1.27 1.27)))
     )
-    (property "Footprint" "ETH1CSMU2:NX5032GA" (at 44.45 120.65 0)
-      (effects (font (size 1.27 1.27)) hide)
-    )
+    (property "Footprint" "ETH1CREF1A:NX5032GA" (at 44.45 120.65 0)
+      (effects (font (size 1.27 1.27)) hide)
+    )

Commit message: Hardware and software
Changed lines of the file:
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@@
+    (effects (font (size 1.27 1.27)) (justify left bottom))
+  )
+  (label "MODE0" (at 53.34 191.77 90) (fields_autoplaced)
     (effects (font (size 1.27 1.27)) (justify left bottom))
   )
   (label "MODE2" (at 57.15 86.36 0) (fields_autoplaced)
-    (effects (font (size 1.27 1.27)) (justify left bottom))
-  )
-  (label "MDIO" (at 88.9 191.77 90) (fields_autoplaced)
     (effects (font (size 1.27 1.27)) (justify left bottom))
   )
@@
     (effects (font (size 1.27 1.27)) (justify left bottom))
   )
-  (label "MODE0" (at 53.34 191.77 90) (fields_autoplaced)
+  (label "RMII_MDIO" (at 88.9 191.77 90) (fields_autoplaced)
     (effects (font (size 1.27 1.27)) (justify left bottom))
   )
@@
     (effects (font (size 1.27 1.27)) (justify left bottom))
   )
-  (label "MDIO" (at 57.15 88.9 0) (fields_autoplaced)
+  (label "RMII_MDIO" (at 54.61 88.9 0) (fields_autoplaced)
     (effects (font (size 1.27 1.27)) (justify left bottom))
   )

Commit message: Hardware
Parts:
- removed FB201: 742792031, Inductor_SMD:L_0805_2012Metric_Pad1.15x1.40mm_HandSolder, symbol Device:Ferrite_Bead
- added FB301: 600, Inductor_SMD:L_0603_1608Metric_Pad1.05x0.95mm_HandSolder, symbol Device:FerriteBead_Small
- L201: symbol ETH1CSMU2:749010012A -> ETH1CREF1A:749010012A
- U201: symbol ETH1CSMU2:LAN8742 -> ETH1CREF1A:LAN8742
- U202, U203: symbol ETH1CSMU2:LC03-3.3 -> ETH1CREF1A:LC03-3.3
Connections:
- net +3.3V: now also FB301.1
- net VCCQ: now also FB301.2
