File: HARDWARE/ETH1CREF1A/Trigger.kicad_sch (KiCad schematic)
At the start: 22 parts, among them U701 TXB0104PW, U702 ADuM5402, U703 74AC125

Commit message: Hardware
Parts:
- L701: footprint ETH1CSMU2:CW252016 -> ETH1CREF1A:CW252016
Changed lines of the file:
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@@
       (effects (font (size 1.27 1.27)))
     )
-    (property "Footprint" "ETH1CSMU2:CW252016" (at 219.71 137.16 0)
+    (property "Footprint" "ETH1CREF1A:CW252016" (at 219.71 137.16 0)
       (effects (font (size 1.27 1.27)) hide)
     )

Commit message: Hardware
Parts:
- U703: symbol ETH1CSMU2:74AC125 -> ETH1CREF1A:74AC125
