File: HARDWARE/ETH1CREF1A/Current_Source.kicad_sch (KiCad schematic)
At the start: 25 parts, among them Q1102 BCP55, Q1103 BCP52, U1101 AD620, U1102 AD620

Commit message: Hardware
Parts:
- removed C904 (x2), C906 (x2): 100n, symbol Device:C
- removed C905 (x2), C907 (x2): 10u/35V, symbol Device:C
- removed D1101, D1102: 1N4148, Diode_THT:D_DO-35_SOD27_P7.62mm_Horizontal, symbol Diode:1N4148
- removed FB902 (x2), FB903 (x2): 600, symbol Device:FerriteBead_Small
- removed Q1102: BCP55, Package_TO_SOT_SMD:SOT-223-3_TabPin2, symbol Transistor_BJT:BCP56
- removed Q1103: BCP52, Package_TO_SOT_SMD:SOT-223-3_TabPin2, symbol Transistor_BJT:BCP51
- removed R1101, R1102: 5k, symbol Device:R
- removed R1103: 100, symbol Device:R
- removed R902 (x2), R903 (x2): 10, symbol Device:R
- removed U1101, U1102: AD620, symbol Amplifier_Instrumentation:AD620
- added C1001: 200p, symbol Device:C
- added R1001: 2k, symbol Device:R
- added R1002: 1Meg, symbol Device:R
- added R1003: 100k, symbol Device:R
- added R1004: 10k, symbol Device:R
- added R1005: 1k, symbol Device:R
- added R1006: TNPU1206100RAZEN00, symbol Device:R
- added R1007: Y000710R0000A9L, symbol Device:R
- added R? (x6): 680, symbol Device:R
- added U1002: ~, symbol ETH1CREF1A:LT5400-3
- added U1003: ADA4898-2, Package_SO:SOIC-8-1EP_3.9x4.9mm_P1.27mm_EP2.41x3.81mm, symbol Amplifier_Operational:ADA4898-2
- added U1004: AD811, symbol ETH1CREF1A:AD811
- added U1005, U1006, U1007, U1008, U1009, U1010: AQY211G2SX, symbol ETH1CREF1A:AQY212GS
- added U601 (x2): DG419DY, Package_SO:SOIC-8_3.9x4.9mm_P1.27mm, symbol Analog_Switch:DG419xY
Connections:
- net +15VF: now also U1003.8 (V+), U1004.7 (V+)
- net -15VF: now also U1003.4 (V-), U1003.9 (EP), U1004.4 (V-)
- net AGNDF: now also U1002.8, U1002.9, U601.2
- new net: R?.2, U1008.1
- new net: R1006.1, U1008.3
- new net: R1001.2, U1002.7, U1004.6, U1005.4, U1006.4, U1007.4, U1008.4, U1009.4, U1010.4
- new net: U1002.5, U601.1
- new net: R1007.1, U1010.3
- new net: R1001.1, U1004.2 (-)
- new net: C1001.2, U1003.1, U1004.3 (+)
- new net: U1002.6, U1003.6 (-), U1003.7
- new net: C1001.1, U1002.1, U1002.2, U1003.2 (-)
- new net: U1002.3, U1002.4, U1003.3 (+)
- new net: R?.2, U1010.1
- new net: R?.2, U1009.1
- new net: R1005.1, U1009.3
- new net: R?.2, U1007.1
- new net: R1002.1, U1005.3
- new net: R1003.1, U1006.3
- new net: R?.2, U1005.1
- new net: R1004.1, U1007.3
- new net: R?.2, U1006.1
- new net +5V: R?.1, R?.1, R?.1, R?.1, R?.1, R?.1
- new net AOUT: R1002.2, R1003.2, R1004.2, R1005.2, R1006.2, R1007.2, U1003.5 (+)
- new net CS_SEL_R10: U1010.2
- new net CS_SEL_R100: U1008.2
- new net CS_SEL_R100k: U1006.2
- new net CS_SEL_R10k: U1007.2
- new net CS_SEL_R1Meg: U1005.2
- new net CS_SEL_R1k: U1009.2
- new net CS_SEL_VSOUR: U601.6
- new net VOUT: U601.8
- no-connect marks 4 -> 0

Commit message: Hardware
Parts:
- added C1002, C1003, C1006, C1007: 100n, symbol Device:C
- added C1004, C1005, C1008, C1009: 1u, symbol Device:C
- C1001: footprint (none) -> Capacitor_SMD:C_0603_1608Metric_Pad1.08x0.95mm_HandSolder
- R1001, R? (x6): footprint (none) -> Resistor_SMD:R_0603_1608Metric_Pad0.98x0.95mm_HandSolder
- U1002: value ~ -> LT5400-3; footprint (none) -> Package_SO:MSOP-8-1EP_3x3mm_P0.65mm_EP1.73x1.85mm_ThermalVias
- U1004: value AD811 -> AD811JRZ; footprint (none) -> Package_SO:SOIC-8_3.9x4.9mm_P1.27mm
- U1005, U1006, U1007, U1008, U1009, U1010: footprint (none) -> ETH1CREF1A:AQY212GS
- renumbered R1002 to R1008, R1003 to R1009, R1004 to R1010, R1005 to R1011, R1006 to R1012, R1007 to R1013
Connections:
- net +15VF: now also C1006.1, C1007.1, C1008.1, C1009.1
- net -15VF: now also C1002.1, C1003.1, C1004.1, C1005.1
- net AGNDF: now also C1002.2, C1003.2, C1004.2, C1005.2, C1006.2, C1007.2, C1008.2, C1009.2

Commit message: Hardware and software
Parts:
- C1002, C1003, C1004, C1005, C1006, C1007, C1008, C1009: footprint (none) -> Capacitor_SMD:C_0603_1608Metric_Pad1.08x0.95mm_HandSolder
- R1008: value 1Meg -> TNPV12061M00BYEN; footprint (none) -> Resistor_SMD:R_1206_3216Metric_Pad1.30x1.75mm_HandSolder
- R1009: value 100k -> TNPU1206100KBZEN00; footprint (none) -> Resistor_SMD:R_1206_3216Metric_Pad1.30x1.75mm_HandSolder
- R1010: value 10k -> TNPU120610K0AWEN00; footprint (none) -> Resistor_SMD:R_1206_3216Metric_Pad1.30x1.75mm_HandSolder
- R1011: value 1k -> TNPU12061K00AWEN00; footprint (none) -> Resistor_SMD:R_1206_3216Metric_Pad1.30x1.75mm_HandSolder
- R1012: footprint (none) -> Resistor_SMD:R_1206_3216Metric_Pad1.30x1.75mm_HandSolder
- R1013: value Y000710R0000A9L -> RNCF1206AKT10R0; footprint (none) -> Resistor_SMD:R_1206_3216Metric_Pad1.30x1.75mm_HandSolder
Other:
- moved on the sheet: R1008, R1009, R1010, R1011, R?, U1005, U1006, U1007, U1009

Commit message: Hardware
Parts:
- removed R? (x6): 680, Resistor_SMD:R_0603_1608Metric_Pad0.98x0.95mm_HandSolder, symbol Device:R
- removed U1005, U1006, U1007, U1008, U1009, U1010: AQY211G2SX, ETH1CREF1A:AQY212GS, symbol ETH1CREF1A:AQY212GS
- added D916 (x6): 1N4148W, Diode_SMD:D_SOD-123, symbol Diode:1N4148W
- added K1001, K1002, K1003, K1004, K1005, K1006: 9012, ETH1CREF1A:9012, symbol ETH1CREF1A:9012
- renumbered C1002 to C1001, C1003 to C1002, C1004 to C1003, C1005 to C1004, C1006 to C1005, C1007 to C1006, C1008 to C1007, C1009 to C1008, C1001 to C1009, R1008 to R1002, R1009 to R1003, R1010 to R1004, R1011 to R1005, R1012 to R1006, R1013 to R1007
Connections:
- net +5V: now also D916.1 (K), D916.1 (K), D916.1 (K), D916.1 (K), D916.1 (K), D916.1 (K), K1001.2, K1002.2, K1003.2, K1004.2, K1005.2, K1006.2
- net CS_SEL_R10: now also D916.2 (A), K1006.3
- net CS_SEL_R100: now also D916.2 (A), K1005.3
- net CS_SEL_R100k: now also D916.2 (A), K1002.3
- net CS_SEL_R10k: now also D916.2 (A), K1003.3
- net CS_SEL_R1Meg: now also D916.2 (A), K1001.3
- net CS_SEL_R1k: now also D916.2 (A), K1004.3
- net at R1006.1: now also K1005.4
- net at R1001.2, U1002.7, U1004.6: now also K1001.1, K1002.1, K1003.1, K1004.1, K1005.1, K1006.1
- net at R1007.1: now also K1006.4
- net at R1005.1: now also K1004.4
- net at R1002.1: now also K1001.4
- net at R1003.1: now also K1002.4
- net at R1004.1: now also K1003.4
Other:
- moved on the sheet: C1001, C1002, C1003, C1004, C1005, C1006, C1007, C1008, C1009, R1001, R1002, R1003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

Commit message: Hardware
Parts:
- added C1001, C1007: 100n, Capacitor_SMD:C_0603_1608Metric_Pad1.08x0.95mm_HandSolder, symbol Device:C
- added C1004, C1010: 1u, Capacitor_SMD:C_0603_1608Metric_Pad1.08x0.95mm_HandSolder, symbol Device:C
- renumbered C1001 to C1002, C1002 to C1003, C1003 to C1005, C1004 to C1006, C1005 to C1008, C1006 to C1009, C1007 to C1011, C1008 to C1012, C1009 to C1013
Connections:
- net +15VF: now also C1007.1, C1010.1
- net -15VF: now also C1001.1, C1004.1
- net AGNDF: now also C1001.2, C1004.2, C1007.2, C1010.2
