File: HARDWARE/ETH1CREF1A/DAC.kicad_sch (KiCad schematic)
At the start: 34 parts, among them U901 AD5791, U902 AD8676, U903 AD8675

Commit message: Hardware
Parts:
- C905, C907, C910, C911, C914, C916: value 22u/35V -> 10u/35V
Changed lines of the file:
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@@
   (symbol (lib_id "Device:C") (at 161.925 155.575 0) (unit 1)
     (in_bom yes) (on_board yes) (dnp no) (fields_autoplaced)
-    (property "Reference" "C911" (at 165.735 154.305 0)
-      (effects (font (size 1.27 1.27)) (justify left))
-    )
-    (property "Value" "22u/35V" (at 165.735 156.845 0)
+    (property "Reference" "C911" (at 165.1 154.305 0)
+      (effects (font (size 1.27 1.27)) (justify left))
+    )
+    (property "Value" "10u/35V" (at 165.1 156.845 0)
       (effects (font (size 1.27 1.27)) (justify left))
     )
@@
       (effects (font (size 1.27 1.27)) (justify left))
     )
-    (property "Value" "22u/35V" (at 107.95 157.48 0)
+    (property "Value" "10u/35V" (at 107.95 157.48 0)
       (effects (font (size 1.27 1.27)) (justify left))
     )
@@
       (effects (font (size 1.27 1.27)) (justify left))
     )
-    (property "Value" "22u/35V" (at 165.1 185.42 0)
+    (property "Value" "10u/35V" (at 165.1 185.42 0)
       (effects (font (size 1.27 1.27)) (justify left))
     )
@@
       (effects (font (size 1.27 1.27)) (justify left))
     )
-    (property "Value" "22u/35V" (at 55.88 158.115 0)
+    (property "Value" "10u/35V" (at 55.88 158.115 0)
       (effects (font (size 1.27 1.27)) (justify left))
     )
@@
   (symbol (lib_id "Device:C") (at 104.775 184.785 0) (unit 1)
     (in_bom yes) (on_board yes) (dnp no) (fields_autoplaced)
-    (property "Reference" "C916" (at 108.585 183.515 0)
-      (effects (font (size 1.27 1.27)) (justify left))
-    )
-    (property "Value" "22u/35V" (at 108.585 186.055 0)
+    (property "Reference" "C916" (at 107.95 183.515 0)
+      (effects (font (size 1.27 1.27)) (justify left))
+    )
+    (property "Value" "10u/35V" (at 107.95 186.055 0)
       (effects (font (size 1.27 1.27)) (justify left))
     )
@@
   (symbol (lib_id "Device:C") (at 51.435 185.42 0) (unit 1)
     (in_bom yes) (on_board yes) (dnp no) (fields_autoplaced)
-    (property "Reference" "C905" (at 55.245 184.15 0)
-      (effects (font (size 1.27 1.27)) (justify left))
-    )
-    (property "Value" "22u/35V" (at 55.245 186.69 0)
-      (effects (font (size 1.27 1.27)) (justify left))
-    )
+    (property "Reference" "C905" (at 54.61 184.15 0)
+      (effects (font (size 1.27 1.27)) (justify left))
+    )
+    (property "Value" "10u/35V" (at 54.61 186.69 0)
+      (effects (font (size 1.27 1.27)) (justify left))
+    )

Commit message: Hardware
Parts:
- added C806, C808: 100n, symbol Device:C
- added C812: 10u/15V, symbol Device:C
- added FB804: 600, symbol Device:FerriteBead_Small
- added JP?: Jumper_2_Bridged, symbol Jumper:Jumper_2_Bridged
- added R804: 10, symbol Device:R
- C811: renamed from C903; value 40u/10V -> 10u/15V
- renumbered C904 to C801, C906 to C802, C905 to C803, C907 to C804, C901 to C805, C902 to C807, C913 to C809, C915 to C810, C914 to C813, C916 to C814, C908 to C815, C909 to C816, C910 to C817, C911 to C818, C912 to C819, FB902 to FB801, FB903 to FB802, FB901 to FB803, FB906 to FB805, FB907 to FB806, FB904 to FB807, FB905 to FB808, R902 to R801, R903 to R802, R901 to R803, R907 to R805, R908 to R806, R904 to R807, R905 to R808, R906 to R809, U902 to U801, U901 to U802, U903 to U803
Connections:
- net AGNDF: now also JP?.1 (A)
- net DGNDF: now also C806.2, C808.2, C812.2, JP?.2 (B)
- net at C805.1, C807.1, C811.1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: no longer U802.10 (IOVCC)
- net +5VF renamed +5V
- new net: C806.1, C808.1, C812.1, FB804.2, R804.2, U802.10 (IOVCC)
- new net +3.3V: FB804.1, R804.1
Other:
- moved on the sheet: C805, C807, C811, C819, FB803, R803, R809, U801A, U801B, U802, U803

Commit message: Hardware
Parts:
- removed JP?: Jumper_2_Bridged, symbol Jumper:Jumper_2_Bridged
- C801, C802, C805, C806, C807, C808, C809, C810, C815, C816, C819: footprint (none) -> Capacitor_SMD:C_0603_1608Metric_Pad1.08x0.95mm_HandSolder
- FB801, FB802, FB803, FB804, FB805, FB806, FB807, FB808: footprint (none) -> Inductor_SMD:L_0603_1608Metric_Pad1.05x0.95mm_HandSolder
- R801, R802, R803, R804, R805, R806, R807, R808, R809: footprint (none) -> Resistor_SMD:R_0603_1608Metric_Pad0.98x0.95mm_HandSolder
- U801: value AD8676 -> AD8676BRZ; footprint (none) -> Package_SO:SOIC-8_3.9x4.9mm_P1.27mm
- U802: value AD5791 -> AD5791ARUZ; footprint (none) -> Package_SO:TSSOP-20_4.4x6.5mm_P0.65mm
- U803: value AD8675 -> AD8675ARZ; footprint (none) -> Package_SO:SOIC-8_3.9x4.9mm_P1.27mm
Connections:
- net +3.3V: now also U802.6 (~{RESET}), U802.7 (~{CLR})
- net +5V: no longer U802.6 (~{RESET}), U802.7 (~{CLR})
- net +10V renamed REF_+10V
- net -10V renamed REF_-10V

Commit message: Hardware and software
Parts:
- C803, C804, C811, C812, C813, C814, C817, C818: footprint (none) -> Capacitor_SMD:C_1206_3216Metric_Pad1.33x1.80mm_HandSolder
Changed lines of the file:
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@@
       (effects (font (size 1.27 1.27)) (justify left))
     )
-    (property "Footprint" "" (at 162.8902 159.385 0)
+    (property "Footprint" "Capacitor_SMD:C_1206_3216Metric_Pad1.33x1.80mm_HandSolder" (at 162.8902 159.385 0)
       (effects (font (size 1.27 1.27)) hide)
     )
@@
       (effects (font (size 1.27 1.27)) (justify left))
     )
-    (property "Footprint" "" (at 105.1052 160.02 0)
+    (property "Footprint" "Capacitor_SMD:C_1206_3216Metric_Pad1.33x1.80mm_HandSolder" (at 105.1052 160.02 0)
       (effects (font (size 1.27 1.27)) hide)
     )
@@
       (effects (font (size 1.27 1.27)) (justify left))
     )
-    (property "Footprint" "" (at 162.2552 187.96 0)
+    (property "Footprint" "Capacitor_SMD:C_1206_3216Metric_Pad1.33x1.80mm_HandSolder" (at 162.2552 187.96 0)
       (effects (font (size 1.27 1.27)) hide)
     )
@@
       (effects (font (size 1.27 1.27)) (justify left))
     )
-    (property "Footprint" "" (at 53.0352 160.655 0)
+    (property "Footprint" "Capacitor_SMD:C_1206_3216Metric_Pad1.33x1.80mm_HandSolder" (at 53.0352 160.655 0)
       (effects (font (size 1.27 1.27)) hide)
     )
@@
       (effects (font (size 1.27 1.27)) (justify left))
     )
-    (property "Footprint" "" (at 99.3902 80.01 0)
+    (property "Footprint" "Capacitor_SMD:C_1206_3216Metric_Pad1.33x1.80mm_HandSolder" (at 99.3902 80.01 0)
       (effects (font (size 1.27 1.27)) hide)
     )
@@
       (effects (font (size 1.27 1.27)) (justify left))
     )
-    (property "Footprint" "" (at 99.3902 61.595 0)
+    (property "Footprint" "Capacitor_SMD:C_1206_3216Metric_Pad1.33x1.80mm_HandSolder" (at 99.3902 61.595 0)
       (effects (font (size 1.27 1.27)) hide)
     )
@@
       (effects (font (size 1.27 1.27)) (justify left))
     )
-    (property "Footprint" "" (at 105.7402 188.595 0)
+    (property "Footprint" "Capacitor_SMD:C_1206_3216Metric_Pad1.33x1.80mm_HandSolder" (at 105.7402 188.595 0)
       (effects (font (size 1.27 1.27)) hide)
     )
@@
       (effects (font (size 1.27 1.27)) (justify left))
     )
-    (property "Footprint" "" (at 52.4002 189.23 0)
-      (effects (font (size 1.27 1.27)) hide)
-    )
+    (property "Footprint" "Capacitor_SMD:C_1206_3216Metric_Pad1.33x1.80mm_HandSolder" (at 52.4002 189.23 0)
+      (effects (font (size 1.27 1.27)) hide)
+    )

Commit message: Hardware
Parts:
- removed C803, C804, C813, C814, C817, C818: 10u/35V, Capacitor_SMD:C_1206_3216Metric_Pad1.33x1.80mm_HandSolder, symbol Device:C
- removed C811, C812: 10u/15V, Capacitor_SMD:C_1206_3216Metric_Pad1.33x1.80mm_HandSolder, symbol Device:C
- removed FB803, FB804: 600, Inductor_SMD:L_0603_1608Metric_Pad1.05x0.95mm_HandSolder, symbol Device:FerriteBead_Small
- removed R803, R804: 10, Resistor_SMD:R_0603_1608Metric_Pad0.98x0.95mm_HandSolder, symbol Device:R
- added C619 (x6): 10u/35V, Capacitor_Tantalum_SMD:CP_EIA-6032-28_Kemet-C_Pad2.25x2.35mm_HandSolder, symbol Device:C_Polarized
- added R805: 10k, Resistor_SMD:R_0603_1608Metric_Pad0.98x0.95mm_HandSolder, symbol Device:R
- C807, C808: value 100n -> 1u
- renumbered C815 to C813, C816 to C814, C819 to C817, FB805 to FB803, FB806 to FB804, FB807 to FB805, FB808 to FB806, R805 to R803, R806 to R804, R807 to R806, R808 to R807, R809 to R808
Connections:
- net +3.3V: now also C806.1, C808.1, U802.10 (IOVCC), R805.2
- net +5V: now also C805.1, C807.1, U802.9 (VCC)
- net AGNDF: now also C619.1, C619.2, C619.2, C619.2, C619.2, C619.2
- net DAC_+15V: now also C619.1
- net DAC_-15V: now also C619.2
- net OPAMP_+15V: now also C619.1
- net OPAMP_-15V: now also C619.1
- net ~{SYNC}: now also R805.1
- net at C810.1, FB804.2, R804.2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: now also C619.1
- net at C809.1, FB803.2, R803.2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: now also C619.1
Other:
- moved on the sheet: C805, C806, C807, C808, C817, R808, U801A, U801B, U802, U803
