File: HARDWARE/ETH1CREF1A/Power.kicad_sch (KiCad schematic)
At the start: 16 parts, among them Q1 IRFR5410, U4 NMK2405SAC, U6 MAX5902, U804 NCV1117DT33T5G

Commit message: Hardware
Parts:
- C819: value 1u -> 10u
Connections:
- net +VDC is gone; now on net +24V: D4.1 (K), Q1.3 (S), R24.1, U6.1 (VS)
- net +24V: no longer C19.1, D5.1 (K), L1.1, Q1.2 (D), U6.2 (DRAIN)
- net +5V: no longer names the net of C819.1, C822.1, U4.7 (+VOUT), U804.3 (VI)
- new net VCCQ: C19.1, D5.1 (K), L1.1, Q1.2 (D), U6.2 (DRAIN)
Other:
- moved on the sheet: C19, C819, C822, C823, C824, C825, D4, D5, D6, L1, Q1, R24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

Commit message: Hardware
Parts:
- removed C819, C823: 10u, Capacitor_SMD:C_1206_3216Metric_Pad1.33x1.80mm_HandSolder, symbol Device:C
- removed C822, C824: 1u, Capacitor_SMD:C_1206_3216Metric_Pad1.33x1.80mm_HandSolder, symbol Device:C
- removed C825: 100n, Capacitor_SMD:C_1206_3216Metric_Pad1.33x1.80mm_HandSolder, symbol Device:C
- removed L1: 23100C, LVPREAMP:23100C, symbol pspice:INDUCTOR
- removed U4: NMK2405SAC, LVPREAMP:NMK_SINGLE, symbol LVPREAMP:NMK_SINGLE
- removed U804: NCV1117DT33T5G, Package_TO_SOT_SMD:TO-252-2, symbol Regulator_Linear:LM1117-3.3
- added C303, C304: 330p/2kV, Capacitor_SMD:C_1210_3225Metric_Pad1.42x2.65mm_HandSolder, symbol Device:C
- added C404, C405, C420, C425: 10u/50V, Capacitor_SMD:C_1206_3216Metric_Pad1.42x1.75mm_HandSolder, symbol Device:C
- added C407, C408, C418, C419, C423, C424, C428, C429: 4u7/50V, Capacitor_SMD:C_1206_3216Metric_Pad1.42x1.75mm_HandSolder, symbol Device:C
- added C410, C411: 1u, Capacitor_SMD:C_0603_1608Metric_Pad1.05x0.95mm_HandSolder, symbol Device:C
- added C412, C413: 1u/HC, Capacitor_SMD:C_1206_3216Metric_Pad1.42x1.75mm_HandSolder, symbol Device:C
- added C416, C417: 4p7, Capacitor_SMD:C_0603_1608Metric_Pad1.05x0.95mm_HandSolder, symbol Device:C
- added C432: 10u/16V, Capacitor_SMD:C_1206_3216Metric_Pad1.42x1.75mm_HandSolder, symbol Device:C
- added C437: 47u/16V, Capacitor_SMD:C_1206_3216Metric_Pad1.42x1.75mm_HandSolder, symbol Device:C
- added D401, D402: PMEG6010EP,115, Diode_SMD:D_SOD-128, symbol Device:D_Schottky
- added L301: 7448014501, ETH1CDMM1:7448014501, symbol ETH1CDMM1:7448014501
- added L402, L403: 74489440068, ETH1CDMM1:74489440068, symbol ETH1CDMM1:74489440068
- added L404: TCK-141, ETH1CDMM1:TCK-141, symbol Device:L
- added R304, R305: OPT, Resistor_SMD:R_0603_1608Metric_Pad0.98x0.95mm_HandSolder, symbol Device:R
- added R402, R404, R407, R409: 1M, Resistor_SMD:R_0603_1608Metric_Pad0.98x0.95mm_HandSolder, symbol Device:R
- added R403, R405: 287k, Resistor_SMD:R_0603_1608Metric_Pad0.98x0.95mm_HandSolder, symbol Device:R
- added R408: 97k6, Resistor_SMD:R_0603_1608Metric_Pad0.98x0.95mm_HandSolder, symbol Device:R
- added R410: 46k4, Resistor_SMD:R_0603_1608Metric_Pad0.98x0.95mm_HandSolder, symbol Device:R
- added U302: THL15-2415WI, ETH1CDMM1:THL15, symbol ETH1CDMM1:THL15-2415WI
- added U403, U404: LT8330_S6, Package_TO_SOT_SMD:TSOT-23-6_HandSoldering, symbol ETH1CDMM1:LT8330_S6
- added U406: MC7815BD2TG, Package_TO_SOT_SMD:TO-263-2, symbol Regulator_Linear:L7815
- added U407: MC7915BD2TG, Package_TO_SOT_SMD:TO-263-2, symbol Regulator_Linear:MC79M15_TO252
- added U408: TSR1-2450, ETH1CDMM1:TSR1, symbol ETH1CDMM1:TSR1-2450
- added U409: LM1117DTX-3.3/NOPB, Package_TO_SOT_SMD:TO-252-2, symbol ETH1CDMM1-rescue:LM1117-3.3-Regulator_Linear
Connections:
- net +3.3V: now also C437.1, U409.2 (VO)
- net GNDPWR: now also L301.1
- net VCCQ: now also L301.2
- new net: C416.2, R407.2, R408.1, U403.3 (FBX)
- new net: C413.2, L403.4, U404.1 (SW)
- new net: C410.1, U403.5 (INTVCC)
- new net: C412.1, D402.2 (A), L402.2
- new net: C412.2, L402.4, U403.1 (SW)
- new net: R404.2, R405.1, U404.4 (EN/UVLO)
- new net: C417.1, C419.1, C424.1, L403.3, R409.1, U407.2 (VI)
- new net: C303.2, L301.3, U302.1 (+VIN)
- new net: C416.1, C418.1, C423.1, D402.1 (K), R407.1, U406.1 (IN)
- new net: C425.1, L404.2, U408.1 (VI)
- new net: C413.1, D401.2 (A), L403.2
- new net: R402.2, R403.1, U403.4 (EN/UVLO)
- new net: C304.2, L301.4, U302.2 (-VIN)
- new net: R304.2, R305.1, U302.4 (TRIM)
- new net: C417.2, R409.2, R410.1, U404.3 (FBX)
- new net: C411.1, U404.5 (INTVCC)
- new net +15VF: C428.1, U406.3 (OUT)
- new net +24VF: C303.1, C404.1, C405.1, C407.1, C408.1, C420.1, L402.1, L403.1, L404.1, R304.1, R402.1, R404.1, U302.3 (+VOUT), U403.6 (VIN), U404.6 (VIN)
- new net +5V: C432.1, U408.3 (VO), U409.3 (VI)
- new net -15VF: C429.1, U407.3 (VO)
- new net AGNDF: C304.1, C404.2, C405.2, C407.2, C408.2, C410.2, C411.2, C418.2, C419.2, C420.2, C423.2, C424.2, C425.2, C428.2, C429.2, C432.2, C437.2, R305.2, R403.2, R405.2, R408.2, R410.2, U302.5 (-VOUT), U403.2 (GND), U404.2 (GND), U406.2 (GND), U407.1 (GND), U408.2 (GND), U409.1 (GND)
- new net DGNDF: D401.1 (K), L402.3
- no-connect marks 1 -> 2
Other:
- moved on the sheet: C19, D4, D5, D6, Q1, R24, R25, U6

Commit message: Hardware
Parts:
- C303, C304: footprint Capacitor_SMD:C_1210_3225Metric_Pad1.42x2.65mm_HandSolder -> Capacitor_SMD:C_1210_3225Metric_Pad1.33x2.70mm_HandSolder
- C404, C405, C407, C408, C412, C413, C418, C419, C420, C423, C424, C425, C428, C429, C432, C437: footprint Capacitor_SMD:C_1206_3216Metric_Pad1.42x1.75mm_HandSolder -> Capacitor_SMD:C_1206_3216Metric_Pad1.33x1.80mm_HandSolder
- C410, C411, C416, C417: footprint Capacitor_SMD:C_0603_1608Metric_Pad1.05x0.95mm_HandSolder -> Capacitor_SMD:C_0603_1608Metric_Pad1.08x0.95mm_HandSolder
- D4: footprint LVPREAMP:DO_214AA_REV -> ETH1CREF1A:DO_214AA_REV
- L301: footprint ETH1CDMM1:7448014501 -> ETH1CREF1A:7448014501
- L402, L403: footprint ETH1CDMM1:74489440068 -> ETH1CREF1A:74489440068
- L404: footprint ETH1CDMM1:TCK-141 -> ETH1CREF1A:TCK-141
- Q1: footprint LVPREAMP:TO-252-2_Rectifier -> ETH1CREF1A:TO-252-2_Rectifier
- U302: footprint ETH1CDMM1:THL15 -> ETH1CREF1A:THL15
- U408: footprint ETH1CDMM1:TSR1 -> ETH1CREF1A:TSR1
Connections:
- net DGNDF is gone; now on net AGNDF: D401.1 (K), L402.3

Commit message: Hardware and software
Parts:
- added C432: 10u/16V, Capacitor_SMD:C_1206_3216Metric_Pad1.33x1.80mm_HandSolder, symbol Device:C
- added C437: 47u/16V, Capacitor_SMD:C_1206_3216Metric_Pad1.33x1.80mm_HandSolder, symbol Device:C
- added J601: Conn_02x06_Odd_Even, Connector_PinHeader_2.54mm:PinHeader_2x06_P2.54mm_Vertical, symbol Connector_Generic:Conn_02x06_Odd_Even
- added U409: LM1117DTX-3.3/NOPB, Package_TO_SOT_SMD:TO-252-2, symbol ETH1CDMM1-rescue:LM1117-3.3-Regulator_Linear
- U407: footprint Package_TO_SOT_SMD:TO-263-2 -> Package_TO_SOT_SMD:TO-252-2
- U408: value TSR1-2450 -> TSR1-2490
- U409: value LM1117DTX-3.3/NOPB -> LM1117DTX-5/NOPB
Connections:
- net +15VF: now also J601.1 (Pin_1), J601.2 (Pin_2)
- net +3.3V: now also C437.1, J601.10 (Pin_10), J601.9 (Pin_9), U409.2 (VO); no longer C437.1, U409.2 (VO)
- net +5V: now also C437.1, U409.2 (VO), C432.1, J601.7 (Pin_7), J601.8 (Pin_8), U409.3 (VI); no longer C432.1, U408.3 (VO), U409.3 (VI)
- net -15VF: now also J601.3 (Pin_3), J601.4 (Pin_4)
- net AGNDF: now also C432.2, C437.2, J601.11 (Pin_11), J601.12 (Pin_12), J601.5 (Pin_5), J601.6 (Pin_6), U409.1 (GND)
- new net: C432.1, U408.3 (VO), U409.3 (VI)
Other:
- moved on the sheet: C420, C425, C432, C437, L404, U408, U409

Commit message: Hardware
Parts:
- removed U6: MAX5902, Package_TO_SOT_SMD:SOT-23-6_Handsoldering, symbol LVPREAMP:MAX5902
- added F601: MF-LSMF185/33X, ETH1CREF1A:Fuse_SMD2920, symbol Device:Fuse
- added U601: MAX5902, Package_TO_SOT_SMD:SOT-23-6_Handsoldering, symbol ETH1CREF1A:MAX5902
- L301: symbol ETH1CDMM1:7448014501 -> ETH1CREF1A:7448014501
- L402, L403: symbol ETH1CDMM1:74489440068 -> ETH1CREF1A:74489440068
- U302: symbol ETH1CDMM1:THL15-2415WI -> ETH1CREF1A:THL15-2415WI
- U403, U404: symbol ETH1CDMM1:LT8330_S6 -> ETH1CREF1A:LT8330_S6
- U406: value MC7815BD2TG -> MC7815CD2TG
- U407: value MC7915BD2TG -> MC7915CD2TR4G; footprint Package_TO_SOT_SMD:TO-252-2 -> Package_TO_SOT_SMD:TO-263-2
- U408: symbol ETH1CDMM1:TSR1-2450 -> ETH1CREF1A:TSR1-2450
- U409: symbol ETH1CDMM1-rescue:LM1117-3.3-Regulator_Linear -> ETH1CREF1A-rescue:LM1117-3.3-Regulator_Linear
Connections:
- net +24V: now also F601.1; no longer D4.1 (K), Q1.3 (S), R24.1
- net GNDPWR: now also U601.4 (GND)
- net VCCQ: now also U601.2 (DRAIN)
- net at Q1.1 (G): now also U601.3 (GATE)
- net at R24.2: now also U601.6 (ON/~{OFF})
- new net: D4.1 (K), F601.2, Q1.3 (S), R24.1, U601.1 (VS)
Other:
- moved on the sheet: C432, C437, D4, U409

Commit message: Hardware
Parts:
- added C19: 2u2/50V, Capacitor_SMD:C_1206_3216Metric_Pad1.33x1.80mm_HandSolder, symbol Device:C
- added C420, C425: 10u/50V, Capacitor_SMD:C_1206_3216Metric_Pad1.33x1.80mm_HandSolder, symbol Device:C
- added L404: TCK-141, ETH1CREF1A:TCK-141, symbol Device:L
- added U408: TSR1-2450, ETH1CREF1A:TSR1, symbol ETH1CREF1A:TSR1-2450
Connections:
- net +24VF: now also C420.1, L404.1
- net +5V: no longer C432.1, U409.3 (VI)
- net AGNDF: now also C420.2, C425.2, U408.2 (GND)
- net GNDPWR: now also C19.2
- net VCCQ: no longer names the net of C19.1, D5.1 (K), L301.2, Q1.2 (D), U601.2 (DRAIN)
- net VCCQ: now also C19.1
- new net: C432.1, U408.3 (VO), U409.3 (VI)
- new net: C425.1, L404.2, U408.1 (VI)
Other:
- moved on the sheet: C19, D5, D6, Q1, R25, U601

Commit message: Hardware
Parts:
- removed J601: Conn_02x06_Odd_Even, Connector_PinHeader_2.54mm:PinHeader_2x06_P2.54mm_Vertical, symbol Connector_Generic:Conn_02x06_Odd_Even
- added J1101: Conn_02x04_Odd_Even, Connector_PinHeader_2.54mm:PinHeader_2x04_P2.54mm_Vertical, symbol Connector_Generic:Conn_02x04_Odd_Even
Connections:
- net +15VF: now also J1101.1 (Pin_1)
- net +3.3V: now also J1101.4 (Pin_4)
- net +5V: now also J1101.2 (Pin_2)
- net -15VF: now also J1101.3 (Pin_3)
- net AGNDF: now also J1101.5 (Pin_5), J1101.6 (Pin_6), J1101.7 (Pin_7), J1101.8 (Pin_8)

Commit message: Hardware
Parts:
- removed C428, C429: 4u7/50V, Capacitor_SMD:C_1206_3216Metric_Pad1.33x1.80mm_HandSolder, symbol Device:C
- removed C437 (x2): 47u/16V, Capacitor_SMD:C_1206_3216Metric_Pad1.33x1.80mm_HandSolder, symbol Device:C
- added C619, C620, C627, C628: 10u/35V, Capacitor_Tantalum_SMD:CP_EIA-6032-28_Kemet-C_Pad2.25x2.35mm_HandSolder, symbol Device:C_Polarized
Connections:
- net +15VF: now also C619.1
- net +3.3V: now also C628.1
- net +5V: now also C627.1
- net -15VF: now also C620.2
- net AGNDF: now also C619.2, C620.1, C627.2, C628.2
