File: HARDWARE/ETH1CREF1A/Reference_Voltage.kicad_sch (KiCad schematic)
At the start: 14 parts, among them U504 LT1021-7, U506 LM399H, U803 AD8676

Commit message: Hardware
Parts:
- added C904 (x2), C906 (x3): 100n, symbol Device:C
- added C905 (x2), C907 (x3): 22u/35V, symbol Device:C
- added FB902 (x2), FB903 (x2): 600, symbol Device:FerriteBead_Small
- added R813, R815: 10k/.1%, symbol Device:R
- added R902 (x2), R903 (x2): 10, symbol Device:R
- added U804: AD8676, symbol ETH1CREF1A:AD8676
- C802: value C -> 10p
- R810, R811: value 3k11 -> 3k11/.1%
- R812: value 32k -> 32k/.1%
- R814: value 75k -> 75k/.1%
Connections:
- net +15VF: now also FB903.1, FB903.1, R903.1, R903.1; no longer U803.8 (V+)
- net -15VF: now also FB902.1, FB902.1, R902.1, R902.1; no longer U803.4 (V-)
- net AGNDF: now also C904.2, C904.2, C905.2, C905.2, C906.2, C906.2, C906.2, C907.2, C907.2, C907.2, U804.3 (+), U804.5 (+)
- net at C511.1, R508.1, R801.2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: now also R813.1
- net at R504.2, U504.2 (Vin): now also C906.1, C907.1
- new net: C904.1, C905.1, FB902.2, R902.2, U804.4 (V-)
- new net: R815.2, U804.1
- new net: R813.2, R815.1, U804.2 (-)
- new net: C906.1, C907.1, FB903.2, R903.2, U803.8 (V+)
- new net: C904.1, C905.1, FB902.2, R902.2, U803.4 (V-)
- new net: C906.1, C907.1, FB903.2, R903.2, U804.8 (V+)
- new net: U804.6 (-), U804.7
Other:
- moved on the sheet: C511, C802, R504, R508, R801, R802, R804, R810, R811, R812, R814, U504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

Commit message: Hardware
Parts:
- removed R504: 4k7/.1%, Resistor_SMD:R_0603_1608Metric_Pad1.05x0.95mm_HandSolder, symbol Device:R
- removed R813, R815: 10k/.1%, symbol Device:R
- removed unit 1 of U804
- added C703, C707, C709: 2u2, symbol Device:C
- added R508: 0, Resistor_SMD:R_0603_1608Metric_Pad1.05x0.95mm_HandSolder, symbol Device:R
- added RN701: MPM2002AT5, symbol Device:VoltageDivider_CenterPin3
- added U702: MAX6350, symbol Reference_Voltage:MAX6350
- added unit 1 of U703
- renumbered C802 to C715, R801 to R706, R814 to R708, R802 to R709, R811 to R710, R810 to R711, R804 to R712, R812 to R713, U803 to U701, U804 to U703
Connections:
- net +15VF: now also C906.1, C907.1, U504.2 (Vin), C703.1, U702.2 (IN)
- net AGNDF: now also C703.2, C707.2, C709.2, RN701.1, U702.4 (GND)
- net at C511.1, R508.1, R706.2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: now also R508.1
- new net: C707.1, U702.3 (NR)
- new net: R508.2, RN701.2, U703.1
- new net: RN701.3, U703.2 (-)
- new net: C709.1, U702.6 (OUT), U703.3 (+)
- no-connect marks 0 -> 1
Other:
- note added: "10k/10k"
- note added: "MAIN OPTION"
- note added: "OPTION 1"
- note added: "OPTION 2"
- moved on the sheet: C511, C715, C906, C907, FB903, R508, R706, R708, R709, R710, R711, R712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

Commit message: Hardware
Parts:
- removed RN701: MPM2002AT5, symbol Device:VoltageDivider_CenterPin3
- added R706: 5k/.1%, symbol Device:R
- added R707: 2k/.1%, symbol Device:R
- C511: footprint Capacitor_SMD:C_0603_1608Metric_Pad1.05x0.95mm_HandSolder -> Capacitor_SMD:C_0603_1608Metric_Pad1.08x0.95mm_HandSolder
- C703: footprint (none) -> Capacitor_SMD:C_1210_3225Metric_Pad1.33x2.70mm_HandSolder
- C715, C904, C906: footprint (none) -> Capacitor_SMD:C_0603_1608Metric_Pad1.08x0.95mm_HandSolder
- C905, C907: value 22u/35V -> 10u/35V
- C905: value 22u/35V -> 10u/35V; footprint (none) -> Capacitor_SMD:C_0603_1608Metric_Pad1.08x0.95mm_HandSolder
- C907: value 22u/35V -> 10u/35V; footprint (none) -> Capacitor_SMD:C_1210_3225Metric_Pad1.33x2.70mm_HandSolder
- FB902, FB903: footprint (none) -> Inductor_SMD:L_0603_1608Metric_Pad1.05x0.95mm_HandSolder
- R508: footprint Resistor_SMD:R_0603_1608Metric_Pad1.05x0.95mm_HandSolder -> Resistor_SMD:R_0603_1608Metric_Pad0.98x0.95mm_HandSolder
- R708: renamed from R706; value 62 -> 7k5; footprint (none) -> Resistor_SMD:R_0603_1608Metric_Pad0.98x0.95mm_HandSolder
- R902, R903: footprint (none) -> Resistor_SMD:R_0603_1608Metric_Pad0.98x0.95mm_HandSolder
- U504: value LT1021-7 -> LT1021DCS8-7#PBF
- U506: footprint ADC_TEST:LMx99 -> ETH1CREF1A:LMx99
- U701, U703: value AD8676 -> AD8676BRZ; footprint (none) -> Package_SO:SOIC-8_3.9x4.9mm_P1.27mm
- U702: value MAX6350 -> MAX6350ESA+; footprint (none) -> Package_SO:SOIC-8_3.9x4.9mm_P1.27mm
- renumbered R708 to R710, R709 to R711, R710 to R712, R711 to R713, R712 to R714, R713 to R715
Connections:
- net AGNDF: now also R706.1
- net at R508.2, U703.1: now also R707.2
- net at U703.2 (-): now also R706.2, R707.1
- net +10V renamed REF_+10V
- net -10V renamed REF_-10V
Other:
- note removed: "10k/10k"

Commit message: Hardware and software
Parts:
- removed R712: 3k11/.1%, symbol Device:R
- C707, C709: footprint (none) -> Capacitor_SMD:C_0603_1608Metric_Pad1.08x0.95mm_HandSolder
- C905, C907: footprint (none) -> Capacitor_SMD:C_1206_3216Metric_Pad1.33x1.80mm_HandSolder
- C907: value 22u/35V -> 10u/35V; footprint (none) -> Capacitor_SMD:C_1206_3216Metric_Pad1.33x1.80mm_HandSolder
- R706, R707, R711, R714: footprint (none) -> Resistor_SMD:R_0603_1608Metric_Pad0.98x0.95mm_HandSolder
- R710: value 75k/.1% -> 6k98/.1%; footprint (none) -> Resistor_SMD:R_0603_1608Metric_Pad0.98x0.95mm_HandSolder
- R712: renamed from R713; value 3k11/.1% -> 1k96/.1%; footprint (none) -> Resistor_SMD:R_0603_1608Metric_Pad0.98x0.95mm_HandSolder
- R713: renamed from R715; value 32k/.1% -> 3k01/.1%; footprint (none) -> Resistor_SMD:R_0603_1608Metric_Pad0.98x0.95mm_HandSolder
Connections:
- net at C715.1, R710.2, U701.2 (-): now also R713.1
Other:
- moved on the sheet: R713
Changed lines of the file:
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@@
     (stroke (width 0) (type default))
   )
-  (wire (pts (xy 213.36 63.5) (xy 215.265 63.5))
+  (wire (pts (xy 208.28 63.5) (xy 215.265 63.5))
     (stroke (width 0) (type default))
   )
@@
     (stroke (width 0) (type default))
   )
-  (wire (pts (xy 193.675 63.5) (xy 195.58 63.5))
+  (wire (pts (xy 193.675 63.5) (xy 200.66 63.5))
     (stroke (width 0) (type default))
   )
@@
   )
   (wire (pts (xy 113.03 159.385) (xy 113.03 155.575))
-    (stroke (width 0) (type default))
-  )
-  (wire (pts (xy 203.2 63.5) (xy 205.74 63.5))
     (stroke (width 0) (type default))
   )
@@
       (effects (font (size 1.27 1.27)) (justify left))
     )
-    (property "Footprint" "" (at 60.0202 54.61 0)
+    (property "Footprint" "Capacitor_SMD:C_0603_1608Metric_Pad1.08x0.95mm_HandSolder" (at 60.0202 54.61 0)
       (effects (font (size 1.27 1.27)) hide)
     )
@@
   (symbol (lib_id "Device:R") (at 203.2 88.9 90) (unit 1)
     (in_bom yes) (on_board yes) (dnp no)
-    (property "Reference" "R713" (at 203.2 83.82 90)
-      (effects (font (size 1.27 1.27)))
-    )
-    (property "Value" "3k11/.1%" (at 203.2 86.36 90)
-      (effects (font (size 1.27 1.27)))
-    )
-    (property "Footprint" "" (at 203.2 90.678 90)
+    (property "Reference" "R712" (at 203.2 83.82 90)
+      (effects (font (size 1.27 1.27)))
+    )
+    (property "Value" "1k96/.1%" (at 203.2 86.36 90)
+      (effects (font (size 1.27 1.27)))
+    )
+    (property "Footprint" "Resistor_SMD:R_0603_1608Metric_Pad0.98x0.95mm_HandSolder" (at 203.2 90.678 90)
       (effects (font (size 1.27 1.27)) hide)
     )
@@
       (project "ETH1CREF1A"
         (path "/f534bde3-7724-4aa2-8c73-8f0531e01e95/846bb202-5e4e-44fb-9116-3eb04dadebb8"
-          (reference "R713") (unit 1)
+          (reference "R712") (unit 1)
         )
       )
@@
   (symbol (lib_id "ETH1CREF1A:AD8676") (at 203.835 109.855 0) (mirror x) (unit 2)
     (in_bom yes) (on_board yes) (dnp no)
-    (property "Reference" "U701" (at 205.105 120.015 0)
-      (effects (font (size 1.27 1.27)))
-    )
-    (property "Value" "AD8676BRZ" (at 205.105 117.475 0)
+    (property "Reference" "U701" (at 208.28 102.235 0)
+      (effects (font (size 1.27 1.27)))
+    )
+    (property "Value" "AD8676BRZ" (at 208.28 104.775 0)
       (effects (font (size 1.27 1.27)))
     )
@@
   (symbol (lib_id "Device:C") (at 66.675 83.82 0) (unit 1)
     (in_bom yes) (on_board yes) (dnp no) (fields_autoplaced)
-    (property "Reference" "C907" (at 70.485 82.55 0)
-      (effects (font (size 1.27 1.27)) (justify left))
-    )
-    (property "Value" "22u/35V" (at 70.485 85.09 0)
-      (effects (font (size 1.27 1.27)) (justify left))
-    )
-    (property "Footprint" "" (at 67.6402 87.63 0)
+    (property "Reference" "C907" (at 69.85 82.55 0)
+      (effects (font (size 1.27 1.27)) (justify left))
+    )
+    (property "Value" "10u/35V" (at 69.85 85.09 0)
+      (effects (font (size 1.27 1.27)) (justify left))
+    )
+    (property "Footprint" "Capacitor_SMD:C_1206_3216Metric_Pad1.33x1.80mm_HandSolder" (at 67.6402 87.63 0)
       (effects (font (size 1.27 1.27)) hide)
     )
@@
   (symbol (lib_id "ETH1CREF1A:AD8676") (at 202.565 76.2 0) (mirror x) (unit 1)
     (in_bom yes) (on_board yes) (dnp no)
-    (property "Reference" "U701" (at 207.01 69.85 0)
-      (effects (font (size 1.27 1.27)))
-    )
-    (property "Value" "AD8676BRZ" (at 207.01 71.755 0)
+    (property "Reference" "U701" (at 208.28 69.215 0)
+      (effects (font (size 1.27 1.27)))
+    )
+    (property "Value" "AD8676BRZ" (at 208.28 71.755 0)
       (effects (font (size 1.27 1.27)))
     )
@@
       (effects (font (size 1.27 1.27)) (justify left))
     )
-    (property "Footprint" "" (at 57.4802 189.23 0)
+    (property "Footprint" "Capacitor_SMD:C_1206_3216Metric_Pad1.33x1.80mm_HandSolder" (at 57.4802 189.23 0)
       (effects (font (size 1.27 1.27)) hide)
     )
@@
       (effects (font (size 1.27 1.27)))
     )
-    (property "Footprint" "" (at 109.22 57.023 90)
+    (property "Footprint" "Resistor_SMD:R_0603_1608Metric_Pad0.98x0.95mm_HandSolder" (at 109.22 57.023 90)
       (effects (font (size 1.27 1.27)) hide)
     )
@@
       (effects (font (size 1.27 1.27)))
     )
-    (property "Footprint" "" (at 119.38 57.023 90)
+    (property "Footprint" "Resistor_SMD:R_0603_1608Metric_Pad0.98x0.95mm_HandSolder" (at 119.38 57.023 90)
       (effects (font (size 1.27 1.27)) hide)
     )
@@
     )
   )
-  (symbol (lib_id "Device:R") (at 209.55 63.5 90) (unit 1)
+  (symbol (lib_id "Device:R") (at 204.47 63.5 90) (unit 1)
     (in_bom yes) (on_board yes) (dnp no)
-    (property "Reference" "R715" (at 209.55 58.42 90)
-      (effects (font (size 1.27 1.27)))
-    )
-    (property "Value" "32k/.1%" (at 209.55 60.96 90)
-      (effects (font (size 1.27 1.27)))
-    )
-    (property "Footprint" "" (at 209.55 65.278 90)
-      (effects (font (size 1.27 1.27)) hide)
-    )
-    (property "Datasheet" "~" (at 209.55 63.5 0)
-      (effects (font (size 1.27 1.27)) hide)
-    )
-    (pin "1")
-    (pin "2")
-    (instances
-      (project "ETH1CREF1A"
-        (path "/f534bde3-7724-4aa2-8c73-8f0531e01e95/846bb202-5e4e-44fb-9116-3eb04dadebb8"
-          (reference "R715") (unit 1)
+    (property "Reference" "R713" (at 204.47 58.42 90)
+      (effects (font (size 1.27 1.27)))
+    )
+    (property "Value" "3k01/.1%" (at 204.47 60.96 90)
+      (effects (font (size 1.27 1.27)))
+    )
+    (property "Footprint" "Resistor_SMD:R_0603_1608Metric_Pad0.98x0.95mm_HandSolder" (at 204.47 65.278 90)
+      (effects (font (size 1.27 1.27)) hide)
+    )
+    (property "Datasheet" "~" (at 204.47 63.5 0)
+      (effects (font (size 1.27 1.27)) hide)
+    )
+    (pin "1")
+    (pin "2")
+    (instances
+      (project "ETH1CREF1A"
+        (path "/f534bde3-7724-4aa2-8c73-8f0531e01e95/846bb202-5e4e-44fb-9116-3eb04dadebb8"
+          (reference "R713") (unit 1)
         )
       )
@@
       (effects (font (size 1.27 1.27)) (justify left))
     )
-    (property "Footprint" "" (at 93.6752 48.26 0)
+    (property "Footprint" "Capacitor_SMD:C_0603_1608Metric_Pad1.08x0.95mm_HandSolder" (at 93.6752 48.26 0)
       (effects (font (size 1.27 1.27)) hide)
     )
@@
       (effects (font (size 1.27 1.27)) (justify left))
     )
-    (property "Footprint" "" (at 131.1402 163.83 0)
+    (property "Footprint" "Capacitor_SMD:C_1206_3216Metric_Pad1.33x1.80mm_HandSolder" (at 131.1402 163.83 0)
       (effects (font (size 1.27 1.27)) hide)
     )
@@
       (effects (font (size 1.27 1.27)))
     )
-    (property "Footprint" "" (at 191.135 109.093 90)
+    (property "Footprint" "Resistor_SMD:R_0603_1608Metric_Pad0.98x0.95mm_HandSolder" (at 191.135 109.093 90)
       (effects (font (size 1.27 1.27)) hide)
     )
@@
       (effects (font (size 1.27 1.27)))
     )
-    (property "Value" "75k/.1%" (at 188.595 71.12 90)
-      (effects (font (size 1.27 1.27)))
-    )
-    (property "Footprint" "" (at 188.595 75.438 90)
+    (property "Value" "6k98/.1%" (at 188.595 71.12 90)
+      (effects (font (size 1.27 1.27)))
+    )
+    (property "Footprint" "Resistor_SMD:R_0603_1608Metric_Pad0.98x0.95mm_HandSolder" (at 188.595 75.438 90)
       (effects (font (size 1.27 1.27)) hide)
     )
@@
         (path "/f534bde3-7724-4aa2-8c73-8f0531e01e95/846bb202-5e4e-44fb-9116-3eb04dadebb8"
           (reference "R710") (unit 1)
-        )
-      )
-    )
-  )
-  (symbol (lib_id "Device:R") (at 199.39 63.5 90) (unit 1)
-    (in_bom yes) (on_board yes) (dnp no)
-    (property "Reference" "R712" (at 199.39 58.42 90)
-      (effects (font (size 1.27 1.27)))
-    )
-    (property "Value" "3k11/.1%" (at 199.39 60.96 90)
-      (effects (font (size 1.27 1.27)))
-    )
-    (property "Footprint" "" (at 199.39 65.278 90)
-      (effects (font (size 1.27 1.27)) hide)
-    )
-    (property "Datasheet" "~" (at 199.39 63.5 0)
-      (effects (font (size 1.27 1.27)) hide)
-    )
-    (pin "1")
-    (pin "2")
-    (instances
-      (project "ETH1CREF1A"
-        (path "/f534bde3-7724-4aa2-8c73-8f0531e01e95/846bb202-5e4e-44fb-9116-3eb04dadebb8"
-          (reference "R712") (unit 1)
         )
       )
@@
       (effects (font (size 1.27 1.27)))
     )
-    (property "Footprint" "" (at 205.105 100.838 90)
-      (effects (font (size 1.27 1.27)) hide)
-    )
+    (property "Footprint" "Resistor_SMD:R_0603_1608Metric_Pad0.98x0.95mm_HandSolder" (at 205.105 100.838 90)
+      (effects (font (size 1.27 1.27)) hide)
+    )

Commit message: Hardware
Parts:
- C703: footprint Capacitor_SMD:C_1210_3225Metric_Pad1.33x2.70mm_HandSolder -> Capacitor_SMD:C_0603_1608Metric_Pad1.08x0.95mm_HandSolder
- U504: symbol ADC_TEST:LT1021-7 -> ETH1CREF1A:LT1021-7
- U506: symbol ADC_TEST:LM399H -> ETH1CREF1A:LM399H
- renumbered U703 to U701, U701 to U705, U703 to U705
Changed lines of the file:
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@@
       (effects (font (size 1.27 1.27)) (justify left))
     )
-    (property "Footprint" "Capacitor_SMD:C_1210_3225Metric_Pad1.33x2.70mm_HandSolder" (at 53.6702 44.45 0)
+    (property "Footprint" "Capacitor_SMD:C_0603_1608Metric_Pad1.08x0.95mm_HandSolder" (at 53.6702 44.45 0)
       (effects (font (size 1.27 1.27)) hide)
     )
@@
     (pin "2")
     (instances
-      (project "ADC_Test"
+      (project "ETH1CREF1A"
         (path "/700b7e2e-569c-4a15-81a0-3588750b2d07/00000000-0000-0000-0000-00005fccc067"
           (reference "R508") (unit 1)
@@
     )
   )
-  (symbol (lib_id "ADC_TEST:AGNDF") (at 104.775 55.245 270) (unit 1)
+  (symbol (lib_id "ETH1CREF1A:AGNDF") (at 104.775 55.245 270) (unit 1)
     (in_bom yes) (on_board yes) (dnp no)
     (property "Reference" "#PWR0523" (at 98.425 55.245 0)
@@
     (pin "1")
     (instances
-      (project "ADC_Test"
+      (project "ETH1CREF1A"
         (path "/700b7e2e-569c-4a15-81a0-3588750b2d07/00000000-0000-0000-0000-00005fccc067"
           (reference "#PWR0523") (unit 1)
@@
   (symbol (lib_id "ETH1CREF1A:AD8676") (at 203.835 109.855 0) (mirror x) (unit 2)
     (in_bom yes) (on_board yes) (dnp no)
-    (property "Reference" "U701" (at 208.28 102.235 0)
+    (property "Reference" "U705" (at 208.28 102.235 0)
       (effects (font (size 1.27 1.27)))
     )
@@
       (project "ETH1CREF1A"
         (path "/f534bde3-7724-4aa2-8c73-8f0531e01e95/846bb202-5e4e-44fb-9116-3eb04dadebb8"
-          (reference "U701") (unit 2)
+          (reference "U705") (unit 2)
         )
       )
@@
     )
   )
-  (symbol (lib_id "ADC_TEST:AGNDF") (at 76.2 57.15 0) (unit 1)
+  (symbol (lib_id "ETH1CREF1A:AGNDF") (at 76.2 57.15 0) (unit 1)
     (in_bom yes) (on_board yes) (dnp no)
     (property "Reference" "#PWR0523" (at 76.2 63.5 0)
@@
     (pin "1")
     (instances
-      (project "ADC_Test"
+      (project "ETH1CREF1A"
         (path "/700b7e2e-569c-4a15-81a0-3588750b2d07/00000000-0000-0000-0000-00005fccc067"
           (reference "#PWR0523") (unit 1)
@@
   (symbol (lib_id "ETH1CREF1A:AD8676") (at 121.92 40.64 0) (unit 1)
     (in_bom yes) (on_board yes) (dnp no) (fields_autoplaced)
-    (property "Reference" "U703" (at 123.19 30.48 0)
+    (property "Reference" "U701" (at 123.19 30.48 0)
       (effects (font (size 1.27 1.27)))
     )
@@
       (project "ETH1CREF1A"
         (path "/f534bde3-7724-4aa2-8c73-8f0531e01e95/846bb202-5e4e-44fb-9116-3eb04dadebb8"
-          (reference "U703") (unit 1)
-        )
-      )
-    )
-  )
-  (symbol (lib_id "ADC_TEST:AGNDF") (at 53.975 88.9 0) (unit 1)
+          (reference "U701") (unit 1)
+        )
+      )
+    )
+  )
+  (symbol (lib_id "ETH1CREF1A:AGNDF") (at 53.975 88.9 0) (unit 1)
     (in_bom yes) (on_board yes) (dnp no)
     (property "Reference" "#PWR0523" (at 53.975 95.25 0)
@@
     (pin "1")
     (instances
-      (project "ADC_Test"
+      (project "ETH1CREF1A"
         (path "/700b7e2e-569c-4a15-81a0-3588750b2d07/00000000-0000-0000-0000-00005fccc067"
           (reference "#PWR0523") (unit 1)
@@
   (symbol (lib_id "ETH1CREF1A:AD8676") (at 202.565 76.2 0) (mirror x) (unit 1)
     (in_bom yes) (on_board yes) (dnp no)
-    (property "Reference" "U701" (at 208.28 69.215 0)
+    (property "Reference" "U705" (at 208.28 69.215 0)
       (effects (font (size 1.27 1.27)))
     )
@@
       (project "ETH1CREF1A"
         (path "/f534bde3-7724-4aa2-8c73-8f0531e01e95/846bb202-5e4e-44fb-9116-3eb04dadebb8"
-          (reference "U701") (unit 1)
+          (reference "U705") (unit 1)
         )
       )
@@
     )
   )
-  (symbol (lib_id "ADC_TEST:AGNDF") (at 149.225 121.92 0) (unit 1)
+  (symbol (lib_id "ETH1CREF1A:AGNDF") (at 149.225 121.92 0) (unit 1)
     (in_bom yes) (on_board yes) (dnp no)
     (property "Reference" "#PWR0523" (at 149.225 128.27 0)
@@
     (pin "1")
     (instances
-      (project "ADC_Test"
+      (project "ETH1CREF1A"
         (path "/700b7e2e-569c-4a15-81a0-3588750b2d07/00000000-0000-0000-0000-00005fccc067"
           (reference "#PWR0523") (unit 1)
@@
     )
   )
-  (symbol (lib_id "ADC_TEST:AGNDF") (at 86.36 88.9 0) (unit 1)
+  (symbol (lib_id "ETH1CREF1A:AGNDF") (at 86.36 88.9 0) (unit 1)
     (in_bom yes) (on_board yes) (dnp no)
     (property "Reference" "#PWR0523" (at 86.36 95.25 0)
@@
     (pin "1")
     (instances
-      (project "ADC_Test"
+      (project "ETH1CREF1A"
         (path "/700b7e2e-569c-4a15-81a0-3588750b2d07/00000000-0000-0000-0000-00005fccc067"
           (reference "#PWR0523") (unit 1)
@@
     )
   )
-  (symbol (lib_id "ADC_TEST:AGNDF") (at 196.215 112.395 270) (unit 1)
+  (symbol (lib_id "ETH1CREF1A:AGNDF") (at 196.215 112.395 270) (unit 1)
     (in_bom yes) (on_board yes) (dnp no)
     (property "Reference" "#PWR0519" (at 189.865 112.395 0)
@@
     (pin "1")
     (instances
-      (project "ADC_Test"
+      (project "ETH1CREF1A"
         (path "/700b7e2e-569c-4a15-81a0-3588750b2d07/00000000-0000-0000-0000-00005fccc067"
           (reference "#PWR0519") (unit 1)
@@
     (pin "2")
     (instances
-      (project "ADC_Test"
+      (project "ETH1CREF1A"
         (path "/700b7e2e-569c-4a15-81a0-3588750b2d07/00000000-0000-0000-0000-00005fccc067"
           (reference "C511") (unit 1)
@@
   (symbol (lib_id "ETH1CREF1A:AD8676") (at 76.835 125.73 0) (unit 2)
     (in_bom yes) (on_board yes) (dnp no) (fields_autoplaced)
-    (property "Reference" "U703" (at 78.105 115.57 0)
+    (property "Reference" "U701" (at 78.105 115.57 0)
       (effects (font (size 1.27 1.27)))
     )
@@
       (project "ETH1CREF1A"
         (path "/f534bde3-7724-4aa2-8c73-8f0531e01e95/846bb202-5e4e-44fb-9116-3eb04dadebb8"
-          (reference "U703") (unit 2)
+          (reference "U701") (unit 2)
         )
       )
@@
   (symbol (lib_id "ETH1CREF1A:AD8676") (at 146.05 168.275 0) (unit 3)
     (in_bom yes) (on_board yes) (dnp no) (fields_autoplaced)
-    (property "Reference" "U703" (at 149.225 167.005 0)
+    (property "Reference" "U705" (at 149.225 167.005 0)
       (effects (font (size 1.27 1.27)) (justify left))
     )
@@
       (project "ETH1CREF1A"
         (path "/f534bde3-7724-4aa2-8c73-8f0531e01e95/846bb202-5e4e-44fb-9116-3eb04dadebb8"
-          (reference "U703") (unit 3)
-        )
-      )
-    )
-  )
-  (symbol (lib_id "ADC_TEST:AGNDF") (at 183.515 73.66 270) (unit 1)
+          (reference "U705") (unit 3)
+        )
+      )
+    )
+  )
+  (symbol (lib_id "ETH1CREF1A:AGNDF") (at 183.515 73.66 270) (unit 1)
     (in_bom yes) (on_board yes) (dnp no)
     (property "Reference" "#PWR0519" (at 177.165 73.66 0)
@@
     (pin "1")
     (instances
-      (project "ADC_Test"
+      (project "ETH1CREF1A"
         (path "/700b7e2e-569c-4a15-81a0-3588750b2d07/00000000-0000-0000-0000-00005fccc067"
           (reference "#PWR0519") (unit 1)
@@
     )
   )
-  (symbol (lib_id "ADC_TEST:LM399H") (at 139.065 114.3 0) (unit 1)
+  (symbol (lib_id "ETH1CREF1A:LM399H") (at 139.065 114.3 0) (unit 1)
     (in_bom yes) (on_board yes) (dnp no)
     (property "Reference" "U506" (at 144.8562 113.1316 0)
@@
     (pin "4")
     (instances
-      (project "ADC_Test"
+      (project "ETH1CREF1A"
         (path "/700b7e2e-569c-4a15-81a0-3588750b2d07/00000000-0000-0000-0000-00005fccc067"
           (reference "U506") (unit 1)
@@
       (project "ETH1CREF1A"
         (path "/f534bde3-7724-4aa2-8c73-8f0531e01e95/846bb202-5e4e-44fb-9116-3eb04dadebb8"
-          (reference "U705") (unit 1)
+          (reference "U704") (unit 1)
         )
       )
@@
     )
   )
-  (symbol (lib_id "ADC_TEST:AGNDF") (at 70.485 123.19 270) (unit 1)
+  (symbol (lib_id "ETH1CREF1A:AGNDF") (at 70.485 123.19 270) (unit 1)
     (in_bom yes) (on_board yes) (dnp no)
     (property "Reference" "#PWR0519" (at 64.135 123.19 0)
@@
     (pin "1")
     (instances
-      (project "ADC_Test"
+      (project "ETH1CREF1A"
         (path "/700b7e2e-569c-4a15-81a0-3588750b2d07/00000000-0000-0000-0000-00005fccc067"
           (reference "#PWR0519") (unit 1)
@@
     (pin "2")
     (instances
-      (project "ADC_Test"
+      (project "ETH1CREF1A"
         (path "/700b7e2e-569c-4a15-81a0-3588750b2d07/00000000-0000-0000-0000-00005fccc067"
           (reference "R508") (unit 1)
@@
     )
   )
-  (symbol (lib_id "ADC_TEST:LT1021-7") (at 86.36 81.28 0) (unit 1)
+  (symbol (lib_id "ETH1CREF1A:LT1021-7") (at 86.36 81.28 0) (unit 1)
     (in_bom yes) (on_board yes) (dnp no)
     (property "Reference" "U504" (at 86.36 71.9582 0)
@@
     (pin "8")
     (instances
-      (project "ADC_Test"
+      (project "ETH1CREF1A"
         (path "/700b7e2e-569c-4a15-81a0-3588750b2d07/00000000-0000-0000-0000-00005fccc067"
           (reference "U504") (unit 1)
@@
       (project "ETH1CREF1A"
         (path "/f534bde3-7724-4aa2-8c73-8f0531e01e95/846bb202-5e4e-44fb-9116-3eb04dadebb8"
-          (reference "U704") (unit 1)
-        )
-      )
+          (reference "U703") (unit 1)
+        )
+      )
