File: HARDWARE/ETH1CREF1A/Reference_Voltage.kicad_sch (KiCad schematic)
At the start: 38 parts, among them U504 LT1021DCS8-7#PBF, U506 LM399H, U701 AD8676BRZ, U702 MAX6350ESA+, U705 AD8676BRZ

Commit message: Hardware
Parts:
- removed C905: 10u/35V, Capacitor_SMD:C_0603_1608Metric_Pad1.08x0.95mm_HandSolder, symbol Device:C
- removed C907: 10u/35V, Capacitor_SMD:C_1206_3216Metric_Pad1.33x1.80mm_HandSolder, symbol Device:C
- added C619 (x2): 10u/35V, Capacitor_Tantalum_SMD:CP_EIA-6032-28_Kemet-C_Pad2.25x2.35mm_HandSolder, symbol Device:C_Polarized
- C907: footprint Capacitor_SMD:C_1210_3225Metric_Pad1.33x2.70mm_HandSolder -> Capacitor_SMD:C_1206_3216Metric_Pad1.33x1.80mm_HandSolder
Connections:
- net AGNDF: now also C619.1, C619.2
- net at C904.1, FB902.2, R902.2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: now also C619.2
- net at C906.1, FB903.2, R903.2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: now also C619.1
Changed lines of the file:
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@@
       (effects (font (size 1.27 1.27)) (justify left))
     )
-    (property "Footprint" "Capacitor_SMD:C_1210_3225Metric_Pad1.33x2.70mm_HandSolder" (at 57.4802 164.465 0)
+    (property "Footprint" "Capacitor_SMD:C_1206_3216Metric_Pad1.33x1.80mm_HandSolder" (at 57.4802 164.465 0)
       (effects (font (size 1.27 1.27)) hide)
     )
@@
         (path "/f534bde3-7724-4aa2-8c73-8f0531e01e95/846bb202-5e4e-44fb-9116-3eb04dadebb8"
           (reference "C705") (unit 1)
+        )
+      )
+    )
+  )
+  (symbol (lib_id "Device:C_Polarized") (at 129.54 185.42 180) (unit 1)
+    (in_bom yes) (on_board yes) (dnp no) (fields_autoplaced)
+    (property "Reference" "C619" (at 132.715 185.039 0)
+      (effects (font (size 1.27 1.27)) (justify right))
+    )
+    (property "Value" "10u/35V" (at 132.715 187.579 0)
+      (effects (font (size 1.27 1.27)) (justify right))
+    )
+    (property "Footprint" "Capacitor_Tantalum_SMD:CP_EIA-6032-28_Kemet-C_Pad2.25x2.35mm_HandSolder" (at 128.5748 181.61 0)
+      (effects (font (size 1.27 1.27)) hide)
+    )
+    (property "Datasheet" "~" (at 129.54 185.42 0)
+      (effects (font (size 1.27 1.27)) hide)
+    )
+    (pin "1")
+    (pin "2")
+    (instances
+      (project "ETH1CREF1A"
+        (path "/f534bde3-7724-4aa2-8c73-8f0531e01e95/62654dcd-3414-4e70-b8e6-16734596bf10"
+          (reference "C619") (unit 1)
+        )
+        (path "/f534bde3-7724-4aa2-8c73-8f0531e01e95/ebac98f6-7cea-4b7b-a7eb-72e971f44089"
+          (reference "C804") (unit 1)
+        )
+        (path "/f534bde3-7724-4aa2-8c73-8f0531e01e95/846bb202-5e4e-44fb-9116-3eb04dadebb8"
+          (reference "C712") (unit 1)
         )
       )
@@
     )
   )
-  (symbol (lib_id "Device:C") (at 130.175 160.02 0) (unit 1)
-    (in_bom yes) (on_board yes) (dnp no) (fields_autoplaced)
-    (property "Reference" "C907" (at 133.35 158.75 0)
-      (effects (font (size 1.27 1.27)) (justify left))
-    )
-    (property "Value" "10u/35V" (at 133.35 161.29 0)
-      (effects (font (size 1.27 1.27)) (justify left))
-    )
-    (property "Footprint" "Capacitor_SMD:C_1206_3216Metric_Pad1.33x1.80mm_HandSolder" (at 131.1402 163.83 0)
-      (effects (font (size 1.27 1.27)) hide)
-    )
-    (property "Datasheet" "~" (at 130.175 160.02 0)
-      (effects (font (size 1.27 1.27)) hide)
-    )
-    (pin "1")
-    (pin "2")
-    (instances
-      (project "ETH1CREF1A"
-        (path "/f534bde3-7724-4aa2-8c73-8f0531e01e95/ebac98f6-7cea-4b7b-a7eb-72e971f44089"
-          (reference "C907") (unit 1)
-        )
-        (path "/f534bde3-7724-4aa2-8c73-8f0531e01e95/846bb202-5e4e-44fb-9116-3eb04dadebb8"
-          (reference "C713") (unit 1)
-        )
-      )
-    )
-  )
   (symbol (lib_id "ETH1CREF1A:AD8676") (at 146.05 168.275 0) (unit 3)
     (in_bom yes) (on_board yes) (dnp no) (fields_autoplaced)
@@
     )
   )
-  (symbol (lib_id "Device:C") (at 129.54 185.42 0) (unit 1)
-    (in_bom yes) (on_board yes) (dnp no) (fields_autoplaced)
-    (property "Reference" "C905" (at 133.35 184.15 0)
-      (effects (font (size 1.27 1.27)) (justify left))
-    )
-    (property "Value" "10u/35V" (at 133.35 186.69 0)
-      (effects (font (size 1.27 1.27)) (justify left))
-    )
-    (property "Footprint" "Capacitor_SMD:C_0603_1608Metric_Pad1.08x0.95mm_HandSolder" (at 130.5052 189.23 0)
-      (effects (font (size 1.27 1.27)) hide)
-    )
-    (property "Datasheet" "~" (at 129.54 185.42 0)
-      (effects (font (size 1.27 1.27)) hide)
-    )
-    (pin "1")
-    (pin "2")
-    (instances
-      (project "ETH1CREF1A"
-        (path "/f534bde3-7724-4aa2-8c73-8f0531e01e95/ebac98f6-7cea-4b7b-a7eb-72e971f44089"
-          (reference "C905") (unit 1)
-        )
-        (path "/f534bde3-7724-4aa2-8c73-8f0531e01e95/846bb202-5e4e-44fb-9116-3eb04dadebb8"
-          (reference "C712") (unit 1)
-        )
-      )
-    )
-  )
   (symbol (lib_id "Device:R") (at 102.235 78.74 270) (unit 1)
     (in_bom yes) (on_board yes) (dnp no)
@@
         )
       )
+    )
+  )
+  (symbol (lib_id "Device:C_Polarized") (at 130.175 160.02 0) (unit 1)
+    (in_bom yes) (on_board yes) (dnp no) (fields_autoplaced)
+    (property "Reference" "C619" (at 133.35 157.861 0)
+      (effects (font (size 1.27 1.27)) (justify left))
+    )
+    (property "Value" "10u/35V" (at 133.35 160.401 0)
+      (effects (font (size 1.27 1.27)) (justify left))
+    )
+    (property "Footprint" "Capacitor_Tantalum_SMD:CP_EIA-6032-28_Kemet-C_Pad2.25x2.35mm_HandSolder" (at 131.1402 163.83 0)
+      (effects (font (size 1.27 1.27)) hide)
+    )
+    (property "Datasheet" "~" (at 130.175 160.02 0)
+      (effects (font (size 1.27 1.27)) hide)
+    )
+    (pin "1")
+    (pin "2")
+    (instances
+      (project "ETH1CREF1A"
+        (path "/f534bde3-7724-4aa2-8c73-8f0531e01e95/62654dcd-3414-4e70-b8e6-16734596bf10"
+          (reference "C619") (unit 1)
+        )
+        (path "/f534bde3-7724-4aa2-8c73-8f0531e01e95/ebac98f6-7cea-4b7b-a7eb-72e971f44089"
+          (reference "C804") (unit 1)
+        )
+        (path "/f534bde3-7724-4aa2-8c73-8f0531e01e95/846bb202-5e4e-44fb-9116-3eb04dadebb8"
+          (reference "C713") (unit 1)
+        )
+      )
