File: HARDWARE/ETH1CREF1A/ETH1CREF1A.kicad_pcb (KiCad board)
At the start: 2 copper layers, 288 parts, among them J201 Conn_02x01, J202 20021111-00010T4LF, J501 C64AC, K901 HE3621A0510, K902 HE3621A0510, K903 HE3621A0510, K904 HE3621A0510, K905 HE3621A0510, K906 HE3621A0510, Q601 IRFR5410, U1001 DG419DY, U1002 LT5400-3, U1003 ADA4898-2, U1004 AD811JRZ, U1005 AQY211G2SX, U1006 AQY211G2SX, U1007 AQY211G2SX, U1008 AQY211G2SX, U1009 AQY211G2SX, U1010 AQY211G2SX, U1101 74HCT595PW, U1102 74HCT595PW, U1103 74HCT595PW, U1104 74HCT595PW, U1105 SN74LVC1T45DRLR, U1106 SN74LVC1T45DRLR, U1107 SN74LVC1T45DRLR, U1108 SN74LVC1T45DRLR, U201 HDC1080, U202 STM32F746ZG, U203 24LC08B-E/MS, U301 LAN8742A, U302 LC03-3.3, U303 LC03-3.3, U401 TXB0104PW, U402 ADuM5402, U403 74AC125, U601 MAX5902, U602 LT8330_S6, U603 LT8330_S6, U604 MC7815BD2TG, U605 MC7915BD2TG, U606 THL15-2415WI, U607 TSR1-2450, U608 LM1117DTX-3.3/NOPB, U701 AD8676BRZ, U702 MAX6350ESA+, U703 AD8676BRZ, U704 LT1021DCS8-7#PBF, U705 LM399H, U801 AD8676BRZ, U802 AD5791ARUZ, U803 AD8675ARZ, U901 AQY211G2SX, U902 AQY211G2SX, U903 AQY211G2SX, U904 AQY211G2SX, U905 AQY211G2SX, U906 AQY211G2SX, U907 AQY211G2SX, U908 AQY211G2SX, U909 AQY211G2SX, U910 AQY211G2SX, U911 AQY211G2SX, U912 AQY211G2SX, U913 ULN2003A, U914 AQY211G2SX, U915 AQY211G2SX, U916 AQY211G2SX, U917 AQY211G2SX, U918 AQY211G2SX, U919 AQY211G2SX, Y201 NX5032GA-16.000M, Y301 NX5032GA-25.000000MHZ-LN-CD-1

Commit message: Hardware and software
Parts:
- removed R901, R902, R903, R904, R905, R906, R907, R908, R909, R910, R911, R912, R913, R914, R915, R916, R917, R918: 680, Resistor_SMD:R_0603_1608Metric_Pad0.98x0.95mm_HandSolder
- removed U901, U902, U903, U904, U905, U906, U907, U908, U909, U910, U911, U912, U914, U915, U916, U917, U918, U919: AQY211G2SX, ETH1CREF1A:AQY212GS
- added C1002: 100n, Capacitor_SMD:C_0603_1608Metric_Pad1.08x0.95mm_HandSolder, F.Cu at (-30.0, 175.1)
- added C1003: 100n, Capacitor_SMD:C_0603_1608Metric_Pad1.08x0.95mm_HandSolder, F.Cu at (-30.0, 177.6)
- added C1004: 1u, Capacitor_SMD:C_0603_1608Metric_Pad1.08x0.95mm_HandSolder, F.Cu at (-30.0, 180.1)
- added C1005: 1u, Capacitor_SMD:C_0603_1608Metric_Pad1.08x0.95mm_HandSolder, F.Cu at (-30.0, 182.6)
- added C1006: 100n, Capacitor_SMD:C_0603_1608Metric_Pad1.08x0.95mm_HandSolder, F.Cu at (-30.0, 185.2)
- added C1007: 100n, Capacitor_SMD:C_0603_1608Metric_Pad1.08x0.95mm_HandSolder, F.Cu at (-30.0, 187.7)
- added C1008: 1u, Capacitor_SMD:C_0603_1608Metric_Pad1.08x0.95mm_HandSolder, F.Cu at (-30.0, 190.2)
- added C1009: 1u, Capacitor_SMD:C_0603_1608Metric_Pad1.08x0.95mm_HandSolder, F.Cu at (-30.0, 192.7)
- added C623: 10u/16V, Capacitor_SMD:C_1206_3216Metric_Pad1.33x1.80mm_HandSolder, F.Cu at (-123.3, 66.6)
- added C625: 47u/16V, Capacitor_SMD:C_1206_3216Metric_Pad1.33x1.80mm_HandSolder, F.Cu at (-123.3, 70.0)
- added C706: 10u/35V, Capacitor_SMD:C_1206_3216Metric_Pad1.33x1.80mm_HandSolder, F.Cu at (-37.2, 175.5)
- added C707: 2u2, Capacitor_SMD:C_0603_1608Metric_Pad1.08x0.95mm_HandSolder, F.Cu at (-42.4, 175.1)
- added C708: 10u/35V, Capacitor_SMD:C_1206_3216Metric_Pad1.33x1.80mm_HandSolder, F.Cu at (-37.2, 178.9)
- added C709: 2u2, Capacitor_SMD:C_0603_1608Metric_Pad1.08x0.95mm_HandSolder, F.Cu at (-42.4, 177.6)
- added C713: 10u/35V, Capacitor_SMD:C_1206_3216Metric_Pad1.33x1.80mm_HandSolder, F.Cu at (-37.2, 182.2)
- added C803: 10u/35V, Capacitor_SMD:C_1206_3216Metric_Pad1.33x1.80mm_HandSolder, F.Cu at (-49.6, 175.5)
- added C804: 10u/35V, Capacitor_SMD:C_1206_3216Metric_Pad1.33x1.80mm_HandSolder, F.Cu at (-49.6, 178.9)
- added C811: 10u/15V, Capacitor_SMD:C_1206_3216Metric_Pad1.33x1.80mm_HandSolder, F.Cu at (-49.6, 182.2)
- added C812: 10u/15V, Capacitor_SMD:C_1206_3216Metric_Pad1.33x1.80mm_HandSolder, F.Cu at (-49.6, 185.6)
- added C813: 10u/35V, Capacitor_SMD:C_1206_3216Metric_Pad1.33x1.80mm_HandSolder, F.Cu at (-49.6, 188.9)
- added C814: 10u/35V, Capacitor_SMD:C_1206_3216Metric_Pad1.33x1.80mm_HandSolder, F.Cu at (-49.6, 192.3)
- added C817: 10u/35V, Capacitor_SMD:C_1206_3216Metric_Pad1.33x1.80mm_HandSolder, F.Cu at (-49.6, 195.6)
- added C818: 10u/35V, Capacitor_SMD:C_1206_3216Metric_Pad1.33x1.80mm_HandSolder, F.Cu at (-49.6, 199.0)
- added D901: 1N4148W, Diode_SMD:D_SOD-123, F.Cu at (113.5, 50.1)
- added D902: 1N4148W, Diode_SMD:D_SOD-123, F.Cu at (113.5, 53.5)
- added D903: 1N4148W, Diode_SMD:D_SOD-123, F.Cu at (113.5, 56.8)
- added D904: 1N4148W, Diode_SMD:D_SOD-123, F.Cu at (113.5, 60.2)
- added D905: 1N4148W, Diode_SMD:D_SOD-123, F.Cu at (113.5, 63.5)
- added D906: 1N4148W, Diode_SMD:D_SOD-123, F.Cu at (113.5, 66.9)
- added D907: 1N4148W, Diode_SMD:D_SOD-123, F.Cu at (113.5, 70.2)
- added D908: 1N4148W, Diode_SMD:D_SOD-123, F.Cu at (119.3, 50.1)
- added D909: 1N4148W, Diode_SMD:D_SOD-123, F.Cu at (119.3, 53.5)
- added D910: 1N4148W, Diode_SMD:D_SOD-123, F.Cu at (119.3, 56.8)
- added D911: 1N4148W, Diode_SMD:D_SOD-123, F.Cu at (119.3, 60.2)
- added D912: 1N4148W, Diode_SMD:D_SOD-123, F.Cu at (119.3, 63.5)
- added D913: 1N4148W, Diode_SMD:D_SOD-123, F.Cu at (119.3, 66.9)
- added D914: 1N4148W, Diode_SMD:D_SOD-123, F.Cu at (119.3, 70.2)
- added D915: 1N4148W, Diode_SMD:D_SOD-123, F.Cu at (125.0, 50.1)
- added D916: 1N4148W, Diode_SMD:D_SOD-123, F.Cu at (125.0, 53.5)
- added D917: 1N4148W, Diode_SMD:D_SOD-123, F.Cu at (125.0, 56.8)
- added D918: 1N4148W, Diode_SMD:D_SOD-123, F.Cu at (125.0, 60.2)
- added J1101: Conn_02x04_Odd_Even, Connector_PinHeader_2.54mm:PinHeader_2x04_P2.54mm_Vertical, F.Cu at (111.7, 111.2)
- added J601: Conn_02x06_Odd_Even, Connector_PinHeader_2.54mm:PinHeader_2x06_P2.54mm_Vertical, F.Cu at (111.7, 90.7)
- added J901: Conn_02x06_Odd_Even, Connector_PinHeader_2.54mm:PinHeader_2x06_P2.54mm_Vertical, F.Cu at (212.7, 52.6)
- added K901: 9012, ETH1CREF1A:9012, F.Cu at (81.7, 51.1)
- added K902: 9012, ETH1CREF1A:9012, F.Cu at (81.7, 56.4)
- added K903: 9012, ETH1CREF1A:9012, F.Cu at (81.7, 61.8)
- added K904: 9012, ETH1CREF1A:9012, F.Cu at (81.7, 67.1)
- added K905: 9012, ETH1CREF1A:9012, F.Cu at (81.7, 72.4)
- added K906: 9012, ETH1CREF1A:9012, F.Cu at (81.7, 77.7)
- added K907: 9012, ETH1CREF1A:9012, F.Cu at (93.3, 51.1)
- added K908: 9012, ETH1CREF1A:9012, F.Cu at (93.3, 56.4)
- added K909: 9012, ETH1CREF1A:9012, F.Cu at (93.3, 61.8)
- added K910: 9012, ETH1CREF1A:9012, F.Cu at (93.3, 67.1)
- added K911: 9012, ETH1CREF1A:9012, F.Cu at (93.3, 72.4)
- added K912: 9012, ETH1CREF1A:9012, F.Cu at (93.3, 77.7)
- added K913: 9012, ETH1CREF1A:9012, F.Cu at (104.8, 51.1)
- added K914: 9012, ETH1CREF1A:9012, F.Cu at (104.8, 56.4)
- added K915: 9012, ETH1CREF1A:9012, F.Cu at (104.8, 61.8)
- added K916: 9012, ETH1CREF1A:9012, F.Cu at (104.8, 67.1)
- added K917: 9012, ETH1CREF1A:9012, F.Cu at (104.8, 72.4)
- added K918: 9012, ETH1CREF1A:9012, F.Cu at (104.8, 77.7)
- added R1008: TNPV12061M00BYEN, Resistor_SMD:R_1206_3216Metric_Pad1.30x1.75mm_HandSolder, F.Cu at (-24.9, 175.5)
- added R1009: TNPU1206100KBZEN00, Resistor_SMD:R_1206_3216Metric_Pad1.30x1.75mm_HandSolder, F.Cu at (-24.9, 178.8)
- added R1010: TNPU120610K0AWEN00, Resistor_SMD:R_1206_3216Metric_Pad1.30x1.75mm_HandSolder, F.Cu at (-24.9, 182.1)
- added R1011: TNPU12061K00AWEN00, Resistor_SMD:R_1206_3216Metric_Pad1.30x1.75mm_HandSolder, F.Cu at (-24.9, 185.4)
- added R1012: TNPU1206100RAZEN00, Resistor_SMD:R_1206_3216Metric_Pad1.30x1.75mm_HandSolder, F.Cu at (-24.9, 188.7)
- added R1013: RNCF1206AKT10R0, Resistor_SMD:R_1206_3216Metric_Pad1.30x1.75mm_HandSolder, F.Cu at (-24.9, 191.9)
- added R706: 5k/.1%, Resistor_SMD:R_0603_1608Metric_Pad0.98x0.95mm_HandSolder, F.Cu at (-42.4, 180.1)
- added R707: 2k/.1%, Resistor_SMD:R_0603_1608Metric_Pad0.98x0.95mm_HandSolder, F.Cu at (-42.4, 182.6)
- added R710: 6k98/.1%, Resistor_SMD:R_0603_1608Metric_Pad0.98x0.95mm_HandSolder, F.Cu at (-42.4, 185.2)
- added R711: 10k/.1%, Resistor_SMD:R_0603_1608Metric_Pad0.98x0.95mm_HandSolder, F.Cu at (-42.4, 187.7)
- added R712: 1k96/.1%, Resistor_SMD:R_0603_1608Metric_Pad0.98x0.95mm_HandSolder, F.Cu at (-42.4, 190.2)
- added R713: 3k01/.1%, Resistor_SMD:R_0603_1608Metric_Pad0.98x0.95mm_HandSolder, F.Cu at (-42.4, 195.2)
- added R714: 10k/.1%, Resistor_SMD:R_0603_1608Metric_Pad0.98x0.95mm_HandSolder, F.Cu at (-42.4, 192.7)
- added U609: LM1117DTX-3.3/NOPB, Package_TO_SOT_SMD:TO-252-2, F.Cu at (-119.4, 60.9)
- C705, C712: value 22u/35V -> 10u/35V
- R708: value 62 -> 7k5
- U1105, U1106, U1107, U1108: footprint Package_TO_SOT_SMD:SOT-563 -> Package_TO_SOT_SMD:SOT-23-6
- U202: value STM32F746ZG -> STM32F429ZIT
- U605: footprint Package_TO_SOT_SMD:TO-263-2 -> Package_TO_SOT_SMD:TO-252-2
- U607: value TSR1-2450 -> TSR1-2490
- U608: value LM1117DTX-3.3/NOPB -> LM1117DTX-5/NOPB
- moved C219 163.8 mm to (-28.4, 108.7)
- moved C220 163.8 mm to (-28.4, 111.2)
- moved C221 163.8 mm to (-28.4, 113.7)
- moved C222 163.8 mm to (-28.4, 116.3)
- moved C703 163.8 mm to (-0.91, 160.2)
- moved C705 163.8 mm to (-0.91, 164.5)
- moved C715 163.8 mm to (-9.92, 141.8)
- moved C815 163.8 mm to (-18.0, 58.2)
- moved C816 163.8 mm to (-18.0, 60.7)
- moved C819 163.8 mm to (-18.0, 63.2)
- moved D201 163.8 mm to (-31.5, 131.4)
- moved D202 163.8 mm to (-31.5, 133.9)
- moved D203 163.8 mm to (-31.5, 136.5)
- moved D401 163.8 mm to (-29.0, 64.7)
- moved D402 163.8 mm to (-32.6, 59.7)
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- renumbered C623 to C624, K901 to K919, K902 to K920, K903 to K921, K904 to K922, K905 to K923, K906 to K924
Connections:
- net /Connect/A renamed /Relays/A_MODULE
- net /Connect/B renamed /Relays/B_MODULE
- net /Connect/C renamed /Relays/C_MODULE
- net /Connect/D renamed /Relays/D_MODULE
- net /Connect/E renamed /Relays/E_MODULE
- net /Connect/F renamed /Relays/F_MODULE
- net /Ethernet/MDIO renamed /Ethernet/RMII_MDIO
- net /Relays/VOUT renamed /Current Source/VOUT
- C622 pad 1: +5V -> Net-(U607-VO)
- C624 pad 1: +3.3V -> +5V
- U1003 pad 5: /Relays/AOUT -> /Current Source/AOUT
- U1101 pad 1: /GPIO/photoMOS10 -> /GPIO/relay10
- U1101 pad 15: /GPIO/photoMOS9 -> /GPIO/relay9
- U1101 pad 2: /GPIO/photoMOS11 -> /GPIO/relay11
- U1101 pad 3: /GPIO/photoMOS12 -> /GPIO/relay12
- U1101 pad 4: /GPIO/photoMOS13 -> /GPIO/relay13
- U1101 pad 5: /GPIO/photoMOS14 -> /GPIO/relay14
- U1101 pad 6: /GPIO/photoMOS15 -> /GPIO/relay15
- U1101 pad 7: /GPIO/photoMOS16 -> /GPIO/relay16
- U1102 pad 15: /GPIO/photoMOS17 -> /GPIO/relay17
- U1103 pad 1: /GPIO/photoMOS2 -> /GPIO/relay2
- U1103 pad 15: /GPIO/photoMOS1 -> /GPIO/relay1
- U1103 pad 2: /GPIO/photoMOS3 -> /GPIO/relay3
- U1103 pad 3: /GPIO/photoMOS4 -> /GPIO/relay4
- U1103 pad 4: /GPIO/photoMOS5 -> /GPIO/relay5
- U1103 pad 5: /GPIO/photoMOS6 -> /GPIO/relay6
- U1103 pad 6: /GPIO/photoMOS7 -> /GPIO/relay7
- U1103 pad 7: /GPIO/photoMOS8 -> /GPIO/relay8
- U1104 pad 7: /GPIO/photoMOS0 -> /GPIO/relay0
- U1105 pad 4: /GPIO/SR_DAT -> /GPIO/SER
- U1106 pad 4: /GPIO/SR_CLK -> /GPIO/SRCLK
- U1107 pad 4: /GPIO/SR_LAT -> /GPIO/RCLK
- U1108 pad 4: /GPIO/SR_OUT -> /GPIO/QH
- U202 pad 1: /MCU/SPI4_SCK -> unconnected-(U202-PE2,TRACECLK,SPI4_SCK,SAI1_MCLK_A,ETH_MII_TXD3,FMC_A23,EVENTOUT-Pad1)
- U202 pad 10: unconnected-(U202-PF0,I2C2_SDA,FMC_A0,EVENTOUT-Pad10) -> /MCU/EEPROM_SDA
- U202 pad 100: unconnected-(U202-PA8,MCO1,TIM1_CH1,TIM8_BKIN2,I2C3_SCL,USART1_CK,OTG_FS_SOF,CAN3_RX,UART7_RX,LCD_B3,LCD_R6,EVENTOUT-Pad100) -> /GPIO/MODE_I2C_SCL
- U202 pad 11: unconnected-(U202-PF1,I2C2_SCL,FMC_A1,EVENTOUT-Pad11) -> /MCU/EEPROM_SCL
- U202 pad 110: /MCU/SPI3_NSS -> /DAC/~{SYNC}
- U202 pad 111: /MCU/SPI3_SCK -> /DAC/SCLK
- U202 pad 112: /MCU/SPI3_MISO -> /DAC/SDO
- U202 pad 113: /MCU/SPI3_MOSI -> /DAC/SDIN
- U202 pad 135: /MCU/SPI1_MOSI -> unconnected-(U202-PB5,TIM3_CH2,I2C1_SMBA,SPI1_MOSI,SPI3_MOSI,I2S3_SD,CAN2_RX,OTG_HS_ULPI_D7,ETH_PPS_OUT,FMC_SDCKE1,DCMI_D10,EVENTOUT-Pad135)
- U202 pad 136: unconnected-(U202-PB6,UART5_TX,TIM4_CH1,HDMI_CEC,I2C1_SCL,DFSDM1_DATIN5,USART1_TX,CAN2_TX,QUADSPI_BK1_NCS,I2C4_SCL,FMC_SDNE1,DCMI_D5,EVENTOUT-Pad136) -> /MCU/SENS_SCL
- U202 pad 137: unconnected-(U202-PB7,TIM4_CH2,I2C1_SDA,DFSDM1_CKIN5,USART1_RX,I2C4_SDA,FMC_NL,DCMI_VSYNC,EVENTOUT-Pad137) -> /MCU/SENS_SDA
- U202 pad 18: /MCU/SPI5_NSS -> /GPIO/SPI5_NSS
- U202 pad 19: /MCU/SPI5_SCK -> /GPIO/SPI5_SCK
- U202 pad 20: /MCU/SPI5_MISO -> /GPIO/SPI5_MISO
- U202 pad 21: /MCU/SPI5_MOSI -> /GPIO/SPI5_MOSI
- U202 pad 3: /MCU/SPI4_NSS -> unconnected-(U202-PE4,TRACED1,SPI4_NSS,SAI1_FS_A,FMC_A20,DCMI_D4,LCD_B0,EVENTOUT-Pad3)
- U202 pad 4: /MCU/SPI4_MISO -> unconnected-(U202-PE5,TRACED2,TIM9_CH1,SPI4_MISO,SAI1_SCK_A,FMC_A21,DCMI_D6,LCD_G0,EVENTOUT-Pad4)
- U202 pad 40: /MCU/SPI1_NSS -> unconnected-(U202-PA4,SPI1_NSS,SPI3_NSS,I2S3_WS,USART2_CK,OTG_HS_SOF,DCMI_HSYNC,LCD_VSYNC,EVENTOUT,ADC1_IN4,ADC2_IN4,DAC_OUT1-Pad40)
- U202 pad 41: /MCU/SPI1_SCK -> unconnected-(U202-PA5,TIM2_CH1,TIM2_ETR,TIM8_CH1N,SPI1_SCK,OTG_HS_ULPI_CK,EVENTOUT,ADC1_IN5,ADC2_IN5,DAC_OUT2-Pad41)
- U202 pad 42: /MCU/SPI1_MISO -> unconnected-(U202-PA6,TIM1_BKIN,TIM3_CH1,TIM8_BKIN,SPI1_MISO,TIM13_CH1,DCMI_PIXCLK,LCD_G2,EVENTOUT,ADC1_IN6,ADC2_IN6-Pad42)
- U202 pad 5: /MCU/SPI4_MOSI -> unconnected-(U202-PE6,TRACED3,TIM9_CH2,SPI4_MOSI,SAI1_SD_A,FMC_A22,DCMI_D7,LCD_G1,EVENTOUT-Pad5)
- U202 pad 73: /MCU/SPI2_NSS -> /GPIO/RCLK
- U202 pad 74: /MCU/SPI2_SCK -> /GPIO/SRCLK
- U202 pad 75: /MCU/SPI2_MISO -> /GPIO/QH
- U202 pad 76: /MCU/SPI2_MOSI -> /GPIO/SER
- U202 pad 81: /MCU/EEPROM_SCL -> unconnected-(U202-PD12,TIM4_CH1,USART3_RTS,FMC_A17,EVENTOUT-Pad81)
- U202 pad 82: /MCU/EEPROM_SDA -> unconnected-(U202-PD13,TIM4_CH2,FMC_A18,EVENTOUT-Pad82)
- U202 pad 99: unconnected-(U202-PC9,MCO2,TIM3_CH4,TIM8_CH4,I2C3_SDA,I2S_CKIN,UART5_CTS,QUADSPI_BK1_IO0,LCD_G3,SDMMC1_D1,DCMI_D3,LCD_B2,EVENTOUT-Pad99) -> /GPIO/MODE_I2C_SDA
- U607 pad 3: +5V -> Net-(U607-VO)
- U608 pad 2: +3.3V -> +5V
- U608 pad 3: +5V -> Net-(U607-VO)
Other:
- board outline added: 160 x 100 mm

Commit message: Hardware
Parts:
- removed K919, K920, K921, K922, K923, K924: HE3621A0510, ETH1CREF1A:HE360_x-5050462-8
- removed R1008: TNPV12061M00BYEN, Resistor_SMD:R_1206_3216Metric_Pad1.30x1.75mm_HandSolder
- removed R1009: TNPU1206100KBZEN00, Resistor_SMD:R_1206_3216Metric_Pad1.30x1.75mm_HandSolder
- removed R1010: TNPU120610K0AWEN00, Resistor_SMD:R_1206_3216Metric_Pad1.30x1.75mm_HandSolder
- removed R1011: TNPU12061K00AWEN00, Resistor_SMD:R_1206_3216Metric_Pad1.30x1.75mm_HandSolder
- removed R1012: TNPU1206100RAZEN00, Resistor_SMD:R_1206_3216Metric_Pad1.30x1.75mm_HandSolder
- removed R1013: RNCF1206AKT10R0, Resistor_SMD:R_1206_3216Metric_Pad1.30x1.75mm_HandSolder
- removed U1005, U1006, U1007, U1008, U1009, U1010: AQY211G2SX, ETH1CREF1A:AQY212GS
- removed U913: ULN2003A, Package_SO:TSSOP-16_4.4x5mm_P0.65mm
- added C1101: 100n, Capacitor_SMD:C_0603_1608Metric_Pad1.08x0.95mm_HandSolder, B.Cu at (148.0, 92.5)
- added C1102: 100n, Capacitor_SMD:C_0603_1608Metric_Pad1.08x0.95mm_HandSolder, B.Cu at (152.0, 89.9)
- added C1103: 100n, Capacitor_SMD:C_0603_1608Metric_Pad1.08x0.95mm_HandSolder, B.Cu at (143.9, 92.5)
- added C1104: 100n, Capacitor_SMD:C_0603_1608Metric_Pad1.08x0.95mm_HandSolder, B.Cu at (142.5, 86.2)
- added C1105: 100n, Capacitor_SMD:C_0603_1608Metric_Pad1.08x0.95mm_HandSolder, B.Cu at (152.0, 92.5)
- added C1106: 100n, Capacitor_SMD:C_0603_1608Metric_Pad1.08x0.95mm_HandSolder, B.Cu at (148.0, 89.9)
- added C1107: 100n, Capacitor_SMD:C_0603_1608Metric_Pad1.08x0.95mm_HandSolder, B.Cu at (139.8, 92.5)
- added C1108: 100n, Capacitor_SMD:C_0603_1608Metric_Pad1.08x0.95mm_HandSolder, B.Cu at (134.1, 86.2)
- added C1109: 100n, Capacitor_SMD:C_0603_1608Metric_Pad1.08x0.95mm_HandSolder, B.Cu at (143.9, 89.9)
- added C1110: 100n, Capacitor_SMD:C_0603_1608Metric_Pad1.08x0.95mm_HandSolder, B.Cu at (139.8, 89.9)
- added C1111: 100n, Capacitor_SMD:C_0603_1608Metric_Pad1.08x0.95mm_HandSolder, B.Cu at (159.3, 86.2)
- added C1112: 100n, Capacitor_SMD:C_0603_1608Metric_Pad1.08x0.95mm_HandSolder, B.Cu at (150.9, 86.2)
- added D1001: 1N4148W, Diode_SMD:D_SOD-123, B.Cu at (154.9, 45.6)
- added D1002: 1N4148W, Diode_SMD:D_SOD-123, B.Cu at (154.9, 49.9)
- added D1003: 1N4148W, Diode_SMD:D_SOD-123, B.Cu at (154.9, 54.2)
- added D1004: 1N4148W, Diode_SMD:D_SOD-123, B.Cu at (154.9, 58.5)
- added D1005: 1N4148W, Diode_SMD:D_SOD-123, B.Cu at (154.9, 62.9)
- added D1006: 1N4148W, Diode_SMD:D_SOD-123, B.Cu at (154.9, 67.2)
- added F601: MF-LSMF185/33X, ETH1CREF1A:Fuse_SMD2920, B.Cu at (216.9, 134.4)
- added H101: MountingHole, MountingHole:MountingHole_3.2mm_M3_DIN965_Pad_TopBottom, F.Cu at (213.0, 46.0)
- added H102: MountingHole, MountingHole:MountingHole_3.2mm_M3_DIN965_Pad_TopBottom, F.Cu at (76.0, 46.0)
- added H103: MountingHole, MountingHole:MountingHole_3.2mm_M3_DIN965_Pad_TopBottom, F.Cu at (76.0, 134.0)
- added K1001: 9012, ETH1CREF1A:9012, F.Cu at (154.9, 47.6)
- added K1002: 9012, ETH1CREF1A:9012, F.Cu at (154.9, 51.9)
- added K1003: 9012, ETH1CREF1A:9012, F.Cu at (154.9, 56.3)
- added K1004: 9012, ETH1CREF1A:9012, F.Cu at (154.9, 60.6)
- added K1005: 9012, ETH1CREF1A:9012, F.Cu at (154.9, 64.9)
- added K1006: 9012, ETH1CREF1A:9012, F.Cu at (154.9, 69.2)
- C1001: value 200p -> 100n
- C1003, C1007: value 100n -> 1u
- C1005: value 1u -> 100n
- C1009: value 1u -> 200p
- C616, C617, C715, D901, D902, D903, D904, D905, D906, D907, D908, D909, D910, D911, D912, D913, D914, D915, D916, D917, D918, R611, R612: moved to B.Cu
- C703: footprint Capacitor_SMD:C_1210_3225Metric_Pad1.33x2.70mm_HandSolder -> Capacitor_SMD:C_0603_1608Metric_Pad1.08x0.95mm_HandSolder
- FB201, FB301: value 742792031 -> 600; footprint Inductor_SMD:L_0805_2012Metric_Pad1.15x1.40mm_HandSolder -> Inductor_SMD:L_0603_1608Metric_Pad1.05x0.95mm_HandSolder
- R1002: value 680 -> TNPV12061M00BYEN; footprint Resistor_SMD:R_0603_1608Metric_Pad0.98x0.95mm_HandSolder -> Resistor_SMD:R_1206_3216Metric_Pad1.30x1.75mm_HandSolder
- R1003: value 680 -> TNPU1206100KBZEN00; footprint Resistor_SMD:R_0603_1608Metric_Pad0.98x0.95mm_HandSolder -> Resistor_SMD:R_1206_3216Metric_Pad1.30x1.75mm_HandSolder
- R1004: value 680 -> TNPU120610K0AWEN00; footprint Resistor_SMD:R_0603_1608Metric_Pad0.98x0.95mm_HandSolder -> Resistor_SMD:R_1206_3216Metric_Pad1.30x1.75mm_HandSolder
- R1005: value 680 -> TNPU12061K00AWEN00; footprint Resistor_SMD:R_0603_1608Metric_Pad0.98x0.95mm_HandSolder -> Resistor_SMD:R_1206_3216Metric_Pad1.30x1.75mm_HandSolder
- R1006: value 680 -> TNPU1206100RAZEN00; footprint Resistor_SMD:R_0603_1608Metric_Pad0.98x0.95mm_HandSolder -> Resistor_SMD:R_1206_3216Metric_Pad1.30x1.75mm_HandSolder
- R1007: value 680 -> RNCF1206AKT10R0; footprint Resistor_SMD:R_0603_1608Metric_Pad0.98x0.95mm_HandSolder -> Resistor_SMD:R_1206_3216Metric_Pad1.30x1.75mm_HandSolder
- U604: value MC7815BD2TG -> MC7815CD2TG
- U605: value MC7915BD2TG -> MC7915CD2TR4G; footprint Package_TO_SOT_SMD:TO-252-2 -> Package_TO_SOT_SMD:TO-263-2
- U703: value AD8676BRZ -> LT1021DCS8-7#PBF
- U704: value LT1021DCS8-7#PBF -> LM399H; footprint Package_SO:SOIC-8_3.9x4.9mm_P1.27mm -> ETH1CREF1A:LMx99
- U705: value LM399H -> AD8676BRZ; footprint ETH1CREF1A:LMx99 -> Package_SO:SOIC-8_3.9x4.9mm_P1.27mm
- moved D601 306.1 mm to (215.0, 134.4), turned to 180 degrees
- moved L603 285.5 mm to (205.6, 130.3), turned to -90 degrees
- moved U601 280.4 mm to (214.2, 113.3)
- moved Q601 268.7 mm to (205.5, 114.9), turned to -90 degrees
- moved U609 265.7 mm to (138.2, 126.2), turned to 90 degrees
- moved L604 261.2 mm to (164.3, 119.5), turned to -90 degrees
- moved C617 260.0 mm to (184.4, 132.2)
- moved C616 254.2 mm to (184.4, 111.9)
- moved U302 254.0 mm to (203.7, 95.8), turned to -90 degrees
- moved R1002 249.8 mm to (163.8, 47.6)
- moved R1003 249.1 mm to (163.8, 51.9)
- moved R1004 248.3 mm to (163.8, 56.3)
- moved R612 248.2 mm to (174.2, 125.2), turned to -90 degrees
- moved U303 248.2 mm to (203.7, 101.9), turned to -90 degrees
- moved R1005 247.5 mm to (163.8, 60.6)
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Connections:
- C1001 pad 1: Net-(U1003A--) -> -15VF
- C1001 pad 2: Net-(U1004-+) -> AGNDF
- C1005 pad 1: -15VF -> +15VF
- C1009 pad 1: +15VF -> Net-(U1003A--)
- C1009 pad 2: AGNDF -> Net-(U1004-+)
- C709 pad 1: Net-(U702-OUT) -> Net-(U701A-+)
- C710 pad 1: Net-(U703C-V-) -> Net-(U705C-V-)
- C711 pad 1: Net-(U703C-V+) -> Net-(U705C-V+)
- C712 pad 1: Net-(U703C-V-) -> Net-(U705C-V-)
- C713 pad 1: Net-(U703C-V+) -> Net-(U705C-V+)
- C714 pad 1: Net-(U701A-+) -> Net-(U705A-+)
- C715 pad 1: Net-(U701A--) -> Net-(U705A--)
- D601 pad 1: +24V -> Net-(D601-K)
- D905 pad 2: /GPIO/relay1 -> /GPIO/relay16
- D906 pad 2: /GPIO/relay5 -> /GPIO/relay1
- D907 pad 2: /GPIO/relay9 -> /GPIO/relay5
- D908 pad 2: /GPIO/relay13 -> /GPIO/relay9
- D909 pad 2: /GPIO/relay2 -> /GPIO/relay13
- D910 pad 2: /GPIO/relay6 -> /GPIO/relay17
- D911 pad 2: /GPIO/relay10 -> /GPIO/relay2
- D912 pad 2: /GPIO/relay7 -> /GPIO/relay6
- D913 pad 2: /GPIO/relay3 -> /GPIO/relay10
- D914 pad 2: /GPIO/relay11 -> /GPIO/relay14
- D915 pad 2: /GPIO/relay14 -> /GPIO/relay7
- D916 pad 2: /GPIO/relay15 -> /GPIO/relay3
- D917 pad 2: /GPIO/relay16 -> /GPIO/relay11
- D918 pad 2: /GPIO/relay17 -> /GPIO/relay15
- FB201 pad 1: /MCU/MCU_VDDA -> +3.3V
- FB201 pad 2: +3.3V -> /MCU/MCU_VDDA
- FB301 pad 1: VCCQ -> +3.3V
- FB301 pad 2: +3.3V -> VCCQ
- FB703 pad 2: Net-(U703C-V-) -> Net-(U705C-V-)
- FB704 pad 2: Net-(U703C-V+) -> Net-(U705C-V+)
- J501 pad A2: /Relays/A_MODULE -> /Relays/A_AOUT
- J501 pad A3: /Relays/B_MODULE -> /Relays/B_AOUT
- J501 pad A4: /Relays/C_MODULE -> /Relays/C_AOUT
- J501 pad A5: /Relays/D_MODULE -> /Relays/D_AOUT
- J501 pad A6: /Relays/E_MODULE -> /Relays/E_AOUT
- J501 pad A7: /Relays/F_MODULE -> /Relays/F_AOUT
- J501 pad C2: /Relays/A_MODULE -> /Relays/A_AOUT
- J501 pad C3: /Relays/B_MODULE -> /Relays/B_AOUT
- J501 pad C4: /Relays/C_MODULE -> /Relays/C_AOUT
- J501 pad C5: /Relays/D_MODULE -> /Relays/D_AOUT
- J501 pad C6: /Relays/E_MODULE -> /Relays/E_AOUT
- J501 pad C7: /Relays/F_MODULE -> /Relays/F_AOUT
- J901 pad 1: /Relays/A_MODULE -> /Relays/A_AOUT
- J901 pad 10: /Relays/E_MODULE -> /Relays/E_AOUT
- J901 pad 11: /Relays/F_MODULE -> /Relays/F_AOUT
- J901 pad 12: /Relays/F_MODULE -> /Relays/F_AOUT
- J901 pad 2: /Relays/A_MODULE -> /Relays/A_AOUT
- J901 pad 3: /Relays/B_MODULE -> /Relays/B_AOUT
- J901 pad 4: /Relays/B_MODULE -> /Relays/B_AOUT
- J901 pad 5: /Relays/C_MODULE -> /Relays/C_AOUT
- J901 pad 6: /Relays/C_MODULE -> /Relays/C_AOUT
- J901 pad 7: /Relays/D_MODULE -> /Relays/D_AOUT
- J901 pad 8: /Relays/D_MODULE -> /Relays/D_AOUT
- J901 pad 9: /Relays/E_MODULE -> /Relays/E_AOUT
- K902 pad 3: /GPIO/relay1 -> /GPIO/relay4
- K903 pad 3: /GPIO/relay2 -> /GPIO/relay8
- K904 pad 3: /GPIO/relay3 -> /GPIO/relay12
- K905 pad 3: /GPIO/relay4 -> /GPIO/relay16
- K906 pad 3: /GPIO/relay5 -> /GPIO/relay1
- K907 pad 3: /GPIO/relay6 -> /GPIO/relay5
- K908 pad 3: /GPIO/relay7 -> /GPIO/relay9
- K909 pad 3: /GPIO/relay8 -> /GPIO/relay13
- K910 pad 3: /GPIO/relay9 -> /GPIO/relay17
- K911 pad 3: /GPIO/relay10 -> /GPIO/relay2
- K912 pad 3: /GPIO/relay11 -> /GPIO/relay6
- K913 pad 3: /GPIO/relay12 -> /GPIO/relay10
- K914 pad 3: /GPIO/relay13 -> /GPIO/relay14
- K915 pad 3: /GPIO/relay14 -> /GPIO/relay7
- K916 pad 3: /GPIO/relay15 -> /GPIO/relay3
- K917 pad 3: /GPIO/relay16 -> /GPIO/relay11
- K918 pad 3: /GPIO/relay17 -> /GPIO/relay15
- Q601 pad 3: +24V -> Net-(D601-K)
- R1002 pad 1: +5V -> Net-(K1001-Pad4)
- R1002 pad 2: Net-(R1002-Pad2) -> /Current Source/AOUT
- R1003 pad 1: +5V -> Net-(K1002-Pad4)
- R1003 pad 2: Net-(R1003-Pad2) -> /Current Source/AOUT
- R1004 pad 1: +5V -> Net-(K1003-Pad4)
- R1004 pad 2: Net-(R1004-Pad2) -> /Current Source/AOUT
- R1005 pad 1: +5V -> Net-(K1004-Pad4)
- R1005 pad 2: Net-(R1005-Pad2) -> /Current Source/AOUT
- R1006 pad 1: +5V -> Net-(K1005-Pad4)
- R1006 pad 2: Net-(R1006-Pad2) -> /Current Source/AOUT
- R1007 pad 1: +5V -> Net-(K1006-Pad4)
- R1007 pad 2: Net-(R1007-Pad2) -> /Current Source/AOUT
- R601 pad 1: +24V -> Net-(D601-K)
- R703 pad 1: Net-(U701A-+) -> Net-(U705A-+)
- R703 pad 2: Net-(U704-Vout) -> Net-(U703-Vout)
- R704 pad 2: Net-(U703C-V-) -> Net-(U705C-V-)
- R705 pad 2: Net-(U703C-V+) -> Net-(U705C-V+)
- R706 pad 2: Net-(U703A--) -> Net-(U701A--)
- R707 pad 1: Net-(U703A--) -> Net-(U701A--)
- R708 pad 2: Net-(U701A-+) -> Net-(U705A-+)
- R709 pad 1: Net-(U701A-+) -> Net-(U705A-+)
- R710 pad 2: Net-(U701A--) -> Net-(U705A--)
- R711 pad 2: Net-(U701B--) -> Net-(U705B--)
- R712 pad 1: Net-(U701A-+) -> Net-(U705A-+)
- R713 pad 1: Net-(U701A--) -> Net-(U705A--)
- R714 pad 1: Net-(U701B--) -> Net-(U705B--)
- U202 pad 114: /MCU/CXN_REL6 -> unconnected-(U202-PD0,CAN1_RX,FMC_D2,EVENTOUT-Pad114)
- U202 pad 115: /MCU/CXN_REL5 -> unconnected-(U202-PD1,CAN1_TX,FMC_D3,EVENTOUT-Pad115)
- U202 pad 116: /MCU/CXN_REL4 -> unconnected-(U202-PD2,TIM3_ETR,UART5_RX,SDIO_CMD,DCMI_D11,EVENTOUT-Pad116)
- U202 pad 117: /MCU/CXN_REL3 -> unconnected-(U202-PD3,SPI2_SCK,I2S2_CK,USART2_CTS,FMC_CLK,DCMI_D5,LCD_G7,EVENTOUT-Pad117)
- U202 pad 118: /MCU/CXN_REL2 -> unconnected-(U202-PD4,USART2_RTS,FMC_NOE,EVENTOUT-Pad118)
- U202 pad 119: /MCU/CXN_REL1 -> unconnected-(U202-PD5,USART2_TX,FMC_NWE,EVENTOUT-Pad119)
- U601 pad 1: +24V -> Net-(D601-K)
- U701 pad 1: /Reference Voltage/REF_+10V -> Net-(R707-Pad2)
- U701 pad 7: /DAC/REF_-10V -> Net-(U701B--)
- U702 pad 6: Net-(U702-OUT) -> Net-(U701A-+)
- U703 pad 1: Net-(R707-Pad2) -> unconnected-(U703-DNC-Pad1)
- U703 pad 2: Net-(U703A--) -> +15VF
- U703 pad 3: Net-(U702-OUT) -> unconnected-(U703-DNC-Pad3)
- U703 pad 4: Net-(U703C-V-) -> AGNDF
- U703 pad 5: AGNDF -> unconnected-(U703-DNC-Pad5)
- U703 pad 6: Net-(U703B--) -> Net-(U703-Vout)
- U703 pad 7: Net-(U703B--) -> unconnected-(U703-DNC-Pad7)
- U703 pad 8: Net-(U703C-V+) -> unconnected-(U703-DNC-Pad8)
- U704 pad 1: unconnected-(U704-DNC-Pad1) -> Net-(U705A-+)
- U704 pad 2: +15VF -> AGNDF
- U704 pad 3: unconnected-(U704-DNC-Pad3) -> +15VF
- U704 pad 4: AGNDF -> -15VF
- U705 pad 1: Net-(U701A-+) -> /Reference Voltage/REF_+10V
- U705 pad 2: AGNDF -> Net-(U705A--)
- U705 pad 3: +15VF -> Net-(U705A-+)
- U705 pad 4: -15VF -> Net-(U705C-V-)
Other:
- copper layers 2 -> 4

Commit message: Hardware
Parts:
- added C609: 2u2/50V, Capacitor_SMD:C_1206_3216Metric_Pad1.33x1.80mm_HandSolder, F.Cu at (216.5, 127.4)
- added C622: 10u/50V, Capacitor_SMD:C_1206_3216Metric_Pad1.33x1.80mm_HandSolder, B.Cu at (165.1, 132.8)
- added C624: 10u/50V, Capacitor_SMD:C_1206_3216Metric_Pad1.33x1.80mm_HandSolder, B.Cu at (160.4, 132.5)
- added J101: 36107406S, ETH1CREF1A:36107406S, F.Cu at (40.9, 66.2)
- added L605: TCK-141, ETH1CREF1A:TCK-141, F.Cu at (165.1, 132.8)
- added U608: TSR1-2450, ETH1CREF1A:TSR1, F.Cu at (155.8, 130.8)
- C201, C202, C203, C204, C205, C206, C207, C208, C209, C210, C211, C212, C213, C214, C215, C216, C217, C220, C221, FB201, R207, R208, R209, U203, Y201: moved to B.Cu
- C621: renamed from C620; moved to B.Cu
- C623: renamed from C621; moved to B.Cu
- C625: renamed from C622; moved to B.Cu
- C626: renamed from C623; moved to B.Cu
- moved C612 309.6 mm to (213.2, 127.4), turned to -90 degrees
- moved R601 293.9 mm to (214.6, 109.3)
- moved C628 293.4 mm to (165.1, 124.2)
- moved R606 289.5 mm to (213.2, 117.2), turned to 90 degrees
- moved C626 282.3 mm to (151.3, 132.3), turned to -90 degrees
- moved D604 282.1 mm to (216.2, 117.2), turned to 90 degrees
- moved D603 280.6 mm to (213.2, 121.4), turned to 90 degrees
- moved C621 239.2 mm to (145.9, 132.2), turned to 90 degrees
- moved C627 234.3 mm to (145.8, 124.0)
- moved C623 233.8 mm to (141.4, 132.1), turned to -90 degrees
- moved C625 223.9 mm to (132.1, 132.1), turned to -90 degrees
- moved D203 198.5 mm to (164.7, 106.9)
- moved Y201 198.2 mm to (148.5, 114.0)
- moved D202 197.8 mm to (164.7, 109.6)
- moved D201 197.2 mm to (164.7, 112.3)
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- renumbered C609 to C610, C610 to C611, C611 to C612, C612 to C613, C613 to C614, C614 to C615, C615 to C616, C616 to C617, C617 to C618, C618 to C619, C619 to C620, C624 to C627, C625 to C628, D604 to D603, D605 to D604, D603 to D605, U608 to U609, U609 to U610
Connections:
- C612 pad 1: VCCQ -> Net-(D603-K)
- C626 pad 1: +5V -> Net-(U608-VO)
- D603 pad 1: VCCQ -> Net-(D603-K)
- L603 pad 2: VCCQ -> Net-(D603-K)
- Q601 pad 2: VCCQ -> Net-(D603-K)
- U601 pad 2: VCCQ -> Net-(D603-K)
- U610 pad 3: +5V -> Net-(U608-VO)

Commit message: Hardware
Parts:
- added C1001: 100n, Capacitor_SMD:C_0603_1608Metric_Pad1.08x0.95mm_HandSolder, B.Cu at (137.0, 51.4)
- added C1004: 1u, Capacitor_SMD:C_0603_1608Metric_Pad1.08x0.95mm_HandSolder, B.Cu at (138.6, 51.4)
- added C1007: 100n, Capacitor_SMD:C_0603_1608Metric_Pad1.08x0.95mm_HandSolder, B.Cu at (142.7, 50.5)
- added C1010: 1u, Capacitor_SMD:C_0603_1608Metric_Pad1.08x0.95mm_HandSolder, B.Cu at (144.3, 50.5)
- C1002: renamed from C1001; moved to B.Cu
- C1003: renamed from C1002; moved to B.Cu
- C1005: renamed from C1003; moved to B.Cu
- C1006: renamed from C1004; moved to B.Cu
- C1008: renamed from C1005; moved to B.Cu
- C1009: renamed from C1006; moved to B.Cu
- C1011: renamed from C1007; moved to B.Cu
- C1012: renamed from C1008; moved to B.Cu
- C218, C219, C222, C301, C303, C304, C310, C311, C312, C313, C401, C402, C403, C404, C405, C406, C407, C408, C409, C606, C607, C608, C610, C613, C614, C615, C616, C619, C620, D602, D605, R201, R202, R203, R205, R210, R306, R307, R308, R309, R311, R312, R313, R314, R315, R316, R317, R318, R319, R401, R404, R603, R605, R608, R609: moved to B.Cu
- J601: value Conn_02x06_Odd_Even -> Conn_02x04_Odd_Even; footprint Connector_PinHeader_2.54mm:PinHeader_2x06_P2.54mm_Vertical -> Connector_PinHeader_2.54mm:PinHeader_2x04_P2.54mm_Vertical
- moved C409 258.0 mm to (214.1, 82.0), turned to 90 degrees
- moved R406 253.5 mm to (214.1, 82.0), turned to -90 degrees
- moved R405 251.4 mm to (211.5, 87.1)
- moved D403 251.3 mm to (216.7, 82.0), turned to 90 degrees
- moved L401 250.5 mm to (215.4, 87.1), turned to 180 degrees
- moved C406 247.1 mm to (202.6, 81.9), turned to -90 degrees
- moved R404 244.6 mm to (204.9, 81.9), turned to -90 degrees
- moved R403 244.3 mm to (203.8, 87.1)
- moved D402 243.3 mm to (209.7, 82.2)
- moved C311 242.8 mm to (188.0, 101.6), turned to 180 degrees
- moved C408 242.1 mm to (198.1, 80.5), turned to -90 degrees
- moved R402 241.0 mm to (200.3, 87.1)
- moved C407 240.8 mm to (196.6, 80.5), turned to -90 degrees
- moved C312 240.3 mm to (188.0, 95.2), turned to 180 degrees
- moved D401 237.8 mm to (207.8, 87.1)
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- renumbered C1009 to C1013
Connections:
- J601 pad 2: +15VF -> +5V
- J601 pad 4: -15VF -> +3.3V
- J601 pad 7: +5V -> AGNDF
- J601 pad 8: +5V -> AGNDF

Commit message: Hardware
Parts:
- removed the C813 at (-49.6, 188.9)
- removed the C814 at (-49.6, 192.3)
- removed the C817 at (-49.6, 195.6)
- removed C818: 10u/35V, Capacitor_SMD:C_1206_3216Metric_Pad1.33x1.80mm_HandSolder
- removed the FB803 at (-18.0, 70.7)
- removed the FB804 at (-18.0, 73.3)
- removed the R803 at (-13.6, 70.7)
- removed the R804 at (-13.6, 73.3)
- added C815: 10u/35V, Capacitor_Tantalum_SMD:CP_EIA-6032-28_Kemet-C_Pad2.25x2.35mm_HandSolder, F.Cu at (122.3, 67.1)
- added C816: 10u/35V, Capacitor_Tantalum_SMD:CP_EIA-6032-28_Kemet-C_Pad2.25x2.35mm_HandSolder, F.Cu at (122.3, 82.6)
- added R805: 10k, Resistor_SMD:R_0603_1608Metric_Pad0.98x0.95mm_HandSolder, B.Cu at (110.2, 77.9)
- C302, C305, C308, C309, C314, C701, C702, C710, C711, C801, C802, C805, C806, C809, C810, FB703, FB704, FB801, FB802, R320, R321, R704, R705, R709, R714, R801, R802: moved to B.Cu
- C619, C620: value 4u7/50V -> 10u/35V; footprint Capacitor_SMD:C_1206_3216Metric_Pad1.33x1.80mm_HandSolder -> Capacitor_Tantalum_SMD:CP_EIA-6032-28_Kemet-C_Pad2.25x2.35mm_HandSolder; moved to F.Cu
- C627, C628: value 47u/16V -> 10u/35V; footprint Capacitor_SMD:C_1206_3216Metric_Pad1.33x1.80mm_HandSolder -> Capacitor_Tantalum_SMD:CP_EIA-6032-28_Kemet-C_Pad2.25x2.35mm_HandSolder
- C705: footprint Capacitor_SMD:C_1210_3225Metric_Pad1.33x2.70mm_HandSolder -> Capacitor_SMD:C_1206_3216Metric_Pad1.33x1.80mm_HandSolder
- C712: footprint Capacitor_SMD:C_0603_1608Metric_Pad1.08x0.95mm_HandSolder -> Capacitor_Tantalum_SMD:CP_EIA-6032-28_Kemet-C_Pad2.25x2.35mm_HandSolder
- C713, C803, C804: footprint Capacitor_SMD:C_1206_3216Metric_Pad1.33x1.80mm_HandSolder -> Capacitor_Tantalum_SMD:CP_EIA-6032-28_Kemet-C_Pad2.25x2.35mm_HandSolder
- C807, C808: value 100n -> 1u; moved to B.Cu
- C811, C812: value 10u/15V -> 10u/35V; footprint Capacitor_SMD:C_1206_3216Metric_Pad1.33x1.80mm_HandSolder -> Capacitor_Tantalum_SMD:CP_EIA-6032-28_Kemet-C_Pad2.25x2.35mm_HandSolder
- C813: renamed from C815; moved to B.Cu
- C814: renamed from C816; moved to B.Cu
- FB803: renamed from FB805; moved to B.Cu
- FB804: renamed from FB806; moved to B.Cu
- FB805: renamed from FB807; moved to B.Cu
- FB806: renamed from FB808; moved to B.Cu
- R803: renamed from R805; moved to B.Cu
- R804: renamed from R806; moved to B.Cu
- R806: renamed from R807; moved to B.Cu
- R807: renamed from R808; moved to B.Cu
- moved R320 242.4 mm to (197.7, 101.6)
- moved R321 240.1 mm to (197.9, 95.2), turned to 180 degrees
- moved C307 239.2 mm to (183.0, 103.4), turned to -90 degrees
- moved C309 237.9 mm to (183.0, 103.4), turned to -90 degrees
- moved C308 236.2 mm to (180.6, 103.4), turned to -90 degrees
- moved C314 234.6 mm to (197.0, 98.4), turned to 180 degrees
- moved C302 231.9 mm to (172.2, 101.3)
- moved C305 231.8 mm to (175.3, 98.8), turned to -90 degrees
- moved C804 197.4 mm to (113.1, 67.1)
- moved C706 195.2 mm to (121.1, 61.4)
- moved FB301 194.1 mm to (180.6, 103.4), turned to 90 degrees
- moved C811 191.3 mm to (103.2, 67.1)
- moved C803 187.2 mm to (113.0, 82.6), turned to 180 degrees
- moved C812 184.3 mm to (103.2, 82.6), turned to 180 degrees
- moved C708 180.7 mm to (90.5, 51.0), turned to 90 degrees
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- renumbered C819 to C817, R809 to R808
Connections:
- C620 pad 1: -15VF -> AGNDF
- C620 pad 2: AGNDF -> -15VF
- C712 pad 1: Net-(U705C-V-) -> AGNDF
- C712 pad 2: AGNDF -> Net-(U705C-V-)
- C803 pad 1: /DAC/DAC_-15V -> AGNDF
- C803 pad 2: AGNDF -> /DAC/DAC_-15V
- C805 pad 1: Net-(U802-VCC) -> +5V
- C806 pad 1: Net-(U802-IOVCC) -> +3.3V
- C807 pad 1: Net-(U802-VCC) -> +5V
- C808 pad 1: Net-(U802-IOVCC) -> +3.3V
- C811 pad 1: Net-(U802-VCC) -> Net-(U801C-V+)
- C812 pad 1: Net-(U802-IOVCC) -> Net-(U801C-V-)
- U802 pad 10: Net-(U802-IOVCC) -> +3.3V
- U802 pad 9: Net-(U802-VCC) -> +5V

Commit message: Hardware
Parts:
- added J102: MS548-10F, ETH1CREF1A:MS548-10F, F.Cu at (108.0, 62.8)
- C703: moved to B.Cu
- J101: value 36107406S -> MS638-10F; footprint ETH1CREF1A:36107406S -> ETH1CREF1A:MS638-10F
- moved J101 65.9 mm to (172.6, 60.8)
- moved R206 34.2 mm to (74.9, 96.0), turned to 0 degrees
- moved R204 31.9 mm to (74.9, 93.3), turned to 180 degrees
- moved C218 28.1 mm to (79.5, 94.6), turned to -90 degrees
- moved U201 28.1 mm to (79.5, 94.6), turned to 90 degrees
- moved C1013 8.61 mm to (142.7, 56.9)
- moved C1008 7.70 mm to (150.8, 57.0)
- moved U1002 7.70 mm to (147.2, 63.7)
- moved U1001 7.69 mm to (147.1, 69.2)
- moved C1001 7.68 mm to (143.6, 52.7)
- moved C1004 7.68 mm to (145.1, 52.7)
- moved C1002 7.67 mm to (145.0, 59.0)
- moved C1005 7.67 mm to (143.4, 59.0)
- moved C1011 7.67 mm to (149.3, 57.0)
- moved U1003 7.67 mm to (147.2, 58.0)
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