File: HARDWARE/ETH1CREF1A/ETH1CREF1A.kicad_pcb (KiCad board)
At the start: 4 copper layers, 160 x 100 mm, 343 parts, among them J101 MS638-10F, J102 MS548-10F, J1101 Conn_02x04_Odd_Even, J201 Conn_02x01, J202 20021111-00010T4LF, J501 C64AC, J601 Conn_02x04_Odd_Even, J901 Conn_02x06_Odd_Even, K1001 9012, K1002 9012, K1003 9012, K1004 9012, K1005 9012, K1006 9012, K901 9012, K902 9012, K903 9012, K904 9012, K905 9012, K906 9012, K907 9012, K908 9012, K909 9012, K910 9012, K911 9012, K912 9012, K913 9012, K914 9012, K915 9012, K916 9012, K917 9012, K918 9012, Q601 IRFR5410, U1001 DG419DY, U1002 LT5400-3, U1003 ADA4898-2, U1004 AD811JRZ, U1101 74HCT595PW, U1102 74HCT595PW, U1103 74HCT595PW, U1104 74HCT595PW, U1105 SN74LVC1T45DRLR, U1106 SN74LVC1T45DRLR, U1107 SN74LVC1T45DRLR, U1108 SN74LVC1T45DRLR, U201 HDC1080, U202 STM32F429ZIT, U203 24LC08B-E/MS, U301 LAN8742A, U302 LC03-3.3, U303 LC03-3.3, U401 TXB0104PW, U402 ADuM5402, U403 74AC125, U601 MAX5902, U602 LT8330_S6, U603 LT8330_S6, U604 MC7815CD2TG, U605 MC7915CD2TR4G, U606 THL15-2415WI, U607 TSR1-2490, U608 TSR1-2450, U609 LM1117DTX-5/NOPB, U610 LM1117DTX-3.3/NOPB, U701 AD8676BRZ, U702 MAX6350ESA+, U703 LT1021DCS8-7#PBF, U704 LM399H, U705 AD8676BRZ, U801 AD8676BRZ, U802 AD5791ARUZ, U803 AD8675ARZ, Y201 NX5032GA-16.000M, Y301 NX5032GA-25.000000MHZ-LN-CD-1

Commit message: Hardware
Parts:
- added C1113: 100n, Capacitor_SMD:C_0603_1608Metric_Pad1.08x0.95mm_HandSolder, B.Cu at (158.9, 82.7)
- added C1114: 100n, Capacitor_SMD:C_0603_1608Metric_Pad1.08x0.95mm_HandSolder, B.Cu at (167.0, 82.7)
- added R1102: 10k, Resistor_SMD:R_0603_1608Metric_Pad0.98x0.95mm_HandSolder, B.Cu at (167.0, 85.0)
- added R1103: 10k, Resistor_SMD:R_0603_1608Metric_Pad0.98x0.95mm_HandSolder, B.Cu at (158.9, 85.0)
- added R1104: 10k, Resistor_SMD:R_0603_1608Metric_Pad0.98x0.95mm_HandSolder, B.Cu at (150.7, 85.0)
- added R1105: 0, Resistor_SMD:R_0603_1608Metric_Pad0.98x0.95mm_HandSolder, B.Cu at (166.9, 91.4)
- added R1106: 1k, Resistor_SMD:R_0603_1608Metric_Pad0.98x0.95mm_HandSolder, F.Cu at (159.8, 91.6)
- added R1107: 0, Resistor_SMD:R_0603_1608Metric_Pad0.98x0.95mm_HandSolder, F.Cu at (166.9, 91.4)
- added U1109: SN74LVC1T45DRLR, Package_TO_SOT_SMD:SOT-23-6, F.Cu at (164.1, 91.4)
- R1101: value 1k -> 10k; moved to B.Cu
- moved J201 36.0 mm to (135.1, 114.6)
- moved R202 36.0 mm to (135.1, 117.3)
- moved R1101 19.1 mm to (142.6, 85.0), turned to 180 degrees
- moved C1102 16.0 mm to (142.6, 82.7)
- moved C1103 15.4 mm to (164.1, 92.6)
- moved U1102 14.5 mm to (142.6, 84.7)
- moved C1105 14.2 mm to (142.6, 92.6)
- moved U1104 10.4 mm to (150.7, 84.7)
- moved C1106 10.2 mm to (142.6, 90.3)
- moved U1103 10.1 mm to (158.9, 84.7)
- moved C1111 9.04 mm to (157.1, 90.3)
- moved C1108 7.88 mm to (147.6, 90.3)
- moved C1112 7.65 mm to (164.1, 90.3)
- moved C1110 7.50 mm to (152.1, 90.3)
- moved C222 5.46 mm to (136.5, 95.6), turned to 180 degrees
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Connections:
- C1109 pad 1: +5V -> +3.3V
- J1101 pad 2: /GPIO/SPI5_NSS -> /GPIO/SPI5_SCK
- J1101 pad 4: /GPIO/SPI5_SCK -> /GPIO/SPI5_MISO
- J1101 pad 6: /GPIO/SPI5_MISO -> /GPIO/SPI5_MOSI
- J1101 pad 8: /GPIO/SPI5_MOSI -> AGNDF
- R1101 pad 1: Net-(U1108-DIR) -> Net-(U1101-~{OE})
- U1101 pad 13: AGNDF -> Net-(U1101-~{OE})
- U1102 pad 13: AGNDF -> Net-(U1101-~{OE})
- U1103 pad 13: AGNDF -> Net-(U1101-~{OE})
- U1104 pad 13: AGNDF -> Net-(U1101-~{OE})
- U202 pad 18: /GPIO/SPI5_NSS -> unconnected-(U202-PF6,TIM10_CH1,SPI5_NSS,SAI1_SD_B,UART7_RX,FMC_NIORD,EVENTOUT,ADC3_IN4-Pad18)
- U202 pad 70: unconnected-(U202-PB11,TIM2_CH4,I2C2_SDA,USART3_RX,OTG_HS_ULPI_D4,ETH_MII_TX_EN,ETH__RMII_TX_EN,LCD_G5,EVENTOUT-Pad70) -> /GPIO/nOE
