File: HARDWARE/ETH1CREF1A/ETH1CREF1A.kicad_sch (KiCad schematic)
At the start: 0 parts

Commit message: Hardware
Other:
- added sheet Current Source (Current_Source.kicad_sch)
Changed lines of the file:
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@@
+    )
+  )
+  (sheet (at 44.45 43.815) (size 26.67 26.035) (fields_autoplaced)
+    (stroke (width 0.1524) (type solid))
+    (fill (color 0 0 0 0.0000))
+    (property "Sheetname" "Current Source" (at 44.45 43.1034 0)
+      (effects (font (size 1.27 1.27)) (justify left bottom))
+    )
+    (property "Sheetfile" "Current_Source.kicad_sch" (at 44.45 70.4346 0)
+      (effects (font (size 1.27 1.27)) (justify left top))
+    )
+    (instances
+      (project "ETH1CREF1A"
+        (path "/f534bde3-7724-4aa2-8c73-8f0531e01e95" (page "11"))
+      )
     )
   )

Commit message: Hardware
Other:
- removed sheet Isolation
- removed sheet Power Float
- added sheet GPIO (GPIO.kicad_sch)
- added sheet Relays (Relays.kicad_sch)
- sheet Connect ports: added A, B, C, D, E, F; removed none
- sheet Current Source ports: added AOUT, CS_SEL_R10, CS_SEL_R100, CS_SEL_R100k, CS_SEL_R10k, CS_SEL_R1Meg, CS_SEL_R1k, CS_SEL_VSOUR, VOUT; removed none
- title: (none) -> ETH1CREF1A

Commit message: Hardware
Other:
- sheet DAC ports: added REF_+10V, REF_-10V; removed none
- sheet GPIO ports: added CS_SEL_R10, CS_SEL_R100, CS_SEL_R100k, CS_SEL_R10k, CS_SEL_R1Meg, CS_SEL_R1k, CS_SEL_VSOUR, SR_CLK, SR_DAT, SR_LAT, SR_OUT, photoMOS[0..17]; removed none
- sheet MCU ports: added CXN_REL1, CXN_REL2, CXN_REL3, CXN_REL4, CXN_REL5, CXN_REL6; removed none
- sheet Reference Voltage ports: added REF_+10V, REF_-10V; removed none
- sheet Relays ports: added AOUT, CXN_REL1, CXN_REL2, CXN_REL3, CXN_REL4, CXN_REL5, CXN_REL6, photoMOS[0..17]; removed none

Commit message: Hardware and software
Parts:
- added J101: RF_Shield_One_Piece, symbol ETH1CDMM1-rescue:RF_Shield_One_Piece-Device
Connections:
- new net AGNDF: J101.1 (Shield)
Other:
- sheet GPIO ports: added MODE_I2C_SCL, MODE_I2C_SDA, QH, RCLK, SER, SPI5_MISO, SPI5_MOSI, SPI5_NSS, SPI5_SCK, SRCLK, relay[0..17]; removed SR_CLK, SR_DAT, SR_LAT, SR_OUT, photoMOS[0..17]
- sheet MCU ports: added MODE_I2C_SCL, MODE_I2C_SDA; removed SPI1_MISO, SPI1_MOSI, SPI1_NSS, SPI1_SCK, SPI4_MISO, SPI4_MOSI, SPI4_NSS, SPI4_SCK
- sheet Relays ports: added relay[0..17]; removed photoMOS[0..17]

Commit message: Hardware
Parts:
- removed J101: RF_Shield_One_Piece, symbol ETH1CDMM1-rescue:RF_Shield_One_Piece-Device
- added H101, H102, H103: MountingHole, MountingHole:MountingHole_3.2mm_M3_DIN965_Pad_TopBottom, symbol Mechanical:MountingHole
- added J101: RFShield_OnePiece, symbol Device:RFShield_OnePiece
Connections:
- net AGNDF: now also J101.1 (Shield)
Other:
- sheet MCU ports: added none; removed CXN_REL1, CXN_REL2, CXN_REL3, CXN_REL4, CXN_REL5, CXN_REL6
- sheet Relays ports: added none; removed CXN_REL1, CXN_REL2, CXN_REL3, CXN_REL4, CXN_REL5, CXN_REL6
Changed lines of the file:
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@@
-    (stroke (width 0) (type default))
-  )
-  (wire (pts (xy 172.72 64.77) (xy 172.72 71.755))
     (stroke (width 0) (type default))
   )
@@
     (stroke (width 0) (type default))
   )
-  (wire (pts (xy 170.815 64.77) (xy 170.815 71.755))
-    (stroke (width 0) (type default))
-  )
   (wire (pts (xy 193.675 76.835) (xy 200.025 76.835))
     (stroke (width 0) (type default))
@@
     (stroke (width 0) (type default))
   )
-  (wire (pts (xy 165.1 64.77) (xy 165.1 71.755))
-    (stroke (width 0) (type default))
-  )
   (wire (pts (xy 193.675 111.76) (xy 200.025 111.76))
     (stroke (width 0) (type default))
@@
     (stroke (width 0) (type default))
   )
-  (wire (pts (xy 174.625 64.77) (xy 174.625 71.755))
-    (stroke (width 0) (type default))
-  )
   (wire (pts (xy 88.9 109.22) (xy 93.345 109.22))
     (stroke (width 0) (type default))
@@
     (stroke (width 0) (type default))
   )
-  (wire (pts (xy 167.005 64.77) (xy 167.005 71.755))
-    (stroke (width 0) (type default))
-  )
   (wire (pts (xy 132.715 80.01) (xy 137.795 80.01))
     (stroke (width 0) (type default))
@@
     (stroke (width 0) (type default))
   )
-  (wire (pts (xy 168.91 64.77) (xy 168.91 71.755))
-    (stroke (width 0) (type default))
-  )
   (bus (pts (xy 132.715 60.325) (xy 137.795 60.325))
     (stroke (width 0) (type default))
@@
     (stroke (width 0) (type default))
   )
-  (symbol (lib_id "ETH1CDMM1-rescue:RF_Shield_One_Piece-Device") (at 72.39 146.05 0) (unit 1)
-    (in_bom yes) (on_board yes) (dnp no)
-    (property "Reference" "J101" (at 88.392 146.3294 0)
-      (effects (font (size 1.27 1.27)) (justify left))
-    )
-    (property "Value" "RF_Shield_One_Piece" (at 88.392 148.6408 0)
-      (effects (font (size 1.27 1.27)) (justify left))
-    )
-    (property "Footprint" "" (at 72.39 148.59 0)
-      (effects (font (size 1.27 1.27)) hide)
-    )
-    (property "Datasheet" "~" (at 72.39 148.59 0)
+  (symbol (lib_id "Mechanical:MountingHole") (at 31.115 167.005 0) (unit 1)
+    (in_bom yes) (on_board yes) (dnp no) (fields_autoplaced)
+    (property "Reference" "H101" (at 34.29 165.735 0)
+      (effects (font (size 1.27 1.27)) (justify left))
+    )
+    (property "Value" "MountingHole" (at 34.29 168.275 0)
+      (effects (font (size 1.27 1.27)) (justify left))
+    )
+    (property "Footprint" "MountingHole:MountingHole_3.2mm_M3_DIN965_Pad_TopBottom" (at 31.115 167.005 0)
+      (effects (font (size 1.27 1.27)) hide)
+    )
+    (property "Datasheet" "~" (at 31.115 167.005 0)
+      (effects (font (size 1.27 1.27)) hide)
+    )
+    (instances
+      (project "ETH1CREF1A"
+        (path "/f534bde3-7724-4aa2-8c73-8f0531e01e95"
+          (reference "H101") (unit 1)
+        )
+      )
+    )
+  )
+  (symbol (lib_id "Mechanical:MountingHole") (at 31.115 180.975 0) (unit 1)
+    (in_bom yes) (on_board yes) (dnp no) (fields_autoplaced)
+    (property "Reference" "H103" (at 34.29 179.705 0)
+      (effects (font (size 1.27 1.27)) (justify left))
+    )
+    (property "Value" "MountingHole" (at 34.29 182.245 0)
+      (effects (font (size 1.27 1.27)) (justify left))
+    )
+    (property "Footprint" "MountingHole:MountingHole_3.2mm_M3_DIN965_Pad_TopBottom" (at 31.115 180.975 0)
+      (effects (font (size 1.27 1.27)) hide)
+    )
+    (property "Datasheet" "~" (at 31.115 180.975 0)
+      (effects (font (size 1.27 1.27)) hide)
+    )
+    (instances
+      (project "ETH1CREF1A"
+        (path "/f534bde3-7724-4aa2-8c73-8f0531e01e95"
+          (reference "H103") (unit 1)
+        )
+      )
+    )
+  )
+  (symbol (lib_id "Device:RFShield_OnePiece") (at 77.47 171.45 0) (unit 1)
+    (in_bom yes) (on_board yes) (dnp no) (fields_autoplaced)
+    (property "Reference" "J101" (at 93.98 170.18 0)
+      (effects (font (size 1.27 1.27)) (justify left))
+    )
+    (property "Value" "RFShield_OnePiece" (at 93.98 172.72 0)
+      (effects (font (size 1.27 1.27)) (justify left))
+    )
+    (property "Footprint" "" (at 77.47 173.99 0)
+      (effects (font (size 1.27 1.27)) hide)
+    )
+    (property "Datasheet" "~" (at 77.47 173.99 0)
       (effects (font (size 1.27 1.27)) hide)
     )
     (pin "1")
     (instances
-      (project "ETH1CDMM1"
-        (path "/a4468fce-770b-419b-b8ef-3da450c0aad6"
-          (reference "J101") (unit 1)
-        )
-      )
       (project "ETH1CREF1A"
         (path "/f534bde3-7724-4aa2-8c73-8f0531e01e95"
@@
     )
   )
-  (symbol (lib_id "ETH1CDMM1:AGNDF") (at 72.39 156.21 0) (unit 1)
-    (in_bom yes) (on_board yes) (dnp no)
-    (property "Reference" "#PWR0101" (at 72.39 162.56 0)
-      (effects (font (size 1.27 1.27)) hide)
-    )
-    (property "Value" "AGNDF" (at 72.517 160.6042 0)
+  (symbol (lib_id "ETH1CREF1A:AGNDF") (at 77.47 181.61 0) (unit 1)
+    (in_bom yes) (on_board yes) (dnp no) (fields_autoplaced)
+    (property "Reference" "#PWR0101" (at 77.47 187.96 0)
+      (effects (font (size 1.27 1.27)) hide)
+    )
+    (property "Value" "AGNDF" (at 77.47 186.69 0)
       (effects (font (size 1.27 1.27)))
     )
-    (property "Footprint" "" (at 72.39 156.21 0)
-      (effects (font (size 1.27 1.27)) hide)
-    )
-    (property "Datasheet" "" (at 72.39 156.21 0)
+    (property "Footprint" "" (at 77.47 181.61 0)
+      (effects (font (size 1.27 1.27)) hide)
+    )
+    (property "Datasheet" "" (at 77.47 181.61 0)
       (effects (font (size 1.27 1.27)) hide)
     )
     (pin "1")
     (instances
-      (project "ETH1CDMM1"
-        (path "/a4468fce-770b-419b-b8ef-3da450c0aad6"
-          (reference "#PWR0101") (unit 1)
-        )
-      )
       (project "ETH1CREF1A"
         (path "/f534bde3-7724-4aa2-8c73-8f0531e01e95"
@@
     )
   )
+  (symbol (lib_id "Mechanical:MountingHole") (at 31.115 173.99 0) (unit 1)
+    (in_bom yes) (on_board yes) (dnp no) (fields_autoplaced)
+    (property "Reference" "H102" (at 34.29 172.72 0)
+      (effects (font (size 1.27 1.27)) (justify left))
+    )
+    (property "Value" "MountingHole" (at 34.29 175.26 0)
+      (effects (font (size 1.27 1.27)) (justify left))
+    )
+    (property "Footprint" "MountingHole:MountingHole_3.2mm_M3_DIN965_Pad_TopBottom" (at 31.115 173.99 0)
+      (effects (font (size 1.27 1.27)) hide)
+    )
+    (property "Datasheet" "~" (at 31.115 173.99 0)
+      (effects (font (size 1.27 1.27)) hide)
+    )
+    (instances
+      (project "ETH1CREF1A"
+        (path "/f534bde3-7724-4aa2-8c73-8f0531e01e95"
+          (reference "H102") (unit 1)
+        )
+      )
+    )
+  )
   (sheet (at 200.025 106.68) (size 25.4 11.43) (fields_autoplaced)
     (stroke (width 0.1524) (type solid))
@@
       (effects (font (size 1.27 1.27)) (justify left))
     )
-    (pin "CXN_REL3" input (at 168.91 64.77 270)
-      (effects (font (size 1.27 1.27)) (justify left))
-    )
-    (pin "CXN_REL2" input (at 167.005 64.77 270)
-      (effects (font (size 1.27 1.27)) (justify left))
-    )
-    (pin "CXN_REL4" input (at 170.815 64.77 270)
-      (effects (font (size 1.27 1.27)) (justify left))
-    )
-    (pin "CXN_REL1" input (at 165.1 64.77 270)
-      (effects (font (size 1.27 1.27)) (justify left))
-    )
-    (pin "CXN_REL5" input (at 172.72 64.77 270)
-      (effects (font (size 1.27 1.27)) (justify left))
-    )
-    (pin "CXN_REL6" input (at 174.625 64.77 270)
-      (effects (font (size 1.27 1.27)) (justify left))
-    )
     (pin "relay[0..17]" bidirectional (at 137.795 60.325 180)
       (effects (font (size 1.27 1.27)) (justify left))
@@
       (effects (font (size 1.27 1.27)) (justify right))
     )
-    (pin "CXN_REL1" output (at 165.1 71.755 90)
-      (effects (font (size 1.27 1.27)) (justify right))
-    )
-    (pin "CXN_REL3" output (at 168.91 71.755 90)
-      (effects (font (size 1.27 1.27)) (justify right))
-    )
-    (pin "CXN_REL2" output (at 167.005 71.755 90)
-      (effects (font (size 1.27 1.27)) (justify right))
-    )
-    (pin "CXN_REL5" output (at 172.72 71.755 90)
-      (effects (font (size 1.27 1.27)) (justify right))
-    )
-    (pin "CXN_REL6" output (at 174.625 71.755 90)
-      (effects (font (size 1.27 1.27)) (justify right))
-    )
-    (pin "CXN_REL4" output (at 170.815 71.755 90)
-      (effects (font (size 1.27 1.27)) (justify right))
-    )

Commit message: Hardware
Parts:
- J101: value RFShield_OnePiece -> 36107406S; footprint (none) -> ETH1CREF1A:36107406S
Changed lines of the file:
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@@
       (effects (font (size 1.27 1.27)) (justify left))
     )
-    (property "Value" "RFShield_OnePiece" (at 93.98 172.72 0)
+    (property "Value" "36107406S" (at 93.98 172.72 0)
       (effects (font (size 1.27 1.27)) (justify left))
     )
-    (property "Footprint" "" (at 77.47 173.99 0)
+    (property "Footprint" "ETH1CREF1A:36107406S" (at 77.47 173.99 0)
       (effects (font (size 1.27 1.27)) hide)
     )

Commit message: Hardware
Parts:
- added J102: MS548-10F, ETH1CREF1A:MS548-10F, symbol Device:RFShield_OnePiece
- J101: value 36107406S -> MS638-10F; footprint ETH1CREF1A:36107406S -> ETH1CREF1A:MS638-10F
Connections:
- net AGNDF: now also J102.1 (Shield)
Other:
- note added: "3670384 3670548"
Changed lines of the file:
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@@
     (stroke (width 0) (type default))
+  )
+  (text "3670384\n3670548" (at 64.77 160.655 0)
+    (effects (font (size 1.27 1.27)) (justify left bottom))
+  )
+  (symbol (lib_id "Device:RFShield_OnePiece") (at 121.92 171.45 0) (unit 1)
+    (in_bom yes) (on_board yes) (dnp no) (fields_autoplaced)
+    (property "Reference" "J102" (at 138.43 170.18 0)
+      (effects (font (size 1.27 1.27)) (justify left))
+    )
+    (property "Value" "MS548-10F" (at 138.43 172.72 0)
+      (effects (font (size 1.27 1.27)) (justify left))
+    )
+    (property "Footprint" "ETH1CREF1A:MS548-10F" (at 121.92 173.99 0)
+      (effects (font (size 1.27 1.27)) hide)
+    )
+    (property "Datasheet" "~" (at 121.92 173.99 0)
+      (effects (font (size 1.27 1.27)) hide)
+    )
+    (pin "1")
+    (instances
+      (project "ETH1CREF1A"
+        (path "/f534bde3-7724-4aa2-8c73-8f0531e01e95"
+          (reference "J102") (unit 1)
+        )
+      )
+    )
+  )
+  (symbol (lib_id "ETH1CREF1A:AGNDF") (at 121.92 181.61 0) (unit 1)
+    (in_bom yes) (on_board yes) (dnp no) (fields_autoplaced)
+    (property "Reference" "#PWR0102" (at 121.92 187.96 0)
+      (effects (font (size 1.27 1.27)) hide)
+    )
+    (property "Value" "AGNDF" (at 121.92 186.69 0)
+      (effects (font (size 1.27 1.27)))
+    )
+    (property "Footprint" "" (at 121.92 181.61 0)
+      (effects (font (size 1.27 1.27)) hide)
+    )
+    (property "Datasheet" "" (at 121.92 181.61 0)
+      (effects (font (size 1.27 1.27)) hide)
+    )
+    (pin "1")
+    (instances
+      (project "ETH1CREF1A"
+        (path "/f534bde3-7724-4aa2-8c73-8f0531e01e95"
+          (reference "#PWR0102") (unit 1)
+        )
+      )
+    )
   )
   (symbol (lib_id "Mechanical:MountingHole") (at 31.115 167.005 0) (unit 1)
@@
       (effects (font (size 1.27 1.27)) (justify left))
     )
-    (property "Value" "36107406S" (at 93.98 172.72 0)
+    (property "Value" "MS638-10F" (at 93.98 172.72 0)
       (effects (font (size 1.27 1.27)) (justify left))
     )
-    (property "Footprint" "ETH1CREF1A:36107406S" (at 77.47 173.99 0)
+    (property "Footprint" "ETH1CREF1A:MS638-10F" (at 77.47 173.99 0)
       (effects (font (size 1.27 1.27)) hide)
     )

Commit message: Hardware
Other:
- sheet GPIO ports: added nOE; removed SPI5_NSS
- sheet MCU ports: added nOE; removed SPI5_NSS
Changed lines of the file:
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@@
+    (stroke (width 0) (type default))
+  )
+  (wire (pts (xy 132.715 76.2) (xy 137.795 76.2))
     (stroke (width 0) (type default))
   )
@@
     (stroke (width 0) (type default))
   )
-  (wire (pts (xy 132.715 87.63) (xy 137.795 87.63))
+  (wire (pts (xy 132.715 89.535) (xy 137.795 89.535))
     (stroke (width 0) (type default))
   )
@@
   )
   (wire (pts (xy 193.675 92.71) (xy 200.025 92.71))
-    (stroke (width 0) (type default))
-  )
-  (wire (pts (xy 132.715 89.535) (xy 137.795 89.535))
     (stroke (width 0) (type default))
   )
@@
       (effects (font (size 1.27 1.27)) (justify right))
     )
-    (pin "SPI5_SCK" input (at 132.715 87.63 0)
-      (effects (font (size 1.27 1.27)) (justify right))
-    )
-    (pin "SPI5_NSS" input (at 132.715 89.535 0)
+    (pin "SPI5_SCK" input (at 132.715 89.535 0)
       (effects (font (size 1.27 1.27)) (justify right))
     )
@@
       (effects (font (size 1.27 1.27)) (justify right))
     )
+    (pin "nOE" input (at 132.715 76.2 0)
+      (effects (font (size 1.27 1.27)) (justify right))
+    )
     (instances
       (project "ETH1CREF1A"
@@
       (effects (font (size 1.27 1.27)) (justify right))
     )
-    (pin "SPI5_SCK" output (at 137.795 87.63 180)
-      (effects (font (size 1.27 1.27)) (justify left))
-    )
-    (pin "SPI5_NSS" output (at 137.795 89.535 180)
+    (pin "SPI5_SCK" output (at 137.795 89.535 180)
       (effects (font (size 1.27 1.27)) (justify left))
     )
@@
       (effects (font (size 1.27 1.27)) (justify left))
     )
+    (pin "nOE" output (at 137.795 76.2 180)
+      (effects (font (size 1.27 1.27)) (justify left))
+    )
