File: HARDWARE/ETH1CREF1A/ETH1CREF1A.kicad_sch (KiCad schematic)
At the start: 5 parts, among them J101 MS638-10F, J102 MS548-10F

Commit message: Hardware
Other:
- note removed: "3670384 3670548"
Changed lines of the file:
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@@
     (stroke (width 0) (type default))
-  )
-  (text "3670384\n3670548" (at 64.77 160.655 0)
-    (effects (font (size 1.27 1.27)) (justify left bottom))
   )
   (symbol (lib_id "Device:RFShield_OnePiece") (at 121.92 171.45 0) (unit 1)
