File: HARDWARE/ETH1CREF1A/MCU.kicad_sch (KiCad schematic)
At the start: 42 parts, among them J1001 Conn_02x01, J1002 20021111-00010T4LF, U1001 HDC1080, U1002 STM32F746ZG, U1003 24LC08B-E/MS, Y1001 NX5032GA-16.000M

Commit message: Hardware
Connections:
- no-connect marks 47 -> 73

Commit message: Hardware
Parts:
- U1002: footprint ETH1CSMU2:TQFP-144_20x20mm_P0.5mm -> ETH1CREF1A:TQFP-144_20x20mm_P0.5mm
- Y1001: footprint ETH1CSMU2:NX3225GD -> ETH1CREF1A:NX3225GD
Connections:
- net CXN_REL6: now reaches U1002.114 (PD0,DFSDM1_CKIN6,DFSDM1_DATIN7,UART4_RX,CAN1_RX,FMC_D2,EVENTOUT)
- net CXN_REL5: now reaches U1002.115 (PD1,DFSDM1_DATIN6,DFSDM1_CKIN7,UART4_TX,CAN1_TX,FMC_D3,EVENTOUT)
- net CXN_REL4: now reaches U1002.116 (PD2,TRACED2,TIM3_ETR,UART5_RX,SDMMC1_CMD,DCMI_D11,EVENTOUT)
- net CXN_REL3: now reaches U1002.117 (PD3,DFSDM1_CKOUT,SPI2_SCK,I2S2_CK,DFSDM1_DATIN0,USART2_CTS,FMC_CLK,DCMI_D5,LCD_G7,EVENTOUT)
- net CXN_REL2: now reaches U1002.118 (PD4,DFSDM1_CKIN0,USART2_RTS,FMC_NOE,EVENTOUT)
- net CXN_REL1: now reaches U1002.119 (PD5,USART2_TX,FMC_NWE,EVENTOUT)
- no-connect marks 73 -> 69
Changed lines of the file:
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@@
   (no_connect (at 372.11 124.46))
   (no_connect (at 372.11 45.72))
+  (no_connect (at 82.55 147.32))
   (no_connect (at 218.44 267.97))
   (no_connect (at 82.55 63.5))
   (no_connect (at 372.11 88.9))
-  (no_connect (at 372.11 86.36))
-  (no_connect (at 372.11 83.82))
-  (no_connect (at 372.11 81.28))
   (no_connect (at 372.11 96.52))
   (no_connect (at 372.11 147.32))
   (no_connect (at 372.11 149.86))
   (no_connect (at 82.55 71.12))
-  (no_connect (at 372.11 76.2))
   (no_connect (at 372.11 154.94))
   (no_connect (at 372.11 91.44))
@@
   (no_connect (at 372.11 185.42))
   (no_connect (at 82.55 88.9))
-  (no_connect (at 372.11 78.74))
   (no_connect (at 372.11 144.78))
   (no_connect (at 82.55 43.18))
@@
   (no_connect (at 82.55 142.24))
   (no_connect (at 82.55 111.76))
-  (no_connect (at 372.11 73.66))
   (no_connect (at 218.44 270.51))
+  (no_connect (at 82.55 38.1))
   (no_connect (at 82.55 40.64))
   (no_connect (at 372.11 33.02))
@@
     (stroke (width 0) (type default))
   )
+  (wire (pts (xy 372.11 83.82) (xy 373.38 83.82))
+    (stroke (width 0) (type default))
+  )
   (wire (pts (xy 19.05 234.95) (xy 19.05 233.68))
     (stroke (width 0) (type default))
   )
+  (wire (pts (xy 373.38 86.36) (xy 372.11 86.36))
+    (stroke (width 0) (type default))
+  )
   (wire (pts (xy 43.18 275.59) (xy 43.18 276.86))
     (stroke (width 0) (type default))
@@
     (stroke (width 0) (type default))
   )
+  (wire (pts (xy 372.11 78.74) (xy 373.38 78.74))
+    (stroke (width 0) (type default))
+  )
   (wire (pts (xy 242.57 228.6) (xy 242.57 229.87))
     (stroke (width 0) (type default))
@@
     (stroke (width 0) (type default))
   )
+  (wire (pts (xy 373.38 76.2) (xy 372.11 76.2))
+    (stroke (width 0) (type default))
+  )
   (wire (pts (xy 372.11 142.24) (xy 398.78 142.24))
     (stroke (width 0) (type default))
@@
     (stroke (width 0) (type default))
   )
+  (wire (pts (xy 372.11 73.66) (xy 373.38 73.66))
+    (stroke (width 0) (type default))
+  )
   (wire (pts (xy 227.33 21.59) (xy 232.41 21.59))
     (stroke (width 0) (type default))
@@
   )
   (wire (pts (xy 256.54 270.51) (xy 269.24 270.51))
+    (stroke (width 0) (type default))
+  )
+  (wire (pts (xy 373.38 81.28) (xy 372.11 81.28))
     (stroke (width 0) (type default))
   )
@@
     (effects (font (size 1.27 1.27)) (justify right))
   )
+  (hierarchical_label "CXN_REL3" (shape output) (at 373.38 81.28 0) (fields_autoplaced)
+    (effects (font (size 1.27 1.27)) (justify left))
+  )
   (hierarchical_label "RMII_TXD1" (shape bidirectional) (at 373.38 66.04 0) (fields_autoplaced)
     (effects (font (size 1.27 1.27)) (justify left))
@@
     (effects (font (size 1.27 1.27)) (justify right))
   )
+  (hierarchical_label "CXN_REL5" (shape output) (at 373.38 76.2 0) (fields_autoplaced)
+    (effects (font (size 1.27 1.27)) (justify left))
+  )
   (hierarchical_label "TRIG_OUT" (shape output) (at 373.38 137.16 0) (fields_autoplaced)
     (effects (font (size 1.27 1.27)) (justify left))
@@
     (effects (font (size 1.27 1.27)) (justify right))
   )
+  (hierarchical_label "CXN_REL1" (shape output) (at 373.38 86.36 0) (fields_autoplaced)
+    (effects (font (size 1.27 1.27)) (justify left))
+  )
   (hierarchical_label "SPI2_NSS" (shape output) (at 373.38 190.5 0) (fields_autoplaced)
     (effects (font (size 1.27 1.27)) (justify left))
@@
     (effects (font (size 1.27 1.27)) (justify left))
   )
+  (hierarchical_label "CXN_REL4" (shape output) (at 373.38 78.74 0) (fields_autoplaced)
+    (effects (font (size 1.27 1.27)) (justify left))
+  )
   (hierarchical_label "SPI1_MOSI" (shape output) (at 373.38 172.72 0) (fields_autoplaced)
     (effects (font (size 1.27 1.27)) (justify left))
@@
     (effects (font (size 1.27 1.27)) (justify left))
   )
+  (hierarchical_label "CXN_REL2" (shape output) (at 373.38 83.82 0) (fields_autoplaced)
+    (effects (font (size 1.27 1.27)) (justify left))
+  )
   (hierarchical_label "SPI2_SCK" (shape output) (at 373.38 193.04 0) (fields_autoplaced)
     (effects (font (size 1.27 1.27)) (justify left))
@@
   (hierarchical_label "SPI1_SCK" (shape output) (at 81.28 93.98 180) (fields_autoplaced)
     (effects (font (size 1.27 1.27)) (justify right))
+  )
+  (hierarchical_label "CXN_REL6" (shape output) (at 373.38 73.66 0) (fields_autoplaced)
+    (effects (font (size 1.27 1.27)) (justify left))
   )
   (symbol (lib_id "Device:R") (at 39.37 247.65 180) (unit 1)
@@
       (effects (font (size 1.27 1.27)) (justify left))
     )
-    (property "Footprint" "ETH1CSMU2:NX3225GD" (at 49.53 27.94 0)
+    (property "Footprint" "ETH1CREF1A:NX3225GD" (at 49.53 27.94 0)
       (effects (font (size 1.27 1.27)) hide)
     )
@@
       (effects (font (size 1.27 1.27)) (justify left))
     )
-    (property "Footprint" "ETH1CSMU2:TQFP-144_20x20mm_P0.5mm" (at 631.19 87.63 0)
-      (effects (font (size 1.27 1.27)) hide)
-    )
+    (property "Footprint" "ETH1CREF1A:TQFP-144_20x20mm_P0.5mm" (at 631.19 87.63 0)
+      (effects (font (size 1.27 1.27)) hide)
+    )

Commit message: Hardware and software
Parts:
- removed U1002: STM32F746ZG, ETH1CREF1A:TQFP-144_20x20mm_P0.5mm, symbol ETH1CSMU2:STM32F746ZG
- added U202: STM32F429ZIT, ETH1CREF1A:TQFP-144_20x20mm_P0.5mm, symbol ETH1CREF1A:STM32F429ZIT
Connections:
- net +3.3V: now also U202.108 (VDD), U202.121 (VDD), U202.131 (VDD), U202.143 (PDR_ON), U202.144 (VDD), U202.17 (VDD), U202.30 (VDD), U202.39 (VDD), U202.52 (VDD), U202.6 (VBAT), U202.62 (VDD), U202.72 (VDD), U202.84 (VDD), U202.95 (VDDUSB)
- net CXN_REL1: now also U202.119 (PD5,USART2_TX,FMC_NWE,EVENTOUT)
- net CXN_REL2: now also U202.118 (PD4,USART2_RTS,FMC_NOE,EVENTOUT)
- net CXN_REL3: now also U202.117 (PD3,SPI2_SCK,I2S2_CK,USART2_CTS,FMC_CLK,DCMI_D5,LCD_G7,EVENTOUT)
- net CXN_REL4: now also U202.116 (PD2,TIM3_ETR,UART5_RX,SDIO_CMD,DCMI_D11,EVENTOUT)
- net CXN_REL5: now also U202.115 (PD1,CAN1_TX,FMC_D3,EVENTOUT)
- net CXN_REL6: now also U202.114 (PD0,CAN1_RX,FMC_D2,EVENTOUT)
- net EEPROM_SCL: now also U202.11 (PF1,I2C2_SCL,FMC_A1,EVENTOUT)
- net EEPROM_SDA: now also U202.10 (PF0,I2C2_SDA,FMC_A0,EVENTOUT)
- net EEPROM_WP: now also U202.89 (PG4,FMC_A14,FMC_BA0,EVENTOUT)
- net GND: now also U202.107 (VSS), U202.120 (VSS), U202.130 (VSS), U202.16 (VSS), U202.31 (VSSA), U202.38 (VSS), U202.51 (VSS), U202.61 (VSS), U202.83 (VSS), U202.94 (VSS)
- net LED_BLUE: now also U202.48 (PB2,BOOT1,EVENTOUT)
- net LED_GREEN: now also U202.50 (PF12,FMC_A6,EVENTOUT)
- net LED_RED: now also U202.49 (PF11,SPI5_MOSI,FMC_SDNRAS,DCMI_D12,EVENTOUT)
- net MCU_DEFAULT: now also U202.63 (PE10,TIM1_CH2N,FMC_D7,EVENTOUT)
- net MCU_VDDA: now also U202.32 (VREF+), U202.33 (VDDA)
- net NRST: now also U202.25 (NRST)
- net REF_CLK: now also U202.35 (PA1,TIM2_CH2,TIM5_CH2,USART2_RTS,UART4_RX,ETH_MII_RX_CLK,ETH__RMII_REF_CLK,EVENTOUT,ADC1_IN1,ADC2_IN1,ADC3_IN1)
- net RMII_CRS_DV: now also U202.43 (PA7,TIM1_CH1N,TIM3_CH2,TIM8_CH1N,SPI1_MOSI,TIM14_CH1,ETH_MII_RX_DV,ETH__RMII_CRS_DV,EVENTOUT,ADC1_IN7,ADC2_IN7)
- net RMII_MDC: now also U202.27 (PC1,ETH_MDC,EVENTOUT,ADC1_IN11,ADC2_IN11,ADC3_IN11)
- net RMII_MDIO: now also U202.36 (PA2,TIM2_CH3,TIM5_CH3,TIM9_CH1,USART2_TX,ETH_MDIO,EVENTOUT,ADC1_IN2,ADC2_IN2,ADC3_IN2)
- net RMII_RXD0: now also U202.44 (PC4,ETH_MII_RXD0,ETH__RMII_RXD0,EVENTOUT,ADC1_IN14,ADC2_IN14)
- net RMII_RXD1: now also U202.45 (PC5,ETH_MII_RXD1,ETH__RMII_RXD1,EVENTOUT,ADC1_IN15,ADC2_IN15)
- net RMII_TXD0: now also U202.128 (PG13,SPI6_SCK,USART6_CTS,ETH_MII_TXD0,ETH_R_MII_TXD0,FMC_A24,EVENTOUT)
- net RMII_TXD1: now also U202.129 (PG14,SPI6_MOSI,USART6_TX,ETH_MII_TXD1,ETH_R_MII_TXD1,FMC_A25,EVENTOUT)
- net RMII_TXEN: now also U202.126 (PG11,ETH_MII_TX_EN,ETH__RMII_TX_EN,FMC_NCE4_2,DCMI_D3,LCD_B3,EVENTOUT)
- net SENS_SCL: now also U202.136 (PB6,TIM4_CH1,I2C1_SCL,USART1_TX,CAN2_TX,FMC_SDNE1,DCMI_D5,EVENTOUT)
- net SENS_SDA: now also U202.137 (PB7,TIM4_CH2,I2C1_SDA,USART1_RX,FMC_NL,DCMI_VSYNC,EVENTOUT)
- net SPI2_MISO: now also U202.75 (PB14,TIM1_CH2N,TIM8_CH2N,SPI2_MISO,I2S2ext_SD,USART3_RTS,TIM12_CH1,OTG_HS_DM,EVENTOUT)
- net SPI2_MOSI: now also U202.76 (PB15,RTC_REFIN,TIM1_CH3N,TIM8_CH3N,SPI2_MOSI,I2S2_SD,TIM12_CH2,OTG_HS_DP,EVENTOUT)
- net SPI2_NSS: now also U202.73 (PB12,TIM1_BKIN,I2C2_SMBA,SPI2_NSS,I2S2_WS,USART3_CK,CAN2_RX,OTG_HS_ULPI_D5,ETH_MII_TXD0,ETH_R_MII_TXD0,OTG_HS_ID,EVENTOUT)
- net SPI2_SCK: now also U202.74 (PB13,TIM1_CH1N,SPI2_SCK,I2S2_CK,USART3_CTS,CAN2_TX,OTG_HS_ULPI_D6,ETH_MII_TXD1,ETH_R_MII_TXD1,EVENTOUT,OTG_HS_VBUS)
- net SPI3_MISO: now also U202.112 (PC11,I2S3ext_SD,SPI3_MISO,USART3_RX,UART4_RX,SDIO_D3,DCMI_D4,EVENTOUT)
- net SPI3_MOSI: now also U202.113 (PC12,SPI3_MOSI,I2S3_SD,USART3_CK,UART5_TX,SDIO_CK,DCMI_D9,EVENTOUT)
- net SPI3_NSS: now also U202.110 (PA15,JTDI,TIM2_CH1,TIM2_ETR,SPI1_NSS,SPI3_NSS,I2S3_WS,EVENTOUT)
- net SPI3_SCK: now also U202.111 (PC10,SPI3_SCK,I2S3_CK,USART3_TX,UART4_TX,SDIO_D2,DCMI_D8,LCD_R2,EVENTOUT)
- net SPI5_MISO: now also U202.20 (PF8,SPI5_MISO,SAI1_SCK_B,TIM13_CH1,FMC_NIOWR,EVENTOUT,ADC3_IN6)
- net SPI5_MOSI: now also U202.21 (PF9,SPI5_MOSI,SAI1_FS_B,TIM14_CH1,FMC_CD,EVENTOUT,ADC3_IN7)
- net SPI5_NSS: now also U202.18 (PF6,TIM10_CH1,SPI5_NSS,SAI1_SD_B,UART7_RX,FMC_NIORD,EVENTOUT,ADC3_IN4)
- net SPI5_SCK: now also U202.19 (PF7,TIM11_CH1,SPI5_SCK,SAI1_MCLK_B,UART7_TX,FMC_NREG,EVENTOUT,ADC3_IN5)
- net TCK_SWCLK: now also U202.109 (PA14,JTCK-SWCLK,EVENTOUT)
- net TMS_SWDIO: now also U202.105 (PA13,JTMS-SWDIO,EVENTOUT)
- net TRIG_EN: now also U202.60 (PE9,TIM1_CH1,FMC_D6,EVENTOUT)
- net TRIG_IN: now also U202.58 (PE7,TIM1_ETR,UART7_Rx,FMC_D4,EVENTOUT)
- net TRIG_OUT: now also U202.59 (PE8,TIM1_CH1N,UART7_Tx,FMC_D5,EVENTOUT)
- net at C1003.1, Y1001.1: now also U202.23 (PH0,EVENTOUT,OSC_IN)
- net at C1005.1, Y1001.2: now also U202.24 (PH1,EVENTOUT,OSC_OUT)
- net at R1009.1: now also U202.138 (BOOT0)
- net at C1006.1: now also U202.71 (VCAP_1)
- net at C1008.1: now also U202.106 (VCAP_2)
- new net MODE_I2C_SCL: U202.100 (PA8,MCO1,TIM1_CH1,I2C3_SCL,USART1_CK,OTG_FS_SOF,LCD_R6,EVENTOUT)
- new net MODE_I2C_SDA: U202.99 (PC9,MCO2,TIM3_CH4,TIM8_CH4,I2C3_SDA,I2S_CKIN,SDIO_D1,DCMI_D3,EVENTOUT)
- no-connect marks 69 -> 73

Commit message: Hardware
Parts:
- removed FB1001: 742792031, Inductor_SMD:L_0805_2012Metric_Pad1.15x1.40mm_HandSolder, symbol Device:Ferrite_Bead
- added FB301: 600, Inductor_SMD:L_0603_1608Metric_Pad1.05x0.95mm_HandSolder, symbol Device:FerriteBead_Small
Connections:
- net +3.3V: now also FB301.1
- net MCU_VDDA: now also FB301.2
- net CXN_REL1: no longer names the net of U202.119 (PD5,USART2_TX,FMC_NWE,EVENTOUT)
- net CXN_REL2: no longer names the net of U202.118 (PD4,USART2_RTS,FMC_NOE,EVENTOUT)
- net CXN_REL3: no longer names the net of U202.117 (PD3,SPI2_SCK,I2S2_CK,USART2_CTS,FMC_CLK,DCMI_D5,LCD_G7,EVENTOUT)
- net CXN_REL4: no longer names the net of U202.116 (PD2,TIM3_ETR,UART5_RX,SDIO_CMD,DCMI_D11,EVENTOUT)
- net CXN_REL5: no longer names the net of U202.115 (PD1,CAN1_TX,FMC_D3,EVENTOUT)
- net CXN_REL6: no longer names the net of U202.114 (PD0,CAN1_RX,FMC_D2,EVENTOUT)
- no-connect marks 73 -> 79

Commit message: Hardware
Changed lines of the file:
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@@
   )
   (symbol (lib_id "ETH1CREF1A:STM32F429ZIT") (at 227.33 125.73 0) (unit 1)
-    (in_bom yes) (on_board yes) (dnp no) (fields_autoplaced)
-    (property "Reference" "U202" (at 249.6059 226.06 0)
+    (in_bom yes) (on_board yes) (dnp no)
+    (property "Reference" "U202" (at 358.775 24.13 0)
       (effects (font (size 1.27 1.27)) (justify left))
     )
-    (property "Value" "STM32F429ZIT" (at 249.6059 228.6 0)
+    (property "Value" "STM32F429ZIT" (at 353.695 26.67 0)
       (effects (font (size 1.27 1.27)) (justify left))
     )

Commit message: Hardware
Connections:
- net nOE: now reaches U202.70 (PB11,TIM2_CH4,I2C2_SDA,USART3_RX,OTG_HS_ULPI_D4,ETH_MII_TX_EN,ETH__RMII_TX_EN,LCD_G5,EVENTOUT)
- net SPI5_NSS: no longer names the net of U202.18 (PF6,TIM10_CH1,SPI5_NSS,SAI1_SD_B,UART7_RX,FMC_NIORD,EVENTOUT,ADC3_IN4)
Changed lines of the file:
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@@
   (no_connect (at 372.11 55.88))
   (no_connect (at 372.11 53.34))
-  (no_connect (at 372.11 187.96))
+  (no_connect (at 82.55 53.34))
   (no_connect (at 372.11 73.66))
   (no_connect (at 372.11 152.4))
@@
     (stroke (width 0) (type default))
   )
+  (wire (pts (xy 372.11 187.96) (xy 373.38 187.96))
+    (stroke (width 0) (type default))
+  )
   (wire (pts (xy 144.78 259.08) (xy 144.78 256.54))
     (stroke (width 0) (type default))
@@
     (stroke (width 0) (type default))
   )
-  (wire (pts (xy 81.28 53.34) (xy 82.55 53.34))
-    (stroke (width 0) (type default))
-  )
   (wire (pts (xy 232.41 228.6) (xy 232.41 229.87))
     (stroke (width 0) (type default))
@@
   )
   (hierarchical_label "RMII_MDIO" (shape bidirectional) (at 81.28 86.36 180) (fields_autoplaced)
-    (effects (font (size 1.27 1.27)) (justify right))
-  )
-  (hierarchical_label "SPI5_NSS" (shape output) (at 81.28 53.34 180) (fields_autoplaced)
     (effects (font (size 1.27 1.27)) (justify right))
   )
@@
     (effects (font (size 1.27 1.27)) (justify right))
   )
+  (hierarchical_label "nOE" (shape output) (at 373.38 187.96 0) (fields_autoplaced)
+    (effects (font (size 1.27 1.27)) (justify left))
+  )
   (hierarchical_label "TRIG_IN" (shape input) (at 373.38 134.62 0) (fields_autoplaced)
