File: HARDWARE/ETH1CREF1A/Relays.kicad_sch (KiCad schematic)
At the start: 42 parts, among them K901 HE3621A0510, K902 HE3621A0510, K903 HE3621A0510, K904 HE3621A0510, K905 HE3621A0510, K906 HE3621A0510, U909 AQY211G2SX

Commit message: Hardware
Parts:
- added U1201: ULN2003A, Package_SO:TSSOP-16_4.4x5mm_P0.65mm, symbol Transistor_Array:ULN2003A
- K901, K902, K903, K904, K905, K906: footprint (none) -> ETH1CREF1A:HE360_x-5050462-8
- R901, R902, R903, R904, R905, R906, R907, R908, R909, R910, R911, R912, R913, R914, R915, R916, R917, R918: renamed from R?; footprint (none) -> Resistor_SMD:R_0603_1608Metric_Pad0.98x0.95mm_HandSolder
- U909: footprint (none) -> ETH1CREF1A:AQY212GS
Connections:
- net +5V: now also U1201.9 (COM)
- net AGNDF: now also U1201.8 (GND)
- net photoMOS2: now reaches U909.2
- net photoMOS14: now reaches U909.2
- net photoMOS16: now reaches U909.2
- net photoMOS1: now reaches U909.2
- net photoMOS5: now reaches U909.2
- net at K901.3: now also U1201.11 (O6)
- net photoMOS12: now reaches U909.2
- net photoMOS15: now reaches U909.2
- net photoMOS3: now reaches U909.2
- net at K905.3: now also U1201.15 (O2)
- net photoMOS6: now reaches U909.2
- net photoMOS8: now reaches U909.2
- net at K902.3: now also U1201.12 (O5)
- net photoMOS10: now reaches U909.2
- net photoMOS13: now reaches U909.2
- net photoMOS0: now reaches U909.2
- net at K906.3: now also U1201.16 (O1)
- net at K903.3: now also U1201.13 (O4)
- net photoMOS4: now reaches U909.2
- net photoMOS9: now reaches U909.2
- net photoMOS7: now reaches U909.2
- net at K904.3: now also U1201.14 (O3)
- net photoMOS11: now reaches U909.2
- net photoMOS17: now reaches U909.2
- new net CXN_REL1: U1201.6 (I6)
- new net CXN_REL2: U1201.5 (I5)
- new net CXN_REL3: U1201.4 (I4)
- new net CXN_REL4: U1201.3 (I3)
- new net CXN_REL5: U1201.2 (I2)
- new net CXN_REL6: U1201.1 (I1)
- no-connect marks 0 -> 2
Other:
- moved on the sheet: K901B, K902B, K903B, K904B, K905B, K906B, R901, R902, R903, R904, R905, R906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

Commit message: Hardware and software
Parts:
- removed R901, R902, R903, R904, R905, R906, R907, R908, R909, R910, R911, R912, R913, R914, R915, R916, R917, R918: 680, Resistor_SMD:R_0603_1608Metric_Pad0.98x0.95mm_HandSolder, symbol Device:R
- removed U909 (x18): AQY211G2SX, ETH1CREF1A:AQY212GS, symbol ETH1CREF1A:AQY212GS
- added D901, D902, D903, D904, D905, D906, D907, D908, D909, D910, D911, D912, D913, D914, D915, D916, D917, D918: 1N4148W, Diode_SMD:D_SOD-123, symbol Diode:1N4148W
- added J901: Conn_02x06_Odd_Even, Connector_PinHeader_2.54mm:PinHeader_2x06_P2.54mm_Vertical, symbol Connector_Generic:Conn_02x06_Odd_Even
- added K901, K902, K903, K904, K905, K906, K907, K908, K909, K910, K911, K912, K913, K914, K915, K916, K917, K918: 9012, ETH1CREF1A:9012, symbol ETH1CREF1A:9012
- renumbered K901 to K919, K902 to K920, K903 to K921, K904 to K922, K905 to K923, K906 to K924
Connections:
- net +5V: now also D901.1 (K), D902.1 (K), D903.1 (K), D904.1 (K), D905.1 (K), D906.1 (K), D907.1 (K), D908.1 (K), D909.1 (K), D910.1 (K), D911.1 (K), D912.1 (K), D913.1 (K), D914.1 (K), D915.1 (K), D916.1 (K), D917.1 (K), D918.1 (K), K901.2, K902.2, K903.2, K904.2, K905.2, K906.2, K907.2, K908.2, K909.2, K910.2, K911.2, K912.2, K913.2, K914.2, K915.2, K916.2, K917.2, K918.2
- net A: now also J901.1 (Pin_1), J901.2 (Pin_2)
- net AGNDF: now also K913.1, K914.1, K915.1, K916.1, K917.1, K918.1
- net AOUT: now also K907.1, K908.1, K909.1, K910.1, K911.1, K912.1
- net A_AOUT: now also K901.4, K907.4, K913.4
- net B: now also J901.3 (Pin_3), J901.4 (Pin_4)
- net B_AOUT: now also K902.4, K908.4, K914.4
- net C: now also J901.5 (Pin_5), J901.6 (Pin_6)
- net C_AOUT: now also K903.4, K909.4, K915.4
- net D: now also J901.7 (Pin_7), J901.8 (Pin_8)
- net D_AOUT: now also K904.4, K910.4, K916.4
- net E: now also J901.10 (Pin_10), J901.9 (Pin_9)
- net E_AOUT: now also K905.4, K911.4, K917.4
- net F: now also J901.11 (Pin_11), J901.12 (Pin_12)
- net F_AOUT: now also K906.4, K912.4, K918.4
- net VOUT: now also K901.1, K902.1, K903.1, K904.1, K905.1, K906.1
- new net relay0: D901.2 (A), K901.3
- new net relay1: D905.2 (A), K902.3
- new net relay10: D911.2 (A), K911.3
- new net relay11: D914.2 (A), K912.3
- new net relay12: D904.2 (A), K913.3
- new net relay13: D908.2 (A), K914.3
- new net relay14: D915.2 (A), K915.3
- new net relay15: D916.2 (A), K916.3
- new net relay16: D917.2 (A), K917.3
- new net relay17: D918.2 (A), K918.3
- new net relay2: D909.2 (A), K903.3
- new net relay3: D913.2 (A), K904.3
- new net relay4: D902.2 (A), K905.3
- new net relay5: D906.2 (A), K906.3
- new net relay6: D910.2 (A), K907.3
- new net relay7: D912.2 (A), K908.3
- new net relay8: D903.2 (A), K909.3
- new net relay9: D907.2 (A), K910.3
Other:
- moved on the sheet: K919A, K919B, K920A, K920B, K921A, K921B, K922A, K922B, K923A, K923B, K924A, K924B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

Commit message: Hardware
Parts:
- removed K919, K920, K921, K922, K923, K924: HE3621A0510, ETH1CREF1A:HE360_x-5050462-8, symbol ETH1CREF1A:HE3621A0510
- removed U1201: ULN2003A, Package_SO:TSSOP-16_4.4x5mm_P0.65mm, symbol Transistor_Array:ULN2003A
- renumbered D917 to D905, D905 to D906, D906 to D907, D907 to D908, D908 to D909, D918 to D910, D909 to D911, D910 to D912, D911 to D913, D915 to D914, D912 to D915, D913 to D916, D914 to D917, D916 to D918, K905 to K902, K909 to K903, K913 to K904, K917 to K905, K902 to K906, K906 to K907, K910 to K908, K914 to K909, K918 to K910, K903 to K911, K907 to K912, K911 to K913, K915 to K914, K908 to K915, K904 to K916, K912 to K917, K916 to K918
Connections:
- net A_AOUT is gone; now on net A: K901.4, K907.4, K913.4
- net B_AOUT is gone; now on net B: K902.4, K908.4, K914.4
- net C_AOUT is gone; now on net C: K903.4, K909.4, K915.4
- net D_AOUT is gone; now on net D: K904.4, K910.4, K916.4
- net E_AOUT is gone; now on net E: K905.4, K911.4, K917.4
- net F_AOUT is gone; now on net F: K906.4, K912.4, K918.4
- no-connect marks 2 -> 0

Commit message: Hardware
Other:
- moved on the sheet: D912, D914, D915, D918, K912B, K914B, K915B, K918B
